File: Version_2.1/Open-Source_Control_Unitary_V2_R1.brd (EAGLE design)
At the start: 121.9 x 127 mm, 357 parts, among them IC10 MCP6002SMT, IC11 MCP6002SMT, IC12 MCP6002SMT, IC14 MCP6001, IC2 ULN2003AD, IC4 74HC165D, IC5 74HC165D, J24 6p-2.54, K1 JS1-24V-F, K2 JS1-24V-F, K3 JS1-24V-F, K4 JS1-24V-F, K5 JS1-24V-F, Q1 MMBT2907, T4 DA2304-AL, U1 OSD3358-512M-ICB, U16 AT97SC3205T-G3M4400B, U2 TPD4S012_DRY_6_P1_M, U21 S25FL127S, U27 LAN8710, U28 TCAN1051HV, U29 MAX3483EESA+T, U4 APX811-31UGSOT, U40 ISO3086TDW, U5 TLVH431, U6 SN74LVC2G241_DCU_8, X1 10118194-0001LF, X10 MC4, X11 MC4, X12 MC4, X2 J0011D01BNL, X21 MC10, X24 MSTBA2, X3 MC4, X31 MC4, X4 CTI-JTAG, X41 MSTBA3, X5 DM3CS-SF, X6 6p-2.54, X7 TH-2X10, Y7 7A-25.000MAAE-T

Commit message: Add files via upload
Routing:
- net MMC0_DAT0: track 67.6 -> 66.8 mm
- net MMC0_DAT1: track 64.0 -> 63.3 mm
- net MMC0_DAT2: track 61.9 -> 61.2 mm
- net MMC0_CMD: track 63.8 -> 63.1 mm
- net MMC0_CLK: track 63.8 -> 63.1 mm
- net MMC0_DAT3: track 65.5 -> 64.8 mm

Commit message: Add files via upload
Parts:
- removed C93: 0.1uF, 6.3V, OSD3358-BSP Ref Design:C0402
- removed OR281, OR285, OR291, R292, R293, R294: 10K, 1%, OSD3358-SM-RED Platform:R0402
- removed OR35, R36, R37, R38: 1.5K, 1%, OSD3358-BSP Ref Design:R0402
- removed R158: 100K, 1%, OSD3358-BSP Ref Design:R0402
- removed R160, R161: 10K, 1%, OSD3358-BSP Ref Design:R0402
- removed TP27, TP28: TPB0,65, OSD3358-BSP Ref Design:TP_B0,65
- removed TP29, TP30: TPB0,65, OSD3358-SM-RED Platform:TP_B0,65
- removed U21: S25FL127S, OSD3358-BSP Ref Design:W-PDFN-8
Changed lines of the file:
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@@
 <element name="X6" library="OSD3358-BSP Ref Design" package="H6-2.54" value="6p-2.54" x="20.32" y="59.69" smashed="yes" rot="R270">
 <attribute name="MPN" value="P125-1106A1BS116A1" x="20.32" y="59.69" size="1.778" layer="27" rot="R270" display="off"/>
+<attribute name="NAME" x="12.573" y="58.293" size="1.016" layer="25" align="top-left"/>
 <attribute name="NAME" x="17.78" y="59.055" size="0.635" layer="33" ratio="10"/>
-<attribute name="NAME" x="12.573" y="58.293" size="1.016" layer="25" align="top-left"/>
 <attribute name="VALUE" x="20.32" y="59.182" size="0.254" layer="27" align="top-center"/>
 </element>
@@
 <attribute name="NAME" x="86.0044" y="78.74" size="0.8128" layer="25" align="bottom-right"/>
 <attribute name="VALUE" x="87.122" y="78.8416" size="0.254" layer="27" align="top-center"/>
-</element>
-<element name="R36" library="OSD3358-BSP Ref Design" package="R0402" value="1.5K, 1%" x="75.057" y="16.1544" smashed="yes">
-<attribute name="NAME" x="73.914" y="16.1544" size="0.8128" layer="25" align="center-right"/>
-<attribute name="VALUE" x="75.057" y="15.748" size="0.254" layer="27" align="top-center"/>
-</element>
-<element name="R37" library="OSD3358-BSP Ref Design" package="R0402" value="1.5K, 1%" x="75.057" y="17.399" smashed="yes">
-<attribute name="NAME" x="73.914" y="17.399" size="0.8128" layer="25" align="center-right"/>
-<attribute name="VALUE" x="75.057" y="16.9926" size="0.254" layer="27" align="top-center"/>
-</element>
-<element name="R38" library="OSD3358-BSP Ref Design" package="R0402" value="1.5K, 1%" x="75.0316" y="18.5928" smashed="yes">
-<attribute name="NAME" x="73.8886" y="18.5928" size="0.8128" layer="25" align="center-right"/>
-<attribute name="VALUE" x="75.0316" y="18.1864" size="0.254" layer="27" align="top-center"/>
-</element>
-<element name="OR35" library="OSD3358-BSP Ref Design" package="R0402" value="1.5K, 1%" x="75.0824" y="14.9606" smashed="yes">
-<attribute name="NAME" x="73.9394" y="14.9606" size="0.8128" layer="25" align="center-right"/>
-<attribute name="VALUE" x="75.0824" y="14.5542" size="0.254" layer="27" align="top-center"/>
 </element>
 <element name="R69" library="OSD3358-BSP Ref Design" package="R0402" value="100, 1%" x="106.172" y="76.454" smashed="yes">
@@
 <attribute name="VALUE" x="44.45" y="58.3184" size="0.254" layer="27" align="top-center"/>
 </element>
-<element name="U21" library="OSD3358-BSP Ref Design" package="W-PDFN-8" value="S25FL127S" x="76.3778" y="4.445" smashed="yes">
-<attribute name="NAME" x="79.8322" y="7.2136" size="0.8128" layer="25"/>
-<attribute name="VALUE" x="76.3778" y="2.7686" size="0.254" layer="27" align="top-center"/>
-</element>
 <element name="C85" library="OSD3358-BSP Ref Design" package="C0402" value="2200pF, 6.3V" x="48.514" y="60.579" smashed="yes" rot="R270">
 <attribute name="NAME" x="48.514" y="58.8518" size="0.8128" layer="25" rot="R90" align="center-right"/>
@@
 <attribute name="NAME" x="38.735" y="61.6966" size="0.8128" layer="25" rot="R90"/>
 <attribute name="VALUE" x="38.5572" y="60.579" size="0.254" layer="27" rot="R90" align="top-center"/>
-</element>
-<element name="R160" library="OSD3358-BSP Ref Design" package="R0402" value="10K, 1%" x="72.0598" y="3.7084" smashed="yes" rot="R270">
-<attribute name="NAME" x="71.1962" y="3.556" size="0.8128" layer="25" rot="R270" align="top-center"/>
-<attribute name="VALUE" x="71.6534" y="3.7084" size="0.254" layer="27" rot="R270" align="top-center"/>
-</element>
-<element name="R161" library="OSD3358-BSP Ref Design" package="R0402" value="10K, 1%" x="69.9262" y="6.1722" smashed="yes" rot="R90">
-<attribute name="NAME" x="70.358" y="6.2484" size="0.8128" layer="25" rot="R90" align="top-center"/>
-<attribute name="VALUE" x="70.3326" y="6.1722" size="0.254" layer="27" rot="R90" align="top-center"/>
-</element>
-<element name="R158" library="OSD3358-BSP Ref Design" package="R0402" value="100K, 1%" x="72.0598" y="6.0706" smashed="yes" rot="R270">
-<attribute name="NAME" x="71.5518" y="4.953" size="0.8128" layer="25" rot="R90"/>
-<attribute name="VALUE" x="72.4662" y="6.0706" size="0.254" layer="27" rot="R90" align="top-center"/>
-</element>
-<element name="C93" library="OSD3358-BSP Ref Design" package="C0402" value="0.1uF, 6.3V" x="68.8086" y="6.1976" smashed="yes" rot="R90">
-<attribute name="NAME" x="67.7672" y="6.1722" size="0.8128" layer="25" rot="R90" align="top-center"/>
-<attribute name="VALUE" x="69.1134" y="6.1976" size="0.254" layer="27" rot="R90" align="top-center"/>
 </element>
 <element name="U$2" library="OSD3358-BSP Ref Design" package="XYZ-LABEL" value="" x="60.96" y="0.635" smashed="yes"/>
@@
 <attribute name="VALUE" x="68.58" y="88.9" size="0.0254" layer="28" rot="MR0"/>
 </element>
-<element name="TP27" library="OSD3358-BSP Ref Design" package="TP_B0,65" value="TPB0,65" x="68.707" y="3.5814" smashed="yes">
-<attribute name="NAME" x="68.5546" y="1.2954" size="0.8128" layer="25" ratio="10"/>
-<attribute name="VALUE" x="68.707" y="3.175" size="0.0254" layer="27"/>
-</element>
-<element name="TP28" library="OSD3358-BSP Ref Design" package="TP_B0,65" value="TPB0,65" x="67.8434" y="3.5814" smashed="yes">
-<attribute name="NAME" x="66.0654" y="1.2954" size="0.8128" layer="25" ratio="10"/>
-<attribute name="VALUE" x="67.8434" y="3.175" size="0.0254" layer="27"/>
-</element>
 <element name="R10" library="OSD3358-BSP Ref Design" package="R0805" value="0, 1%" x="12.7" y="97.5868" smashed="yes">
 <attribute name="NAME" x="12.319" y="98.7298" size="0.8128" layer="25"/>
 <attribute name="VALUE" x="12.5476" y="96.4184" size="0.254" layer="27"/>
-</element>
-<element name="TP29" library="OSD3358-SM-RED Platform" package="TP_B0,65" value="TPB0,65" x="68.707" y="4.3688" smashed="yes">
-<attribute name="NAME" x="68.5546" y="1.7526" size="0.8128" layer="25" ratio="10"/>
-<attribute name="VALUE" x="68.707" y="3.9624" size="0.0254" layer="27"/>
-</element>
-<element name="TP30" library="OSD3358-SM-RED Platform" package="TP_B0,65" value="TPB0,65" x="67.8434" y="4.3688" smashed="yes">
-<attribute name="NAME" x="66.0654" y="1.8034" size="0.8128" layer="25" ratio="10"/>
-<attribute name="VALUE" x="67.8434" y="3.9624" size="0.0254" layer="27"/>
 </element>
 <element name="U1" library="Octavo-Systems" package="OSD335X-BGA-400" value="OSD3358-512M-ICB" x="60.96" y="88.9" smashed="yes" rot="R270">
@@
 <attribute name="VALUE" x="121.539" y="75.184" size="1.27" layer="27" ratio="10" rot="R90"/>
 </element>
-<element name="OR285" library="OSD3358-SM-RED Platform" package="R0402" value="10K, 1%" x="69.0118" y="14.2748" smashed="yes" rot="R270">
-<attribute name="NAME" x="67.9958" y="14.0208" size="0.8128" layer="25" rot="R90" align="center"/>
-<attribute name="VALUE" x="69.4182" y="14.2748" size="0.254" layer="27" rot="R90" align="top-center"/>
-</element>
-<element name="OR281" library="OSD3358-SM-RED Platform" package="R0402" value="10K, 1%" x="67.8942" y="14.2748" smashed="yes" rot="R90">
-<attribute name="NAME" x="67.0052" y="14.1224" size="0.8128" layer="25" rot="R90" align="center"/>
-<attribute name="VALUE" x="68.3006" y="14.2748" size="0.254" layer="27" rot="R90" align="top-center"/>
-</element>
-<element name="R292" library="OSD3358-SM-RED Platform" package="R0402" value="10K, 1%" x="67.4878" y="19.3802" smashed="yes" rot="R90">
-<attribute name="NAME" x="66.9798" y="18.2626" size="0.8128" layer="25" rot="R90" align="center-right"/>
-<attribute name="VALUE" x="67.8942" y="19.3802" size="0.254" layer="27" rot="R90" align="top-center"/>
-</element>
-<element name="R293" library="OSD3358-SM-RED Platform" package="R0402" value="10K, 1%" x="68.4276" y="19.3802" smashed="yes" rot="R90">
-<attribute name="NAME" x="68.3768" y="16.9164" size="0.8128" layer="25" rot="R90" align="center"/>
-<attribute name="VALUE" x="68.834" y="19.3802" size="0.254" layer="27" rot="R90" align="top-center"/>
-</element>
-<element name="R294" library="OSD3358-SM-RED Platform" package="R0402" value="10K, 1%" x="69.3674" y="19.3802" smashed="yes" rot="R90">
-<attribute name="NAME" x="69.3674" y="16.9418" size="0.8128" layer="25" rot="R90" align="center"/>
-<attribute name="VALUE" x="69.7738" y="19.3802" size="0.254" layer="27" rot="R90" align="top-center"/>
-</element>
-<element name="OR291" library="OSD3358-SM-RED Platform" package="R0402" value="10K, 1%" x="66.548" y="19.3802" smashed="yes" rot="R90">
-<attribute name="NAME" x="66.04" y="18.2626" size="0.8128" layer="25" rot="R90" align="center-right"/>
-<attribute name="VALUE" x="66.9544" y="19.3802" size="0.254" layer="27" rot="R90" align="top-center"/>
-</element>
 <element name="RTC1" library="SparkFun-Clocks" library_urn="urn:adsk.eagle:library:511" package="SO08" package3d_urn="urn:adsk.eagle:package:37530/1" value="DS3231MZ+" x="66.929" y="71.12" smashed="yes" rot="R270">
 <attribute name="NAME" x="66.929" y="74.0918" size="1.016" layer="25" ratio="10" align="bottom-center"/>
@@
 <element name="J24" library="OSD3358-SM-RED Platform" package="H3-2.54" value="6p-2.54" x="98.425" y="104.14" smashed="yes">
 <attribute name="MPN" value="P125-1106A1BS116A1" x="98.425" y="104.14" size="1.778" layer="27" display="off"/>
+<attribute name="NAME" x="99.06" y="101.6" size="0.635" layer="33" ratio="10" rot="R90"/>
 <attribute name="NAME" x="98.425" y="100.1014" size="0.889" layer="25" ratio="10" align="top-center"/>
-<attribute name="NAME" x="99.06" y="101.6" size="0.635" layer="33" ratio="10" rot="R90"/>
 <attribute name="VALUE" x="98.425" y="102.87" size="0.254" layer="27" align="center"/>
 </element>

Commit message: Add files via upload
Parts:
- moved J17 4.44 mm to (114.3, 72.4)
Routing:
- net 24VAC_IN: track 48.0 -> 158.0 mm
- net 24VDC_AUX: track 222.4 -> 277.3 mm, vias 3 -> 7
- net N$111: track 5.55 -> 2.12 mm
- net N$110: track 53.1 -> 53.9 mm, vias 3 -> 1
Changed lines of the file:
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@@
 <layer number="17" name="Pads" color="2" fill="1" visible="yes" active="yes"/>
 <layer number="18" name="Vias" color="2" fill="1" visible="yes" active="yes"/>
-<layer number="19" name="Unrouted" color="6" fill="1" visible="no" active="yes"/>
+<layer number="19" name="Unrouted" color="6" fill="1" visible="yes" active="yes"/>
 <layer number="20" name="Dimension" color="15" fill="1" visible="yes" active="yes"/>
 <layer number="21" name="tPlace" color="6" fill="1" visible="yes" active="yes"/>
@@
 <text x="120.904" y="103.505" size="1.27" layer="21" ratio="20" align="center">10</text>
 <text x="120.904" y="92.71" size="1.27" layer="21" ratio="20" align="center">1</text>
-<text x="112.776" y="72.39" size="1.27" layer="21" ratio="20" align="center-left">BOOT</text>
+<text x="116.713" y="70.866" size="1.27" layer="21" ratio="20" align="top-left">BOOT</text>
 <text x="109.474" y="113.03" size="1.016" layer="21" ratio="20" rot="R90" align="bottom-center">24V</text>
 <text x="109.474" y="118.11" size="1.016" layer="21" ratio="20" rot="R90" align="bottom-center">GND</text>
@@
 <attribute name="VALUE" x="68.072" y="66.8782" size="0.254" layer="27" align="top-center"/>
 </element>
-<element name="J17" library="OSD3358-SM-RED Platform" package="H2-2.54" value="" x="109.855" y="72.39" smashed="yes" rot="R270">
-<attribute name="NAME" x="108.585" y="71.755" size="0.635" layer="33" ratio="10"/>
-<attribute name="NAME" x="112.4966" y="71.0184" size="0.889" layer="25" ratio="11" rot="R180"/>
-<attribute name="VALUE" x="107.95" y="69.85" size="0.889" layer="27" ratio="11"/>
+<element name="J17" library="OSD3358-SM-RED Platform" package="H2-2.54" value="" x="114.3" y="72.39" smashed="yes" rot="R270">
+<attribute name="NAME" x="113.03" y="71.755" size="0.635" layer="33" ratio="10"/>
+<attribute name="NAME" x="111.6584" y="71.0184" size="0.889" layer="25" ratio="11" rot="R180"/>
+<attribute name="VALUE" x="112.395" y="69.85" size="0.889" layer="27" ratio="11"/>
 </element>
 <element name="K1" library="relay" library_urn="urn:adsk.eagle:library:339" package="JS-M" package3d_urn="urn:adsk.eagle:package:24452/1" value="JS1-24V-F" x="95.25" y="49.53" smashed="yes">
@@
 <wire x1="36.3474" y1="86.9696" x2="36.3474" y2="83.9724" width="0.1524" layer="16"/>
 <wire x1="36.3474" y1="83.9724" x2="35.2552" y2="82.8802" width="0.1524" layer="16"/>
-<wire x1="46.6344" y1="57.912" x2="30.988" y2="57.912" width="0.1524" layer="16"/>
-<wire x1="30.988" y1="57.912" x2="29.718" y2="59.182" width="0.1524" layer="16"/>
+<wire x1="46.863" y1="58.166" x2="30.734" y2="58.166" width="0.1524" layer="16"/>
+<wire x1="30.734" y1="58.166" x2="29.718" y2="59.182" width="0.1524" layer="16"/>
 <wire x1="29.718" y1="59.182" x2="29.718" y2="81.6102" width="0.1524" layer="16"/>
 <wire x1="29.718" y1="81.6102" x2="30.988" y2="82.8802" width="0.1524" layer="16"/>
 <wire x1="30.988" y1="82.8802" x2="35.2552" y2="82.8802" width="0.1524" layer="16"/>
-<wire x1="46.6344" y1="57.912" x2="47.5234" y2="58.801" width="0.1524" layer="16"/>
+<wire x1="47.498" y1="58.801" x2="47.5234" y2="58.801" width="0.1524" layer="16"/>
+<wire x1="47.498" y1="58.801" x2="46.863" y2="58.166" width="0.1524" layer="16"/>
 <wire x1="47.5234" y1="58.801" x2="47.1454" y2="59.179" width="0.1524" layer="1"/>
 <wire x1="47.1454" y1="59.179" x2="46.35" y2="59.179" width="0.1524" layer="1"/>
-<wire x1="47.5234" y1="58.801" x2="48.133" y2="58.1914" width="0.1524" layer="16"/>
-<wire x1="67.7164" y1="60.9092" x2="64.9986" y2="58.1914" width="0.1524" layer="16"/>
-<wire x1="48.133" y1="58.1914" x2="64.9986" y2="58.1914" width="0.1524" layer="16"/>
+<wire x1="47.5234" y1="58.801" x2="48.1584" y2="58.166" width="0.1524" layer="16"/>
+<wire x1="67.7164" y1="60.9092" x2="56.388" y2="60.9092" width="0.1524" layer="16"/>
+<wire x1="56.388" y1="60.9092" x2="53.6448" y2="58.166" width="0.1524" layer="16"/>
+<wire x1="48.1584" y1="58.166" x2="53.6448" y2="58.166" width="0.1524" layer="16"/>
 <via x="67.7164" y="60.9092" extent="1-16" drill="0.3048"/>
 <wire x1="67.7164" y1="60.9092" x2="82.9818" y2="60.9092" width="0.1524" layer="1"/>
@@
 <wire x1="102.616" y1="107.95" x2="107.696" y2="113.03" width="1.27" layer="16"/>
 <wire x1="107.696" y1="113.03" x2="111.76" y2="113.03" width="1.27" layer="16"/>
-<wire x1="8.128" y1="58.039" x2="102.616" y2="107.95" width="0" layer="19" extent="1-1"/>
+<wire x1="8.128" y1="58.039" x2="29.1592" y2="58.039" width="1.27" layer="16"/>
+<wire x1="29.1592" y1="58.039" x2="30.2006" y2="56.9976" width="1.27" layer="16"/>
+<wire x1="30.2006" y1="56.9976" x2="54.1782" y2="56.9976" width="1.27" layer="16"/>
+<wire x1="54.1782" y1="56.9976" x2="55.7022" y2="58.5216" width="1.27" layer="16"/>
+<wire x1="106.0196" y1="60.6552" x2="106.0196" y2="65.405" width="1.27" layer="16"/>
+<wire x1="106.0196" y1="65.405" x2="109.22" y2="68.6054" width="1.27" layer="16"/>
+<wire x1="109.22" y1="68.6054" x2="109.22" y2="69.469" width="1.27" layer="16"/>
+<wire x1="55.7022" y1="58.5216" x2="103.886" y2="58.5216" width="1.27" layer="16"/>
+<wire x1="103.886" y1="58.5216" x2="106.0196" y2="60.6552" width="1.27" layer="16"/>
+<wire x1="109.22" y1="69.469" x2="113.919" y2="77.1652" width="0" layer="19" extent="1-16"/>
 </signal>
 <signal name="24VDC_AUX">
@@
 <wire x1="107.761" y1="44.831" x2="109.8423" y2="44.831" width="0.3048" layer="1"/>
 <wire x1="101.95" y1="39.02" x2="107.761" y2="44.831" width="0.3048" layer="1"/>
-<wire x1="95.885" y1="63.373" x2="95.885" y2="58.8518" width="0.8128" layer="16"/>
-<wire x1="95.885" y1="58.8518" x2="99.2068" y2="55.53" width="0.8128" layer="16"/>
-<wire x1="99.2068" y1="55.53" x2="101.95" y2="55.53" width="0.8128" layer="16"/>
 <wire x1="101.95" y1="55.53" x2="101.95" y2="58.801" width="0.3048" layer="1"/>
 <wire x1="101.95" y1="58.801" x2="103.22" y2="60.071" width="0.3048" layer="1"/>
-<wire x1="103.22" y1="60.071" x2="109.1946" y2="60.071" width="0.3048" layer="1"/>
-<wire x1="109.8423" y1="59.4233" x2="109.8423" y2="58.166" width="0.3048" layer="1"/>
-<wire x1="109.1946" y1="60.071" x2="109.8423" y2="59.4233" width="0.3048" layer="1"/>
+<wire x1="103.22" y1="60.071" x2="108.5723" y2="60.071" width="0.3048" layer="1"/>
+<wire x1="108.5723" y1="60.071" x2="109.8423" y2="58.801" width="0.3048" layer="1"/>
+<wire x1="109.8423" y1="58.801" x2="109.8423" y2="58.166" width="0.3048" layer="1"/>
 <wire x1="88.265" y1="108.839" x2="94.488" y2="108.839" width="0.2032" layer="1"/>
 <wire x1="94.488" y1="108.839" x2="95.758" y2="110.109" width="0.2032" layer="1"/>
@@
 <wire x1="95.885" y1="63.373" x2="96.266" y2="63.754" width="0.8128" layer="16"/>
 <wire x1="98.425" y1="101.6" x2="96.266" y2="99.441" width="0.8128" layer="16"/>
+<wire x1="97.282" y1="63.754" x2="96.901" y2="63.373" width="0.8128" layer="16"/>
+<via x="102.616" y="63.754" extent="1-16" drill="0.3048"/>
+<via x="101.6" y="63.754" extent="1-16" drill="0.3048"/>
+<wire x1="101.6" y1="63.754" x2="97.282" y2="63.754" width="0.8128" layer="16"/>
+<polygon width="0.254" layer="16">
+<vertex x="102.87" y="64.262"/>
+<vertex x="101.346" y="64.262"/>
+<vertex x="101.092" y="64.008"/>
+<vertex x="101.092" y="62.484"/>
+<vertex x="101.346" y="62.23"/>
+<vertex x="102.87" y="62.23"/>
+<vertex x="103.124" y="62.484"/>
+<vertex x="103.124" y="64.008"/>
+</polygon>
+<polygon width="0.254" layer="1">
+<vertex x="102.87" y="62.23"/>
+<vertex x="101.346" y="62.23"/>
+<vertex x="101.092" y="62.484"/>
+<vertex x="101.092" y="64.008"/>
+<vertex x="101.346" y="64.262"/>
+<vertex x="102.87" y="64.262"/>
+<vertex x="103.124" y="64.008"/>
+<vertex x="103.124" y="62.484"/>
+</polygon>
+<via x="102.616" y="62.738" extent="1-16" drill="0.3048"/>
+<via x="101.6" y="62.738" extent="1-16" drill="0.3048"/>
+<wire x1="102.616" y1="62.738" x2="104.14" y2="61.214" width="0.8128" layer="1"/>
+<wire x1="109.474" y1="61.214" x2="110.871" y2="59.817" width="0.8128" layer="1"/>
+<wire x1="110.871" y1="59.817" x2="110.871" y2="9.4742" width="0.8128" layer="1"/>
+<wire x1="110.871" y1="9.4742" x2="109.093" y2="7.6962" width="0.8128" layer="1"/>
+<wire x1="104.14" y1="61.214" x2="109.474" y2="61.214" width="0.8128" layer="1"/>
+<wire x1="109.474" y1="61.214" x2="108.5723" y2="60.071" width="0" layer="19" extent="1-1"/>
 </signal>
 <signal name="N$93">
@@
 <wire x1="68.072" y1="69.977" x2="68.072" y2="61.9252" width="0.3048" layer="16"/>
 <wire x1="68.072" y1="61.9252" x2="69.469" y2="60.5282" width="0.3048" layer="16"/>
-<wire x1="69.469" y1="60.5282" x2="88.646" y2="60.5282" width="0.3048" layer="16"/>
 <wire x1="68.072" y1="69.977" x2="68.58" y2="70.485" width="0.3048" layer="16"/>
-<via x="97.282" y="60.5282" extent="1-16" drill="0.3048"/>
-<via x="88.646" y="60.5282" extent="1-16" drill="0.3048"/>
-<wire x1="97.282" y1="60.5282" x2="88.646" y2="60.5282" width="0.3048" layer="1"/>
-<wire x1="97.282" y1="60.5282" x2="101.6" y2="60.5282" width="0.254" layer="16"/>
-<wire x1="101.6" y1="60.5282" x2="104.14" y2="63.0682" width="0.254" layer="16"/>
-<wire x1="104.14" y1="63.0682" x2="104.14" y2="68.58" width="0.254" layer="16"/>
+<wire x1="69.469" y1="60.5282" x2="102.87" y2="60.5282" width="0.3048" layer="16"/>
+<wire x1="102.87" y1="60.5282" x2="104.14" y2="61.7982" width="0.3048" layer="16"/>
+<wire x1="104.14" y1="61.7982" x2="104.14" y2="68.58" width="0.3048" layer="16"/>
 </signal>
 <signal name="RTC_RST">
@@
 <wire x1="106.7308" y1="76.454" x2="107.95" y2="76.454" width="0.1524" layer="1"/>
 <wire x1="107.95" y1="76.454" x2="108.585" y2="75.819" width="0.1524" layer="1"/>
-<wire x1="108.585" y1="75.819" x2="108.585" y2="72.39" width="0.1524" layer="1"/>
+<wire x1="108.585" y1="75.819" x2="113.03" y2="72.39" width="0" layer="19" extent="1-1"/>
 </signal>
 <signal name="BO1_NO">

Commit message: Add files via upload
Parts:
- R1, R2: value 1.5K, 1% -> 1K
- R168, R171, R172, R173, R174, R175: value 10K, 1% -> 10K
Routing:
- net 24VDC_AUX: track 277.3 -> 112.3 mm
- net 24VAC_IN: track 158.0 -> 11.2 mm, vias 0 -> 9
- net GND: track 206.9 -> 163.5 mm
- net N$111: track 2.12 -> 7.98 mm
- net LCD_DATA2: track 46.8 -> 46.3 mm
- added copper zone on layer 1, net 24VAC_IN
- added copper zone on layer 16, net 24VAC_IN

Commit message: Add files via upload
Parts:
- removed D20, D21: SMBJ7.0CA, diode:SMBJ
- added D9: CDSOT23-T24CAN, OSD3358-SM-RED Platform:SOT23-3
- added OIC14: MCP6001, adam - ics:SOT23-5
- C11: value 220uF, 6.3V T491C227K006AT -> 220uF, 6.3V, T491C227K006AT
- C406: value 4.7uF, 16V -> 4.7uF, 16V, T491A475K016AT; device SparkFun-Capacitors:1206 -> OSD3358-SM-RED Platform:A/3216-18R
- IC14: value MCP6001 -> MCP6002SMT; device adam - ics:SOT23-5 -> adam - ics:SOIC8
- moved C7 76.4 mm to (66.8, 5.84), turned to 90 degrees
- moved IC14 75.1 mm to (-13.1, -10.3), turned to 0 degrees
- moved D8 29.2 mm to (101.1, 3.81), turned to 270 degrees
- moved R1 28.6 mm to (99.1, 3.81), turned to 90 degrees
- moved D2 28.4 mm to (103.1, 3.81), turned to 270 degrees
- moved R2 24.0 mm to (97.0, 3.81), turned to 90 degrees
- moved U28 11.2 mm to (72.4, 5.84), turned to 0 degrees
- turned C406 to 270 degrees
Connections:
- new net N$16: OIC14.1, OIC14.4
- new net V+: IC14.8
- new net V-: IC14.4
- net 1P8V_REF: no longer IC14.1, IC14.4
- net AGND: now also OIC14.2; no longer IC14.2
- net CAN_H: now also D9.2; no longer D20.C
- net CAN_L: now also D9.1; no longer D21.C
- net CGND: no longer D20.A, D21.A
- net GND: now also C7.2
- net ISO_GND: now also C406.-; no longer C406.2
- net ISO_VCC: now also C406.+; no longer C406.1
- net SYS_ADC_1P8V: now also OIC14.3; no longer IC14.3
- net SYS_VDD1_3P3V: now also C7.1, OIC14.5; no longer IC14.5
Routing:
- net CAN1_TXD: track 45.2 -> 239.6 mm, vias 0 -> 2
- net CAN1_RXD: track 43.7 -> 225.9 mm, vias 0 -> 2
- net CAN_L: track 0.00 -> 35.3 mm
- net CAN_H: track 0.00 -> 34.8 mm
- net N$6: track 0.09 -> 7.03 mm
- net GND: track 163.5 -> 168.7 mm, vias 185 -> 187
- net 1P8V_REF: track 238.0 -> 234.2 mm
- net N$16: track 0.00 -> 3.76 mm
- net SYS_VDD1_3P3V: track 78.5 -> 81.6 mm, vias 38 -> 39
- net N$5: track 0.09 -> 2.11 mm
Other:
- board text added: "24"
- board text added: "VDC"
- board text removed: "24VDC"
