File: Version_2.1/Open-Source_Control_Unitary_V2_R1.brd (EAGLE design)
At the start: 121.9 x 127 mm, 338 parts, among them IC10 MCP6002SMT, IC11 MCP6002SMT, IC12 MCP6002SMT, IC14 MCP6002SMT, IC2 ULN2003AD, IC4 74HC165D, IC5 74HC165D, J24 6p-2.54, K1 JS1-24V-F, K2 JS1-24V-F, K3 JS1-24V-F, K4 JS1-24V-F, K5 JS1-24V-F, Q1 MMBT2907, T4 DA2304-AL, U1 OSD3358-512M-ICB, U16 AT97SC3205T-G3M4400B, U2 TPD4S012_DRY_6_P1_M, U27 LAN8710, U28 TCAN1051HV, U29 MAX3483EESA+T, U4 APX811-31UGSOT, U40 ISO3086TDW, U5 TLVH431, U6 SN74LVC2G241_DCU_8, X1 10118194-0001LF, X10 MC4, X11 MC4, X12 MC4, X2 J0011D01BNL, X21 MC10, X24 MSTBA2, X3 MC4, X31 MC4, X4 CTI-JTAG, X41 MSTBA3, X5 DM3CS-SF, X6 6p-2.54, X7 TH-2X10, Y7 7A-25.000MAAE-T

Commit message: Add files via upload
Parts:
- removed OIC14: MCP6001, adam - ics:SOT23-5
- moved IC14 76.8 mm to (56.9, 21.3), turned to 180 degrees
- renumbered C7 to C801, D2 to D801, D8 to D802, D9 to D805, R1 to R802, R2 to R801, X31 to X8
Connections:
- removed net 1P8V_REF: IC10.8, IC11.8, IC12.8, R212.2, R222.2, R232.2, R242.2, R252.2, R262.2
- removed net N$16: OIC14.1, OIC14.4
- removed net V+: IC14.8
- removed net V-: IC14.4
- new net 1P8V_REF_1: IC10.8, IC11.8, IC14.1, IC14.2, R212.2, R222.2, R232.2, R242.2
- new net 1P8V_REF_2: IC12.8, IC14.6, IC14.7, R252.2, R262.2
- net 24VDC_AUX: now also X8.4
- net AGND: now also IC14.4, R181.2, R182.2, R183.2, R184.2, R185.2, R186.2; no longer OIC14.2
- net CAN_H: now also X8.2
- net CAN_L: now also X8.1
- net CGND: no longer R181.2, R182.2, R183.2, R184.2, R185.2, R186.2
- net GND: now also D805.3, X8.3
- net SYS_ADC_1P8V: now also IC14.3, IC14.5; no longer OIC14.3
- net SYS_VDD1_3P3V: now also IC14.8; no longer OIC14.5
Routing:
- net 1P8V_REF: track 234.2 -> 0.00 mm, vias 12 -> 0
- net 1P8V_REF_1: track 0.00 -> 123.7 mm, vias 0 -> 8
- net 1P8V_REF_2: track 0.00 -> 54.7 mm, vias 0 -> 4
- net CGND: track 71.9 -> 20.0 mm
- net AGND: track 139.8 -> 168.9 mm
- net CAN_H: track 34.8 -> 40.7 mm
- net CAN_L: track 35.3 -> 40.5 mm
- net SYS_ADC_1P8V: track 72.3 -> 68.2 mm
- net N$16: track 3.76 -> 0.00 mm
- net AIN5: track 73.7 -> 72.1 mm
- net GND: track 168.7 -> 169.8 mm, vias 187 -> 188
- net N$129: track 125.6 -> 124.9 mm
- net SYS_VDD1_3P3V: track 81.6 -> 82.1 mm
- removed copper zone on layer 1, net 1P8V_REF

Commit message: Add files via upload
Routing:
- net 1P8V_REF_1: track 123.7 -> 143.7 mm
- net 1P8V_REF_2: track 54.7 -> 69.3 mm
- net AIN6: track 82.3 -> 84.9 mm
- net SYS_ADC_1P8V: track 68.2 -> 70.3 mm
- net AIN5: track 72.1 -> 70.7 mm
- net AIN3: track 55.2 -> 54.2 mm
- net AIN2: track 47.3 -> 48.0 mm
