File: Version_2.1/Open-Source_Control_Unitary_V2_R1.brd (EAGLE design)
At the start: 121.9 x 127 mm, 337 parts, among them IC10 MCP6002SMT, IC11 MCP6002SMT, IC12 MCP6002SMT, IC14 MCP6002SMT, IC2 ULN2003AD, IC4 74HC165D, IC5 74HC165D, J24 6p-2.54, K1 JS1-24V-F, K2 JS1-24V-F, K3 JS1-24V-F, K4 JS1-24V-F, K5 JS1-24V-F, Q1 MMBT2907, T4 DA2304-AL, U1 OSD3358-512M-ICB, U16 AT97SC3205T-G3M4400B, U2 TPD4S012_DRY_6_P1_M, U27 LAN8710, U28 TCAN1051HV, U29 MAX3483EESA+T, U4 APX811-31UGSOT, U40 ISO3086TDW, U5 TLVH431, U6 SN74LVC2G241_DCU_8, X1 10118194-0001LF, X10 MC4, X11 MC4, X12 MC4, X2 J0011D01BNL, X21 MC10, X24 MSTBA2, X3 MC4, X4 CTI-JTAG, X41 MSTBA3, X5 DM3CS-SF, X6 6p-2.54, X7 TH-2X10, X8 MC4, Y7 7A-25.000MAAE-T

Commit message: Add files via upload
Parts:
- added J4, J5, J6: (no value), OSD3358-SM-RED Platform:H2-2.54
- moved U$1 6.35 mm to (66.0, 16.5)
- turned J3 to 90 degrees
- renumbered J17 to J3
Connections:
- net EHRPWM1A: now also J4.1
- net EHRPWM2A: now also J5.1
- net EHRPWM2B: now also J6.1
- net GND: now also J3.2, J4.2, J5.2, J6.2; no longer J3.1
- net N$111: now also J3.1; no longer J3.2
Routing:
- net EHRPWM1A: track 109.2 -> 118.3 mm, vias 3 -> 2
- net EHRPWM2A: track 107.2 -> 113.1 mm, vias 3 -> 2
- net MMC0_DAT2: track 61.2 -> 56.5 mm
- net MMC0_DAT3: track 64.8 -> 60.7 mm
- net MMC0_CMD: track 63.1 -> 59.5 mm
- net EHRPWM2B: track 107.2 -> 110.6 mm, vias 3 -> 2
- net MMC0_CD: track 78.1 -> 75.9 mm
- net MMC0_CLK: track 63.1 -> 61.8 mm
- net MMC0_DAT1: track 63.3 -> 62.0 mm
- net MMC0_DAT0: track 66.8 -> 65.5 mm

Commit message: Add files via upload
Parts:
- added TP17, TP18, TP19, TP20: TESTPAD/W_HOLE_1X1, OSD3358-SM-RED Platform:TESTPAD/W_HOLE_1X1
- moved R163 2.48 mm to (65.8, 66.3), turned to 0 degrees
- moved C104 2.43 mm to (68.0, 67.3), turned to 0 degrees
- moved R170 1.02 mm to (68.0, 66.3)
- moved R169 1.02 mm to (68.0, 65.3)
Connections:
- removed net OSC1_GND: RTC1.5, U1.W13
- net GND: now also RTC1.5, U1.W13
- net I2C0_SCL: now also TP18.P$1
- net I2C0_SDA: now also TP17.P$1
- net I2C1_SCL: now also TP20.P$1
- net I2C1_SDA: now also TP19.P$1
Routing:
- net GND: track 169.8 -> 184.2 mm
- net OSC1_GND: track 12.9 -> 0.00 mm
- net I2C1_SCL: track 33.0 -> 38.4 mm
- net I2C1_SDA: track 29.3 -> 33.6 mm
- net I2C0_SCL: track 33.8 -> 35.2 mm
- net RTC_RST: track 52.8 -> 53.9 mm, vias 3 -> 2
- net SYS_VDD1_3P3V: track 82.1 -> 81.4 mm, vias 39 -> 40
