File: Version_2.1/Open-Source_Control_Unitary_V2_R1.sch (EAGLE design)
At the start: 355 parts, among them IC10 MCP6002SMT, IC11 MCP6002SMT, IC12 MCP6002SMT, IC14 MCP6001, IC2 ULN2003AD, IC4 74HC165D, IC5 74HC165D, J24 6p-2.54, K1 JS1-24V-F, K2 JS1-24V-F, K3 JS1-24V-F, K4 JS1-24V-F, K5 JS1-24V-F, Q1 MMBT2907, T4 DA2304-AL, U1 OSD3358-512M-ICB, U16 AT97SC3205T-G3M4400B, U2 TPD4S012_DRY_6_P1_M, U21 S25FL127S, U27 LAN8710, U28 TCAN1051HV, U29 MAX3483EESA+T, U4 APX811-31UGSOT, U40 ISO3086TDW, U5 TLVH431, U6 SN74LVC2G241_DCU_8, X1 10118194-0001LF, X10 MC4, X11 MC4, X12 MC4, X2 J0011D01BNL, X21 MC10, X24 MSTBA2, X3 MC4, X31 MC4, X4 CTI-JTAG, X41 MSTBA3, X5 DM3CS-SF, X6 6p-2.54, X7 TH-2X10, Y7 7A-25.000MAAE-T

Commit message: Add files via upload
Other:
- note added: "Reset supervisor circuit: Reset asserted if VCC drops below V threshold, push button or POR. De-asserted after 240ms"
- note removed: "Reset supervisor circuit"
- moved on the sheet: X31.1, X31.2, X31.3, X31.4
Changed lines of the file:
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@@
 paper in landscape;
 0.69 scaling factor.</text>
-<text x="63.5" y="38.1" size="2.54" layer="150" rot="MR0">Reset supervisor circuit</text>
+<text x="71.12" y="30.48" size="2.54" layer="150" rot="MR0">Reset supervisor circuit:
+Reset asserted if VCC
+drops below V threshold,
+push button or POR.
+De-asserted after 240ms</text>
 <text x="10.16" y="121.92" size="2.54" layer="150">The OSD335x-SM contains
 4.7k pull-up resistors on I2C0.
@@
 <attribute name="VALUE" x="485.14" y="322.58" size="1.778" layer="96" align="top-right"/>
 </instance>
-<instance part="X31" gate=".1" x="1089.66" y="787.4" smashed="yes">
-<attribute name="NAME" x="1082.04" y="789.305" size="1.524" layer="95"/>
-</instance>
-<instance part="X31" gate=".2" x="1089.66" y="782.32" smashed="yes">
-<attribute name="NAME" x="1082.04" y="784.225" size="1.524" layer="95"/>
-</instance>
-<instance part="X31" gate=".3" x="1089.66" y="777.24" smashed="yes">
-<attribute name="NAME" x="1082.04" y="779.145" size="1.524" layer="95"/>
-</instance>
-<instance part="X31" gate=".4" x="1089.66" y="772.16" smashed="yes">
-<attribute name="NAME" x="1082.04" y="774.065" size="1.524" layer="95"/>
+<instance part="X31" gate=".1" x="1087.12" y="805.18" smashed="yes">
+<attribute name="NAME" x="1079.5" y="807.085" size="1.524" layer="95"/>
+</instance>
+<instance part="X31" gate=".2" x="1087.12" y="800.1" smashed="yes">
+<attribute name="NAME" x="1079.5" y="802.005" size="1.524" layer="95"/>
+</instance>
+<instance part="X31" gate=".3" x="1087.12" y="795.02" smashed="yes">
+<attribute name="NAME" x="1079.5" y="796.925" size="1.524" layer="95"/>
+</instance>
+<instance part="X31" gate=".4" x="1087.12" y="789.94" smashed="yes">
+<attribute name="NAME" x="1079.5" y="791.845" size="1.524" layer="95"/>
 </instance>
 <instance part="U29" gate="A" x="883.92" y="807.72" smashed="yes">

Commit message: Add files via upload
Parts:
- removed C93: 0.1uF, 6.3V, OSD3358-SM-RED Platform:CC0402
- removed OR281, OR285, OR291, R160, R161, R292, R293, R294: 10K, 1%, OSD3358-SM-RED Platform:R-US_R0402
- removed OR35, R36, R37, R38: 1.5K, 1%, OSD3358-SM-RED Platform:R-US_R0402
- removed R158: 100K, 1%, OSD3358-SM-RED Platform:R-US_R0402
- removed TP27, TP28, TP29, TP30: TPB0,65, OSD3358-SM-RED Platform:TPB0,65
- removed U21: S25FL127S, OSD3358-SM-RED Platform:S25FL127S
Other:
- note removed: "There are many footprint compatible (8-WSON) parts for the NOR flash if the listed part is not available."

Commit message: Add files via upload
Parts:
- R1, R2: value 1.5K, 1% -> 1K
- R168, R171, R172, R173, R174, R175: value 10K, 1% -> 10K
Other:
- moved on the sheet: C7
Changed lines of the file:
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@@
 <part name="GND125" library="OSD3358-SM-RED Platform" deviceset="GND" device=""/>
 <part name="GND126" library="OSD3358-SM-RED Platform" deviceset="GND" device=""/>
-<part name="R168" library="OSD3358-SM-RED Platform" deviceset="R-US_" device="R0402" value="10K, 1%"/>
+<part name="R168" library="OSD3358-SM-RED Platform" deviceset="R-US_" device="R0402" value="10K"/>
 <part name="D19" library="OSD3358-SM-RED Platform" deviceset="LTST-C191KRKT" device="LED_EIA-STD" value="LTST-C191KRKT"/>
 <part name="GND128" library="OSD3358-SM-RED Platform" deviceset="GND" device=""/>
@@
 <part name="D34" library="OSD3358-SM-RED Platform" deviceset="LTST-C191KRKT" device="LED_EIA-STD" value="LTST-C191KRKT"/>
 <part name="D35" library="OSD3358-SM-RED Platform" deviceset="LTST-C191KRKT" device="LED_EIA-STD" value="LTST-C191KRKT"/>
-<part name="R173" library="OSD3358-SM-RED Platform" deviceset="R-US_" device="R0402" value="10K, 1%"/>
-<part name="R174" library="OSD3358-SM-RED Platform" deviceset="R-US_" device="R0402" value="10K, 1%"/>
-<part name="R175" library="OSD3358-SM-RED Platform" deviceset="R-US_" device="R0402" value="10K, 1%"/>
-<part name="R172" library="OSD3358-SM-RED Platform" deviceset="R-US_" device="R0402" value="10K, 1%"/>
-<part name="R171" library="OSD3358-SM-RED Platform" deviceset="R-US_" device="R0402" value="10K, 1%"/>
+<part name="R173" library="OSD3358-SM-RED Platform" deviceset="R-US_" device="R0402" value="10K"/>
+<part name="R174" library="OSD3358-SM-RED Platform" deviceset="R-US_" device="R0402" value="10K"/>
+<part name="R175" library="OSD3358-SM-RED Platform" deviceset="R-US_" device="R0402" value="10K"/>
+<part name="R172" library="OSD3358-SM-RED Platform" deviceset="R-US_" device="R0402" value="10K"/>
+<part name="R171" library="OSD3358-SM-RED Platform" deviceset="R-US_" device="R0402" value="10K"/>
 <part name="GND39" library="OSD3358-SM-RED Platform" deviceset="GND" device=""/>
 <part name="U$8" library="OSD3358-SM-RED Platform" deviceset="24VDC_AUX" device=""/>
@@
 <part name="D2" library="OSD3358-SM-RED Platform" deviceset="LTST-C191KFKT" device="LED_EIA-STD" value="LTST-C191KFKT"/>
 <part name="D8" library="OSD3358-SM-RED Platform" deviceset="LTST-C191KGKT" device="LED_EIA-STD" value="LTST-C191KGKT"/>
-<part name="R1" library="OSD3358-SM-RED Platform" deviceset="R-US_" device="R0402" value="1.5K, 1%"/>
-<part name="R2" library="OSD3358-SM-RED Platform" deviceset="R-US_" device="R0402" value="1.5K, 1%"/>
+<part name="R1" library="OSD3358-SM-RED Platform" deviceset="R-US_" device="R0402" value="1K"/>
+<part name="R2" library="OSD3358-SM-RED Platform" deviceset="R-US_" device="R0402" value="1K"/>
 <part name="GND1" library="OSD3358-SM-RED Platform" deviceset="GND" device=""/>
 <part name="GND2" library="OSD3358-SM-RED Platform" deviceset="GND" device=""/>
@@
 <attribute name="VALUE" x="939.8" y="779.78" size="1.778" layer="96"/>
 </instance>
-<instance part="C7" gate="G$1" x="899.16" y="660.4" smashed="yes">
-<attribute name="NAME" x="891.54" y="657.86" size="1.778" layer="95"/>
-<attribute name="VALUE" x="883.92" y="655.32" size="1.778" layer="96"/>
+<instance part="C7" gate="G$1" x="904.24" y="662.94" smashed="yes">
+<attribute name="NAME" x="896.62" y="660.4" size="1.778" layer="95"/>
+<attribute name="VALUE" x="889" y="657.86" size="1.778" layer="96"/>
 </instance>
 <instance part="R303" gate="G$1" x="962.66" y="812.8" smashed="yes" rot="R90">

Commit message: Add files via upload
Parts:
- removed D20, D21: SMBJ7.0CA, diode:SUPPRESSOR-SMBJ
- added D9: CDSOT23-T24CAN, OSD3358-SM-RED Platform:CDSOT23-T24CAN
- added OIC14: MCP6001, adam - ics:MCP6001
- C11: value 220uF, 6.3V T491C227K006AT -> 220uF, 6.3V, T491C227K006AT
- C406: value 4.7uF, 16V -> 4.7uF, 16V, T491A475K016AT; device SparkFun-Capacitors:4.7UF-1206-16V-(+80/-20%) -> OSD3358-SM-RED Platform:CPOL-USA/3216-18R
- IC14: value MCP6001 -> MCP6002SMT; device adam - ics:MCP6001 -> adam - ics:MCP6002SMT
Connections:
- new net N$16: OIC14.-IN, OIC14.OUT
- net 1P8V_REF: no longer IC14.-IN, IC14.OUT
- net AGND: now also OIC14.V-; no longer IC14.V-
- net CAN_H: now also D9.2; no longer D20.C
- net CAN_L: now also D9.1; no longer D21.C
- net CGND: no longer D20.A, D21.A
- net GND: now also C7.2
- net ISO_GND: now also C406.-; no longer C406.2
- net ISO_VCC: now also C406.+; no longer C406.1
- net SYS_ADC_1P8V: now also OIC14.+IN; no longer IC14.+IN
- net SYS_VDD1_3P3V: now also C7.1, OIC14.V+; no longer IC14.V+
Other:
- moved on the sheet: C7

Commit message: Add files via upload
Parts:
- removed D9: CDSOT23-T24CAN, OSD3358-SM-RED Platform:CDSOT23-T24CAN
- removed OIC14: MCP6001, adam - ics:MCP6001
- removed R1, R2: 1K, OSD3358-SM-RED Platform:R-US_R0402
- removed X31: MC4, con-phoenix-381_l:MC4
- added D805: CDSOT23-T24CAN, OSD3358-SM-RED Platform:CDSOT23-T24CAN
- added R801, R802: 1K, OSD3358-SM-RED Platform:R-US_R0402
- added X8: MC4, con-phoenix-381_l:MC4
- renumbered C7 to C801, D2 to D801, D8 to D802
Connections:
- removed net 1P8V_REF: IC10A.V+, IC11A.V+, IC12A.V+, R212.2, R222.2, R232.2, R242.2, R252.2, R262.2
- removed net N$16: OIC14.-IN, OIC14.OUT
- new net 1P8V_REF_1: IC10A.V+, IC11A.V+, IC14A.-IN, IC14A.OUT, R212.2, R222.2, R232.2, R242.2
- new net 1P8V_REF_2: IC12A.V+, IC14B.-IN, IC14B.OUT, R252.2, R262.2
- net 24VDC_AUX: now also X8.4.SK
- net AGND: now also IC14A.V-, R181.2, R182.2, R183.2, R184.2, R185.2, R186.2; no longer OIC14.V-
- net CAN_H: now also D805.2, X8.2.SK; no longer D9.2
- net CAN_L: now also D805.1, X8.1.SK; no longer D9.1
- net CGND: no longer R181.2, R182.2, R183.2, R184.2, R185.2, R186.2
- net GND: now also D805.3, R801.2, R802.2, X8.3.SK; no longer R1.2, R2.2
- net N$5: now also R802.1; no longer R1.1
- net N$6: now also R801.1; no longer R2.1
- net SYS_ADC_1P8V: now also IC14A.+IN, IC14B.+IN; no longer OIC14.+IN
- net SYS_VDD1_3P3V: now also IC14A.V+; no longer OIC14.V+
Other:
- moved on the sheet: IC14A, IC14B

Commit message: Add files via upload
Parts:
- removed J17: (no value), OSD3358-SM-RED Platform:826646-2
- added J3, J4, J5, J6: (no value), OSD3358-SM-RED Platform:826646-2
Connections:
- net EHRPWM1A: now also J4.1
- net EHRPWM2A: now also J5.1
- net EHRPWM2B: now also J6.1
- net GND: now also J3.2, J4.2, J5.2, J6.2; no longer J17.1
- net N$111: now also J3.1; no longer J17.2
Changed lines of the file:
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@@
 <part name="R170" library="OSD3358-SM-RED Platform" deviceset="R-US_" device="R0402" value="1.5K, 1%"/>
 <part name="GND159" library="OSD3358-SM-RED Platform" deviceset="GND" device=""/>
-<part name="J17" library="OSD3358-SM-RED Platform" deviceset="826646-2" device=""/>
+<part name="J3" library="OSD3358-SM-RED Platform" deviceset="826646-2" device=""/>
 <part name="K1" library="relay" library_urn="urn:adsk.eagle:library:339" deviceset="JS-M1*" device="" package3d_urn="urn:adsk.eagle:package:24452/1" technology="-12V-5" value="JS1-24V-F"/>
 <part name="K2" library="relay" library_urn="urn:adsk.eagle:library:339" deviceset="JS-M1*" device="" package3d_urn="urn:adsk.eagle:package:24452/1" technology="-12V-5" value="JS1-24V-F"/>
@@
 <part name="SUPPLY28" library="OSD3358-SM-RED Platform" deviceset="AGND" device=""/>
 <part name="SUPPLY29" library="OSD3358-SM-RED Platform" deviceset="SYS_ADC_1P8V" device=""/>
+<part name="J4" library="OSD3358-SM-RED Platform" deviceset="826646-2" device=""/>
+<part name="J5" library="OSD3358-SM-RED Platform" deviceset="826646-2" device=""/>
+<part name="J6" library="OSD3358-SM-RED Platform" deviceset="826646-2" device=""/>
+<part name="GND24" library="OSD3358-SM-RED Platform" deviceset="GND" device=""/>
+<part name="GND30" library="OSD3358-SM-RED Platform" deviceset="GND" device=""/>
+<part name="GND31" library="OSD3358-SM-RED Platform" deviceset="GND" device=""/>
 </parts>
 <sheets>
@@
 <attribute name="VALUE" x="510.54" y="464.82" size="1.778" layer="96"/>
 </instance>
-<instance part="J17" gate="G$1" x="528.32" y="477.52" smashed="yes" rot="R180">
-<attribute name="NAME" x="528.32" y="469.9" size="1.778" layer="95" ratio="10" rot="R180"/>
-<attribute name="VALUE" x="528.32" y="480.06" size="1.778" layer="96" ratio="10" rot="R180"/>
+<instance part="J3" gate="G$1" x="525.78" y="469.9" smashed="yes" rot="MR0">
+<attribute name="NAME" x="525.78" y="477.52" size="1.778" layer="95" ratio="10" rot="MR0"/>
+<attribute name="VALUE" x="525.78" y="467.36" size="1.778" layer="96" ratio="10" rot="MR0"/>
 </instance>
 <instance part="K1" gate="1" x="962.66" y="1130.3" smashed="yes">
@@
 <attribute name="VALUE" x="762" y="1004.824" size="1.778" layer="96" align="center"/>
 </instance>
+<instance part="J4" gate="G$1" x="1094.74" y="802.64" smashed="yes" rot="MR0">
+<attribute name="NAME" x="1094.74" y="810.26" size="1.778" layer="95" ratio="10" rot="MR0"/>
+<attribute name="VALUE" x="1094.74" y="800.1" size="1.778" layer="96" ratio="10" rot="MR0"/>
+</instance>
+<instance part="J5" gate="G$1" x="1094.74" y="784.86" smashed="yes" rot="MR0">
+<attribute name="NAME" x="1094.74" y="792.48" size="1.778" layer="95" ratio="10" rot="MR0"/>
+<attribute name="VALUE" x="1094.74" y="782.32" size="1.778" layer="96" ratio="10" rot="MR0"/>
+</instance>
+<instance part="J6" gate="G$1" x="1094.74" y="767.08" smashed="yes" rot="MR0">
+<attribute name="NAME" x="1094.74" y="774.7" size="1.778" layer="95" ratio="10" rot="MR0"/>
+<attribute name="VALUE" x="1094.74" y="764.54" size="1.778" layer="96" ratio="10" rot="MR0"/>
+</instance>
+<instance part="GND24" gate="1" x="1082.04" y="800.1" smashed="yes">
+<attribute name="VALUE" x="1079.5" y="797.56" size="1.778" layer="96"/>
+</instance>
+<instance part="GND30" gate="1" x="1082.04" y="782.32" smashed="yes">
+<attribute name="VALUE" x="1079.5" y="779.78" size="1.778" layer="96"/>
+</instance>
+<instance part="GND31" gate="1" x="1082.04" y="764.54" smashed="yes">
+<attribute name="VALUE" x="1079.5" y="762" size="1.778" layer="96"/>
+</instance>
 </instances>
 <busses>
@@
 <pinref part="GND159" gate="1" pin="GND"/>
 <wire x1="513.08" y1="472.44" x2="513.08" y2="469.9" width="0.1524" layer="91"/>
-<pinref part="J17" gate="G$1" pin="1"/>
-<wire x1="518.16" y1="472.44" x2="513.08" y2="472.44" width="0.1524" layer="91"/>
+<pinref part="J3" gate="G$1" pin="2"/>
+<wire x1="515.62" y1="472.44" x2="513.08" y2="472.44" width="0.1524" layer="91"/>
 </segment>
 <segment>
@@
 <wire x1="325.12" y1="1016" x2="325.12" y2="1005.84" width="0.1524" layer="91"/>
 </segment>
+<segment>
+<pinref part="J4" gate="G$1" pin="2"/>
+<pinref part="GND24" gate="1" pin="GND"/>
+<wire x1="1084.58" y1="805.18" x2="1082.04" y2="805.18" width="0.1524" layer="91"/>
+<wire x1="1082.04" y1="805.18" x2="1082.04" y2="802.64" width="0.1524" layer="91"/>
+</segment>
+<segment>
+<pinref part="J5" gate="G$1" pin="2"/>
+<wire x1="1084.58" y1="787.4" x2="1082.04" y2="787.4" width="0.1524" layer="91"/>
+<pinref part="GND30" gate="1" pin="GND"/>
+<wire x1="1082.04" y1="787.4" x2="1082.04" y2="784.86" width="0.1524" layer="91"/>
+</segment>
+<segment>
+<pinref part="J6" gate="G$1" pin="2"/>
+<wire x1="1084.58" y1="769.62" x2="1082.04" y2="769.62" width="0.1524" layer="91"/>
+<pinref part="GND31" gate="1" pin="GND"/>
+<wire x1="1082.04" y1="769.62" x2="1082.04" y2="767.08" width="0.1524" layer="91"/>
+</segment>
 </net>
 <net name="PWR_BUT" class="0">
@@
 <label x="1018.54" y="71.12" size="1.778" layer="95"/>
 </segment>
+<segment>
+<pinref part="J6" gate="G$1" pin="1"/>
+<wire x1="1084.58" y1="772.16" x2="1064.26" y2="772.16" width="0.1524" layer="91"/>
+<label x="1064.26" y="772.16" size="1.778" layer="95"/>
+</segment>
 </net>
 <net name="EHRPWM2A" class="0">
@@
 <label x="1018.54" y="73.66" size="1.778" layer="95"/>
 </segment>
+<segment>
+<pinref part="J5" gate="G$1" pin="1"/>
+<wire x1="1084.58" y1="789.94" x2="1064.26" y2="789.94" width="0.1524" layer="91"/>
+<label x="1064.26" y="789.94" size="1.778" layer="95"/>
+</segment>
 </net>
 <net name="EHRPWM1B" class="0">
@@
 <label x="1018.54" y="124.46" size="1.778" layer="95"/>
 </segment>
+<segment>
+<pinref part="J4" gate="G$1" pin="1"/>
+<wire x1="1084.58" y1="807.72" x2="1064.26" y2="807.72" width="0.1524" layer="91"/>
+<label x="1064.26" y="807.72" size="1.778" layer="95"/>
+</segment>
 </net>
 <net name="MMC0_DAT3" class="0">
@@
 <wire x1="513.08" y1="482.6" x2="480.06" y2="482.6" width="0.1524" layer="91"/>
 <pinref part="R69" gate="G$1" pin="2"/>
-<pinref part="J17" gate="G$1" pin="2"/>
-<wire x1="518.16" y1="474.98" x2="513.08" y2="474.98" width="0.1524" layer="91"/>
+<pinref part="J3" gate="G$1" pin="1"/>
+<wire x1="515.62" y1="474.98" x2="513.08" y2="474.98" width="0.1524" layer="91"/>
 </segment>
 </net>

Commit message: Add files via upload
Parts:
- added TP17, TP18, TP19, TP20: TESTPAD/W_HOLE_1X1, OSD3358-SM-RED Platform:TESTPAD/W_HOLE_1X1
Connections:
- removed net OSC1_GND: RTC1.GND, U1B.OSC1_GND
- net GND: now also RTC1.GND, U1B.OSC1_GND
- net I2C0_SCL: now also TP18.TP
- net I2C0_SDA: now also TP17.TP
- net I2C1_SCL: now also TP20.TP
- net I2C1_SDA: now also TP19.TP
Other:
- note added: "AT97SC3205T I2C Address: 0x29"
- note added: "DS3231 I2C Address: 0x68"
Changed lines of the file:
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@@
 <part name="GND30" library="OSD3358-SM-RED Platform" deviceset="GND" device=""/>
 <part name="GND31" library="OSD3358-SM-RED Platform" deviceset="GND" device=""/>
+<part name="TP17" library="OSD3358-SM-RED Platform" deviceset="TESTPAD/W_HOLE_1X1" device=""/>
+<part name="TP18" library="OSD3358-SM-RED Platform" deviceset="TESTPAD/W_HOLE_1X1" device=""/>
+<part name="TP19" library="OSD3358-SM-RED Platform" deviceset="TESTPAD/W_HOLE_1X1" device=""/>
+<part name="TP20" library="OSD3358-SM-RED Platform" deviceset="TESTPAD/W_HOLE_1X1" device=""/>
 </parts>
 <sheets>
@@
 <text x="96.52" y="1026.16" size="2.54" layer="150" align="center-left">VDC
 </text>
+<text x="10.16" y="104.14" size="2.54" layer="150">AT97SC3205T I2C Address:  0x29</text>
+<text x="797.56" y="127" size="2.54" layer="150">DS3231 I2C Address:  0x68</text>
 </plain>
 <instances>
@@
 </instance>
 <instance part="R11" gate="G$1" x="53.34" y="83.82" smashed="yes">
-<attribute name="NAME" x="48.26" y="86.36" size="1.778" layer="95"/>
-<attribute name="VALUE" x="55.88" y="86.36" size="1.778" layer="96"/>
+<attribute name="NAME" x="45.72" y="81.28" size="1.778" layer="95"/>
+<attribute name="VALUE" x="55.88" y="81.28" size="1.778" layer="96"/>
 </instance>
 <instance part="R5" gate="G$1" x="121.92" y="66.04" smashed="yes" rot="R180">
@@
 <attribute name="VALUE" x="1079.5" y="762" size="1.778" layer="96"/>
 </instance>
+<instance part="TP17" gate="G$1" x="60.96" y="86.36" smashed="yes" rot="R180">
+<attribute name="NAME" x="53.34" y="88.9" size="1.778" layer="95"/>
+</instance>
+<instance part="TP18" gate="G$1" x="60.96" y="96.52" smashed="yes" rot="R180">
+<attribute name="NAME" x="53.34" y="99.06" size="1.778" layer="95"/>
+</instance>
+<instance part="TP19" gate="G$1" x="858.52" y="129.54" smashed="yes" rot="R180">
+<attribute name="NAME" x="845.82" y="129.54" size="1.778" layer="95"/>
+</instance>
+<instance part="TP20" gate="G$1" x="858.52" y="127" smashed="yes" rot="R180">
+<attribute name="NAME" x="845.82" y="127" size="1.778" layer="95"/>
+</instance>
 </instances>
 <busses>
@@
 <wire x1="1082.04" y1="769.62" x2="1082.04" y2="767.08" width="0.1524" layer="91"/>
 </segment>
+<segment>
+<pinref part="RTC1" gate="G$1" pin="GND"/>
+<pinref part="GND157" gate="1" pin="GND"/>
+<wire x1="919.48" y1="477.52" x2="922.02" y2="477.52" width="0.1524" layer="91"/>
+<wire x1="922.02" y1="477.52" x2="922.02" y2="469.9" width="0.1524" layer="91"/>
+<wire x1="922.02" y1="469.9" x2="868.68" y2="469.9" width="0.1524" layer="91"/>
+<junction x="922.02" y="469.9"/>
+<label x="868.68" y="469.9" size="1.778" layer="95"/>
+</segment>
+<segment>
+<pinref part="U1" gate="B" pin="OSC1_GND"/>
+<wire x1="553.72" y1="167.64" x2="530.86" y2="167.64" width="0.1524" layer="91"/>
+<label x="530.86" y="167.64" size="1.778" layer="95"/>
+</segment>
 </net>
 <net name="PWR_BUT" class="0">
@@
 <wire x1="78.74" y1="99.06" x2="78.74" y2="96.52" width="0.1524" layer="91"/>
 <junction x="78.74" y="96.52"/>
+<pinref part="TP18" gate="G$1" pin="TP"/>
 </segment>
 </net>
@@
 <wire x1="88.9" y1="99.06" x2="88.9" y2="86.36" width="0.1524" layer="91"/>
 <junction x="88.9" y="86.36"/>
+<pinref part="TP17" gate="G$1" pin="TP"/>
 </segment>
 </net>
@@
 </segment>
 </net>
-<net name="OSC1_GND" class="0">
-<segment>
-<pinref part="RTC1" gate="G$1" pin="GND"/>
-<pinref part="GND157" gate="1" pin="GND"/>
-<wire x1="919.48" y1="477.52" x2="922.02" y2="477.52" width="0.1524" layer="91"/>
-<wire x1="922.02" y1="477.52" x2="922.02" y2="469.9" width="0.1524" layer="91"/>
-<wire x1="922.02" y1="469.9" x2="868.68" y2="469.9" width="0.1524" layer="91"/>
-<junction x="922.02" y="469.9"/>
-<label x="868.68" y="469.9" size="1.778" layer="95"/>
-</segment>
-<segment>
-<pinref part="U1" gate="B" pin="OSC1_GND"/>
-<wire x1="553.72" y1="167.64" x2="530.86" y2="167.64" width="0.1524" layer="91"/>
-<label x="530.86" y="167.64" size="1.778" layer="95"/>
-</segment>
-</net>
 <net name="JTAG_EMU1" class="0">
 <segment>
@@
 <wire x1="914.4" y1="129.54" x2="861.06" y2="129.54" width="0.1524" layer="91"/>
 <label x="861.06" y="129.54" size="1.778" layer="95"/>
+<pinref part="TP19" gate="G$1" pin="TP"/>
 </segment>
 <segment>
@@
 <wire x1="914.4" y1="127" x2="861.06" y2="127" width="0.1524" layer="91"/>
 <label x="861.06" y="127" size="1.778" layer="95"/>
+<pinref part="TP20" gate="G$1" pin="TP"/>
 </segment>
 <segment>
