File: Version_2.2/Open-Source_Control_V2_R2.brd (EAGLE design)
At the start: 121.9 x 129.5 mm, 344 parts, among them IC10 MCP6002SMT, IC11 MCP6002SMT, IC12 MCP6002SMT, IC14 MCP6002SMT, IC2 ULN2003AD, IC4 74HC165D, IC5 74HC165D, J24 6p-2.54, K1 JS1-24V-F, K2 JS1-24V-F, K3 JS1-24V-F, K4 JS1-24V-F, K5 JS1-24V-F, Q1 MMBT2907, T4 DA2304-AL, U1 OSD3358-512M-ICB, U16 AT97SC3205T-G3M4400B, U2 TPD4S012_DRY_6_P1_M, U27 LAN8710, U28 TCAN1051HV, U29 MAX3483EESA+T, U4 APX811-31UGSOT, U40 ISO3086TDW, U5 TLVH431, U6 SN74LVC2G241_DCU_8, X1 10118194-0001LF, X10 MC4, X11 MC4, X12 MC4, X2 J0011D01BNL, X21 MC10, X24 MSTBA2, X3 MC4, X4 CTI-JTAG, X41 MSTBA3, X5 DM3CS-SF, X6 6p-2.54, X7 TH-2X10, X8 MC4, Y7 7A-25.000MAAE-T

Commit message: Add files via upload
Connections:
- removed net I2C1_SCL: R169.1, RTC1.8, TP20.P$1, U1.V5
- removed net I2C1_SDA: R170.1, RTC1.7, TP19.P$1, U1.V6
- new net I2C2_SCL: R169.1, RTC1.8, TP20.P$1, U1.Y8
- new net I2C2_SDA: R170.1, RTC1.7, TP19.P$1, U1.W8
- net TPM_GPIO1: now also U1.V6; no longer U1.W8
- net TPM_GPIO2: now also U1.V5; no longer U1.Y8
Routing:
- net I2C1_SCL: track 38.3 -> 0.00 mm, vias 2 -> 0
- net I2C2_SCL: track 0.00 -> 37.1 mm, vias 0 -> 2
- net I2C1_SDA: track 35.0 -> 0.00 mm, vias 2 -> 0
- net I2C2_SDA: track 0.00 -> 31.6 mm, vias 0 -> 2
- net GPIO0_7: track 49.7 -> 51.3 mm
- net TPM_GPIO1: track 39.3 -> 37.7 mm
- net TPM_GPIO2: track 38.9 -> 39.5 mm
- net I2C0_SCL: track 35.2 -> 35.0 mm, vias 2 -> 1

Commit message: Add files via upload
Routing:
- net N$120: track 88.1 -> 87.3 mm
- net N$119: track 92.4 -> 91.6 mm
- net N$124: track 108.9 -> 108.1 mm
- net N$129: track 124.9 -> 124.1 mm
- net N$128: track 104.7 -> 103.9 mm
- net CAN1_RXD: track 226.5 -> 227.1 mm
Changed lines of the file:
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@@
 <wire x1="73.7362" y1="4.318" x2="78.994" y2="4.318" width="0.1524" layer="1"/>
 <wire x1="78.994" y1="4.318" x2="83.312" y2="8.636" width="0.1524" layer="1"/>
-<wire x1="83.312" y1="8.636" x2="88.1634" y2="8.636" width="0.1524" layer="1"/>
-<wire x1="88.1634" y1="8.636" x2="89.4334" y2="7.366" width="0.1524" layer="1"/>
-<wire x1="89.4334" y1="7.366" x2="102.489" y2="7.366" width="0.1524" layer="1"/>
-<wire x1="102.489" y1="7.366" x2="103.124" y2="6.731" width="0.1524" layer="1"/>
-<wire x1="103.124" y1="6.731" x2="103.124" y2="5.8293" width="0.1524" layer="1"/>
+<wire x1="83.312" y1="8.636" x2="101.854" y2="8.636" width="0.1524" layer="1"/>
+<wire x1="101.854" y1="8.636" x2="103.124" y2="7.366" width="0.1524" layer="1"/>
+<wire x1="103.124" y1="7.366" x2="103.124" y2="5.8293" width="0.1524" layer="1"/>
 </signal>
 <signal name="CAN1_RXD">
@@
 <wire x1="72.7202" y1="3.81" x2="79.248" y2="3.81" width="0.1524" layer="1"/>
 <wire x1="79.248" y1="3.81" x2="83.566" y2="8.128" width="0.1524" layer="1"/>
-<wire x1="83.566" y1="8.128" x2="87.884" y2="8.128" width="0.1524" layer="1"/>
-<wire x1="87.884" y1="8.128" x2="89.154" y2="6.858" width="0.1524" layer="1"/>
-<wire x1="89.154" y1="6.858" x2="100.0633" y2="6.858" width="0.1524" layer="1"/>
-<wire x1="100.0633" y1="6.858" x2="101.092" y2="5.8293" width="0.1524" layer="1"/>
+<wire x1="83.566" y1="8.128" x2="99.822" y2="8.128" width="0.1524" layer="1"/>
+<wire x1="99.822" y1="8.128" x2="101.092" y2="6.858" width="0.1524" layer="1"/>
+<wire x1="101.092" y1="6.858" x2="101.092" y2="5.8293" width="0.1524" layer="1"/>
 </signal>
 <signal name="USB0_P">
@@
 <wire x1="95.7834" y1="74.295" x2="99.441" y2="74.295" width="0.3048" layer="1"/>
 <wire x1="99.441" y1="74.295" x2="100.711" y2="73.025" width="0.3048" layer="1"/>
-<wire x1="100.711" y1="73.025" x2="100.711" y2="59.4868" width="0.3048" layer="1"/>
-<wire x1="100.711" y1="59.4868" x2="99.441" y2="58.2168" width="0.3048" layer="1"/>
-<wire x1="99.441" y1="58.2168" x2="78.3336" y2="58.2168" width="0.3048" layer="1"/>
+<wire x1="100.711" y1="73.025" x2="100.711" y2="60.8584" width="0.3048" layer="1"/>
+<wire x1="100.711" y1="60.8584" x2="98.0694" y2="58.2168" width="0.3048" layer="1"/>
+<wire x1="98.0694" y1="58.2168" x2="78.3336" y2="58.2168" width="0.3048" layer="1"/>
 <wire x1="78.3336" y1="58.2168" x2="77.0636" y2="56.9468" width="0.3048" layer="1"/>
 <wire x1="77.0636" y1="56.9468" x2="77.0636" y2="47.498" width="0.3048" layer="1"/>
@@
 <wire x1="95.7834" y1="73.025" x2="98.9076" y2="73.025" width="0.3048" layer="1"/>
 <wire x1="98.9076" y1="73.025" x2="100.1776" y2="71.755" width="0.3048" layer="1"/>
-<wire x1="100.1776" y1="71.755" x2="100.1776" y2="60.0202" width="0.3048" layer="1"/>
-<wire x1="100.1776" y1="60.0202" x2="98.9076" y2="58.7502" width="0.3048" layer="1"/>
-<wire x1="98.9076" y1="58.7502" x2="77.8002" y2="58.7502" width="0.3048" layer="1"/>
-<wire x1="77.8002" y1="58.7502" x2="76.5302" y2="57.4802" width="0.3048" layer="1"/>
+<wire x1="100.1776" y1="71.755" x2="100.1776" y2="61.0616" width="0.3048" layer="1"/>
+<wire x1="100.1776" y1="61.0616" x2="97.8662" y2="58.7502" width="0.3048" layer="1"/>
+<wire x1="97.8662" y1="58.7502" x2="78.1304" y2="58.7502" width="0.3048" layer="1"/>
+<wire x1="78.1304" y1="58.7502" x2="76.5302" y2="57.15" width="0.3048" layer="1"/>
 <wire x1="79.09" y1="44.8" x2="77.8002" y2="44.8" width="0.3048" layer="1"/>
 <wire x1="77.8002" y1="44.8" x2="76.5302" y2="46.07" width="0.3048" layer="1"/>
-<wire x1="76.5302" y1="46.07" x2="76.5302" y2="57.4802" width="0.3048" layer="1"/>
+<wire x1="76.5302" y1="46.07" x2="76.5302" y2="57.15" width="0.3048" layer="1"/>
 <wire x1="79.09" y1="44.8" x2="80.4982" y2="44.8" width="0.3048" layer="1"/>
 <wire x1="107.2896" y1="47.4472" x2="108.331" y2="47.4472" width="0.3048" layer="1"/>
@@
 <wire x1="95.7834" y1="71.755" x2="98.3742" y2="71.755" width="0.3048" layer="1"/>
 <wire x1="98.3742" y1="71.755" x2="99.6442" y2="70.485" width="0.3048" layer="1"/>
-<wire x1="99.6442" y1="70.485" x2="99.6442" y2="60.5536" width="0.3048" layer="1"/>
-<wire x1="99.6442" y1="60.5536" x2="98.3742" y2="59.2836" width="0.3048" layer="1"/>
-<wire x1="98.3742" y1="59.2836" x2="77.2668" y2="59.2836" width="0.3048" layer="1"/>
-<wire x1="77.2668" y1="59.2836" x2="75.9968" y2="58.0136" width="0.3048" layer="1"/>
-<wire x1="75.9968" y1="58.0136" x2="75.9968" y2="30.988" width="0.3048" layer="1"/>
+<wire x1="99.6442" y1="70.485" x2="99.6442" y2="61.2394" width="0.3048" layer="1"/>
+<wire x1="99.6442" y1="61.2394" x2="97.6884" y2="59.2836" width="0.3048" layer="1"/>
+<wire x1="97.6884" y1="59.2836" x2="77.9272" y2="59.2836" width="0.3048" layer="1"/>
+<wire x1="77.9272" y1="59.2836" x2="75.9968" y2="57.3532" width="0.3048" layer="1"/>
+<wire x1="75.9968" y1="57.3532" x2="75.9968" y2="30.988" width="0.3048" layer="1"/>
 <wire x1="75.9968" y1="30.988" x2="77.2668" y2="29.718" width="0.3048" layer="1"/>
 <wire x1="77.2668" y1="29.718" x2="100.522" y2="29.718" width="0.3048" layer="1"/>
@@
 <wire x1="95.7834" y1="70.485" x2="97.8408" y2="70.485" width="0.3048" layer="1"/>
 <wire x1="97.8408" y1="70.485" x2="99.1108" y2="69.215" width="0.3048" layer="1"/>
-<wire x1="99.1108" y1="69.215" x2="99.1108" y2="61.087" width="0.3048" layer="1"/>
-<wire x1="99.1108" y1="61.087" x2="97.8408" y2="59.817" width="0.3048" layer="1"/>
-<wire x1="97.8408" y1="59.817" x2="76.7334" y2="59.817" width="0.3048" layer="1"/>
-<wire x1="76.7334" y1="59.817" x2="75.4634" y2="58.547" width="0.3048" layer="1"/>
-<wire x1="75.4634" y1="58.547" x2="75.4634" y2="29.56" width="0.3048" layer="1"/>
+<wire x1="99.1108" y1="69.215" x2="99.1108" y2="61.4172" width="0.3048" layer="1"/>
+<wire x1="99.1108" y1="61.4172" x2="97.5106" y2="59.817" width="0.3048" layer="1"/>
+<wire x1="97.5106" y1="59.817" x2="77.724" y2="59.817" width="0.3048" layer="1"/>
+<wire x1="77.724" y1="59.817" x2="75.4634" y2="57.5564" width="0.3048" layer="1"/>
+<wire x1="75.4634" y1="57.5564" x2="75.4634" y2="29.56" width="0.3048" layer="1"/>
 <wire x1="75.4634" y1="29.56" x2="76.7334" y2="28.29" width="0.3048" layer="1"/>
 <wire x1="76.7334" y1="28.29" x2="79.09" y2="28.29" width="0.3048" layer="1"/>
@@
 <wire x1="98.5774" y1="67.945" x2="98.5774" y2="61.6204" width="0.3048" layer="1"/>
 <wire x1="98.5774" y1="61.6204" x2="97.3074" y2="60.3504" width="0.3048" layer="1"/>
-<wire x1="97.3074" y1="60.3504" x2="76.2" y2="60.3504" width="0.3048" layer="1"/>
-<wire x1="76.2" y1="60.3504" x2="74.93" y2="59.0804" width="0.3048" layer="1"/>
-<wire x1="74.93" y1="59.0804" x2="74.93" y2="23.622" width="0.3048" layer="1"/>
+<wire x1="97.3074" y1="60.3504" x2="77.5208" y2="60.3504" width="0.3048" layer="1"/>
+<wire x1="77.5208" y1="60.3504" x2="74.93" y2="57.7596" width="0.3048" layer="1"/>
+<wire x1="74.93" y1="57.7596" x2="74.93" y2="23.622" width="0.3048" layer="1"/>
 <wire x1="74.93" y1="23.622" x2="76.2" y2="22.352" width="0.3048" layer="1"/>
 <wire x1="76.2" y1="22.352" x2="100.68" y2="22.352" width="0.3048" layer="1"/>
