File: Version_2.2/Open-Source_Control_V2_R2.sch (EAGLE design)
At the start: 342 parts, among them IC10 MCP6002SMT, IC11 MCP6002SMT, IC12 MCP6002SMT, IC14 MCP6002SMT, IC2 ULN2003AD, IC4 74HC165D, IC5 74HC165D, J24 6p-2.54, K1 JS1-24V-F, K2 JS1-24V-F, K3 JS1-24V-F, K4 JS1-24V-F, K5 JS1-24V-F, Q1 MMBT2907, T4 DA2304-AL, U1 OSD3358-512M-ICB, U16 AT97SC3205T-G3M4400B, U2 TPD4S012_DRY_6_P1_M, U27 LAN8710, U28 TCAN1051HV, U29 MAX3483EESA+T, U4 APX811-31UGSOT, U40 ISO3086TDW, U5 TLVH431, U6 SN74LVC2G241_DCU_8, X1 10118194-0001LF, X10 MC4, X11 MC4, X12 MC4, X2 J0011D01BNL, X21 MC10, X24 MSTBA2, X3 MC4, X4 CTI-JTAG, X41 MSTBA3, X5 DM3CS-SF, X6 6p-2.54, X7 TH-2X10, X8 MC4, Y7 7A-25.000MAAE-T

Commit message: Add files via upload
Connections:
- removed net GPIO0_4: U1C.SPI0_D1, U29.!RE, U29.DE
- new net GPIO0_7: U1C.ECAP0_IN_PWM0_OUT, U29.!RE, U29.DE
- new net PR1_PRU0_PRU_R30_6: U1C.MCASP0_AXR1
- new net PR1_PRU0_PRU_R30_7: U1C.MCASP0_AHCLKX
- new net PR1_UART0_RXD: U1C.SPI0_D1
- new net PR1_UART0_TXD: U1C.SPI0_CS0
Changed lines of the file:
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@@
-</segment>
-</net>
-<net name="GPIO0_4" class="0">
-<segment>
-<pinref part="U1" gate="C" pin="SPI0_D1"/>
-<wire x1="914.4" y1="99.06" x2="861.06" y2="99.06" width="0.1524" layer="91"/>
-<label x="861.06" y="99.06" size="1.778" layer="95"/>
-</segment>
-<segment>
-<pinref part="U29" gate="A" pin="DE"/>
-<wire x1="878.84" y1="797.56" x2="873.76" y2="797.56" width="0.1524" layer="91"/>
-<pinref part="U29" gate="A" pin="!RE"/>
-<wire x1="873.76" y1="797.56" x2="810.26" y2="797.56" width="0.1524" layer="91"/>
-<wire x1="878.84" y1="800.1" x2="873.76" y2="800.1" width="0.1524" layer="91"/>
-<wire x1="873.76" y1="800.1" x2="873.76" y2="797.56" width="0.1524" layer="91"/>
-<junction x="873.76" y="797.56"/>
-<label x="810.26" y="797.56" size="1.778" layer="95"/>
 </segment>
 </net>
@@
 </segment>
 </net>
+<net name="PR1_UART0_TXD" class="0">
+<segment>
+<pinref part="U1" gate="C" pin="SPI0_CS0"/>
+<wire x1="914.4" y1="96.52" x2="861.06" y2="96.52" width="0.1524" layer="91"/>
+<label x="861.06" y="96.52" size="1.778" layer="95"/>
+</segment>
+</net>
+<net name="PR1_PRU0_PRU_R30_7" class="0">
+<segment>
+<pinref part="U1" gate="C" pin="MCASP0_AHCLKX"/>
+<wire x1="914.4" y1="48.26" x2="861.06" y2="48.26" width="0.1524" layer="91"/>
+<label x="861.06" y="48.26" size="1.778" layer="95"/>
+</segment>
+</net>
+<net name="PR1_PRU0_PRU_R30_6" class="0">
+<segment>
+<pinref part="U1" gate="C" pin="MCASP0_AXR1"/>
+<wire x1="914.4" y1="50.8" x2="861.06" y2="50.8" width="0.1524" layer="91"/>
+<label x="861.06" y="50.8" size="1.778" layer="95"/>
+</segment>
+</net>
+<net name="PR1_UART0_RXD" class="0">
+<segment>
+<pinref part="U1" gate="C" pin="SPI0_D1"/>
+<wire x1="914.4" y1="99.06" x2="861.06" y2="99.06" width="0.1524" layer="91"/>
+<label x="861.06" y="99.06" size="1.778" layer="95"/>
+</segment>
+</net>
+<net name="GPIO0_7" class="0">
+<segment>
+<pinref part="U1" gate="C" pin="ECAP0_IN_PWM0_OUT"/>
+<wire x1="914.4" y1="33.02" x2="861.06" y2="33.02" width="0.1524" layer="91"/>
+<label x="861.06" y="33.02" size="1.778" layer="95"/>
+</segment>
+<segment>
+<pinref part="U29" gate="A" pin="DE"/>
+<wire x1="878.84" y1="797.56" x2="873.76" y2="797.56" width="0.1524" layer="91"/>
+<pinref part="U29" gate="A" pin="!RE"/>
+<wire x1="873.76" y1="797.56" x2="810.26" y2="797.56" width="0.1524" layer="91"/>
+<wire x1="878.84" y1="800.1" x2="873.76" y2="800.1" width="0.1524" layer="91"/>
+<wire x1="873.76" y1="800.1" x2="873.76" y2="797.56" width="0.1524" layer="91"/>
+<junction x="873.76" y="797.56"/>
+<label x="810.26" y="797.56" size="1.778" layer="95"/>
+</segment>
+</net>
