File: Version_2.2/Open-Source_Control_V2_R2.sch (EAGLE design)
At the start: 345 parts, among them IC10 MCP6002SMT, IC11 MCP6002SMT, IC12 MCP6002SMT, IC14 MCP6002SMT, IC2 ULN2003AD, IC4 74HC165D, IC5 74HC165D, J24 6p-2.54, K1 JS1-24V-F, K2 JS1-24V-F, K3 JS1-24V-F, K4 JS1-24V-F, K5 JS1-24V-F, Q1 MMBT2907, T4 DA2304-AL, U1 OSD3358-512M-ICB, U16 AT97SC3205T-G3M4400B, U2 TPD4S012_DRY_6_P1_M, U27 LAN8710, U28 TCAN1051HV, U29 MAX3483EESA+T, U4 APX811-31UGSOT, U40 ISO3086TDW, U5 TLVH431, U6 SN74LVC2G241_DCU_8, X1 10118194-0001LF, X10 MC4, X11 MC4, X12 MC4, X2 J0011D01BNL, X21 MC10, X24 MSTBA2, X3 MC4, X4 CTI-JTAG, X41 MSTBA3, X5 DM3CS-SF, X6 6p-2.54, X7 TH-2X10, X8 MC4, Y7 7A-25.000MAAE-T

Commit message: Add files via upload
Parts:
- D19, D31, D32, D33, D34, D35: value LTST-C191KRKT -> LTST-C191KGKT; device OSD3358-SM-RED Platform:LTST-C191KRKTLED_EIA-STD -> OSD3358-SM-RED Platform:LTST-C191KGKTLED_EIA-STD
- D301: value LTST-C191KGKT -> LTST-C191KRKT
- D302: value LTST-C191KFKT -> LTST-C191KGKT; device OSD3358-SM-RED Platform:LTST-C191KFKTLED_EIA-STD -> OSD3358-SM-RED Platform:LTST-C191KRKTLED_EIA-STD
- D401: value LTST-C191KGKT -> LTST-C191KRKT; device OSD3358-SM-RED Platform:LTST-C191KGKTLED_EIA-STD -> OSD3358-SM-RED Platform:LTST-C191KRKTLED_EIA-STD
- D402: value LTST-C191KFKT -> LTST-C191KGKT; device OSD3358-SM-RED Platform:LTST-C191KFKTLED_EIA-STD -> OSD3358-SM-RED Platform:LTST-C191KGKTLED_EIA-STD
- D801: value LTST-C191KFKT -> LTST-C191KRKT; device OSD3358-SM-RED Platform:LTST-C191KFKTLED_EIA-STD -> OSD3358-SM-RED Platform:LTST-C191KRKTLED_EIA-STD
Changed lines of the file:
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@@
 <part name="GND116" library="OSD3358-SM-RED Platform" deviceset="GND" device=""/>
 <part name="SUPPLY112" library="OSD3358-SM-RED Platform" deviceset="SYS_VDD1_3P3V" device=""/>
-<part name="D402" library="OSD3358-SM-RED Platform" deviceset="LTST-C191KFKT" device="LED_EIA-STD" value="LTST-C191KFKT"/>
-<part name="D401" library="OSD3358-SM-RED Platform" deviceset="LTST-C191KGKT" device="LED_EIA-STD" value="LTST-C191KGKT"/>
+<part name="D402" library="OSD3358-SM-RED Platform" deviceset="LTST-C191KGKT" device="LED_EIA-STD" value="LTST-C191KGKT"/>
+<part name="D401" library="OSD3358-SM-RED Platform" deviceset="LTST-C191KRKT" device="LED_EIA-STD" value="LTST-C191KRKT"/>
 <part name="R401" library="OSD3358-SM-RED Platform" deviceset="R-US_" device="R0402" value="1K"/>
 <part name="R402" library="OSD3358-SM-RED Platform" deviceset="R-US_" device="R0402" value="1K"/>
@@
 <part name="GND126" library="OSD3358-SM-RED Platform" deviceset="GND" device=""/>
 <part name="R168" library="OSD3358-SM-RED Platform" deviceset="R-US_" device="R0402" value="10K"/>
-<part name="D19" library="OSD3358-SM-RED Platform" deviceset="LTST-C191KRKT" device="LED_EIA-STD" value="LTST-C191KRKT"/>
+<part name="D19" library="OSD3358-SM-RED Platform" deviceset="LTST-C191KGKT" device="LED_EIA-STD" value="LTST-C191KGKT"/>
 <part name="GND128" library="OSD3358-SM-RED Platform" deviceset="GND" device=""/>
 <part name="U$7" library="OSD3358-SM-RED Platform" deviceset="24VDC_AUX" device=""/>
@@
 <part name="X21" library="con-phoenix-381_l" deviceset="MC10" device=""/>
 <part name="IC2" library="uln-udn" library_urn="urn:adsk.eagle:library:407" deviceset="ULN2003A" device="D" package3d_urn="urn:adsk.eagle:package:30247/1"/>
-<part name="D31" library="OSD3358-SM-RED Platform" deviceset="LTST-C191KRKT" device="LED_EIA-STD" value="LTST-C191KRKT"/>
-<part name="D32" library="OSD3358-SM-RED Platform" deviceset="LTST-C191KRKT" device="LED_EIA-STD" value="LTST-C191KRKT"/>
-<part name="D33" library="OSD3358-SM-RED Platform" deviceset="LTST-C191KRKT" device="LED_EIA-STD" value="LTST-C191KRKT"/>
-<part name="D34" library="OSD3358-SM-RED Platform" deviceset="LTST-C191KRKT" device="LED_EIA-STD" value="LTST-C191KRKT"/>
-<part name="D35" library="OSD3358-SM-RED Platform" deviceset="LTST-C191KRKT" device="LED_EIA-STD" value="LTST-C191KRKT"/>
+<part name="D31" library="OSD3358-SM-RED Platform" deviceset="LTST-C191KGKT" device="LED_EIA-STD" value="LTST-C191KGKT"/>
+<part name="D32" library="OSD3358-SM-RED Platform" deviceset="LTST-C191KGKT" device="LED_EIA-STD" value="LTST-C191KGKT"/>
+<part name="D33" library="OSD3358-SM-RED Platform" deviceset="LTST-C191KGKT" device="LED_EIA-STD" value="LTST-C191KGKT"/>
+<part name="D34" library="OSD3358-SM-RED Platform" deviceset="LTST-C191KGKT" device="LED_EIA-STD" value="LTST-C191KGKT"/>
+<part name="D35" library="OSD3358-SM-RED Platform" deviceset="LTST-C191KGKT" device="LED_EIA-STD" value="LTST-C191KGKT"/>
 <part name="R173" library="OSD3358-SM-RED Platform" deviceset="R-US_" device="R0402" value="10K"/>
 <part name="R174" library="OSD3358-SM-RED Platform" deviceset="R-US_" device="R0402" value="10K"/>
@@
 <part name="GND36" library="OSD3358-SM-RED Platform" deviceset="GND" device=""/>
 <part name="X3" library="con-phoenix-381_l" deviceset="MC4" device=""/>
-<part name="D801" library="OSD3358-SM-RED Platform" deviceset="LTST-C191KFKT" device="LED_EIA-STD" value="LTST-C191KFKT"/>
+<part name="D801" library="OSD3358-SM-RED Platform" deviceset="LTST-C191KRKT" device="LED_EIA-STD" value="LTST-C191KRKT"/>
 <part name="D802" library="OSD3358-SM-RED Platform" deviceset="LTST-C191KGKT" device="LED_EIA-STD" value="LTST-C191KGKT"/>
 <part name="R802" library="OSD3358-SM-RED Platform" deviceset="R-US_" device="R0402" value="1K"/>
@@
 <part name="GND8" library="OSD3358-SM-RED Platform" deviceset="GND" device=""/>
 <part name="GND9" library="OSD3358-SM-RED Platform" deviceset="GND" device=""/>
-<part name="D301" library="OSD3358-SM-RED Platform" deviceset="LTST-C191KGKT" device="LED_EIA-STD" value="LTST-C191KGKT"/>
-<part name="D302" library="OSD3358-SM-RED Platform" deviceset="LTST-C191KFKT" device="LED_EIA-STD" value="LTST-C191KFKT"/>
+<part name="D301" library="OSD3358-SM-RED Platform" deviceset="LTST-C191KGKT" device="LED_EIA-STD" value="LTST-C191KRKT"/>
+<part name="D302" library="OSD3358-SM-RED Platform" deviceset="LTST-C191KRKT" device="LED_EIA-STD" value="LTST-C191KGKT"/>
 <part name="GND10" library="OSD3358-SM-RED Platform" deviceset="GND" device=""/>
 <part name="GND14" library="OSD3358-SM-RED Platform" deviceset="GND" device=""/>

Commit message: Add files via upload
Parts:
- added R215, R225, R235, R245, R255, R265: 100K, OSD3358-SM-RED Platform:R-US_R0805
Connections:
- net AGND: now also R215.2, R225.2, R235.2, R245.2, R255.2, R265.2; no longer IC14A.V-
- net AIN1: now also R215.1
- net AIN2: now also R225.1
- net AIN3: now also R235.1
- net AIN4: now also R245.1
- net AIN5: now also R255.1
- net AIN6: now also R265.1
- net GND: now also IC14A.V-

Commit message: Add files via upload
Parts:
- added J7: (no value), OSD3358-SM-RED Platform:826646-2
Connections:
- net AGND: now also J7.1
- net GND: now also J7.2
Other:
- note added: "Jumper AGND to GND This is optional. Already connected inside SiP"
Changed lines of the file:
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@@
 <part name="R255" library="OSD3358-SM-RED Platform" deviceset="R-US_" device="R0805" value="100K"/>
 <part name="R265" library="OSD3358-SM-RED Platform" deviceset="R-US_" device="R0805" value="100K"/>
+<part name="J7" library="OSD3358-SM-RED Platform" deviceset="826646-2" device=""/>
+<part name="SUPPLY34" library="OSD3358-SM-RED Platform" deviceset="AGND" device=""/>
+<part name="GND34" library="OSD3358-SM-RED Platform" deviceset="GND" device=""/>
 </parts>
 <sheets>
@@
 RS-485 to UART4 or
 PRU1 UART0</text>
+<text x="731.52" y="1064.26" size="2.54" layer="150">Jumper AGND to GND
+This is optional. Already
+connected inside SiP</text>
 </plain>
 <instances>
@@
 <attribute name="VALUE" x="686.562" y="951.23" size="1.778" layer="96" rot="MR270"/>
 </instance>
+<instance part="J7" gate="G$1" x="759.46" y="1051.56" smashed="yes" rot="MR0">
+<attribute name="NAME" x="759.46" y="1059.18" size="1.778" layer="95" ratio="10" rot="MR0"/>
+<attribute name="VALUE" x="759.46" y="1049.02" size="1.778" layer="96" ratio="10" rot="MR0"/>
+</instance>
+<instance part="SUPPLY34" gate="G$1" x="734.06" y="1043.94" smashed="yes">
+<attribute name="VALUE" x="734.06" y="1040.384" size="1.778" layer="96" align="center"/>
+</instance>
+<instance part="GND34" gate="1" x="744.22" y="1043.94" smashed="yes">
+<attribute name="VALUE" x="741.68" y="1041.4" size="1.778" layer="96"/>
+</instance>
 </instances>
 <busses>
@@
 <wire x1="744.22" y1="1125.22" x2="744.22" y2="1117.6" width="0.1524" layer="91"/>
 </segment>
+<segment>
+<pinref part="GND34" gate="1" pin="GND"/>
+<wire x1="744.22" y1="1046.48" x2="744.22" y2="1054.1" width="0.1524" layer="91"/>
+<pinref part="J7" gate="G$1" pin="2"/>
+<wire x1="744.22" y1="1054.1" x2="749.3" y2="1054.1" width="0.1524" layer="91"/>
+</segment>
 </net>
 <net name="PWR_BUT" class="0">
@@
 <wire x1="683.26" y1="1117.6" x2="683.26" y2="1120.14" width="0.1524" layer="91"/>
 </segment>
+<segment>
+<pinref part="SUPPLY34" gate="G$1" pin="AGND"/>
+<wire x1="734.06" y1="1046.48" x2="734.06" y2="1056.64" width="0.1524" layer="91"/>
+<pinref part="J7" gate="G$1" pin="1"/>
+<wire x1="734.06" y1="1056.64" x2="749.3" y2="1056.64" width="0.1524" layer="91"/>
+</segment>
 </net>
