File: Version_2.3/Open-Source_Control_V2_R3.brd (EAGLE design)
At the start: 121.9 x 129.5 mm, 354 parts, among them IC10 MCP6002SMT, IC11 MCP6002SMT, IC12 MCP6002SMT, IC14 MCP6002SMT, IC2 ULN2003AD, IC4 74HC165D, IC5 74HC165D, J24 6p-2.54, K1 JS1-24V-F, K2 JS1-24V-F, K3 JS1-24V-F, K4 JS1-24V-F, K5 JS1-24V-F, Q1 MMBT2907, T4 DA2304-AL, U1 OSD3358-512M-ICB, U16 AT97SC3205T-G3M4400B, U2 TPD4S012_DRY_6_P1_M, U27 LAN8710, U28 TCAN1051HV, U29 MAX3483EESA+T, U4 APX811-31UGSOT, U40 ISO3086TDW, U5 TLVH431, U6 SN74LVC2G241_DCU_8, X1 10118194-0001LF, X10 MC4, X11 MC4, X12 MC4, X2 J0011D01BNL, X21 MC10, X24 MSTBA2, X3 MC4, X4 CTI-JTAG, X41 MSTBA3, X5 DM3CS-SF, X6 6p-2.54, X7 TH-2X10, X8 MC4, Y7 ABM3-25.000MHZ-J2Y-T

Commit message: Add files via upload
Parts:
- Y7: value ABM3-25.000MHZ-J2Y-T -> ECS-250-12-30-GN-TR
Changed lines of the file:
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@@
 <element name="X6" library="OSD3358-BSP Ref Design" package="H6-2.54" value="6p-2.54" x="20.32" y="60.96" smashed="yes" rot="R270">
 <attribute name="MPN" value="P125-1106A1BS116A1" x="20.32" y="60.96" size="1.778" layer="27" rot="R270" display="off"/>
+<attribute name="NAME" x="28.067" y="62.357" size="1.016" layer="25" align="top-left"/>
 <attribute name="NAME" x="17.78" y="60.325" size="0.635" layer="33" ratio="10"/>
-<attribute name="NAME" x="28.067" y="62.357" size="1.016" layer="25" align="top-left"/>
 <attribute name="VALUE" x="20.32" y="60.452" size="0.254" layer="27" align="top-center"/>
 </element>
@@
 <attribute name="VALUE" x="36.3982" y="75.565" size="0.254" layer="27" rot="R90" align="top-center"/>
 </element>
-<element name="Y7" library="Open-Source_Control_V2_R2" package="XTAL_2-SMD(5X3.2MM)" value="ABM3-25.000MHZ-J2Y-T" x="35.56" y="72.644" smashed="yes" rot="R180">
+<element name="Y7" library="Open-Source_Control_V2_R2" package="XTAL_2-SMD(5X3.2MM)" value="ECS-250-12-30-GN-TR" x="35.56" y="72.644" smashed="yes" rot="R180">
 <attribute name="NAME" x="32.4358" y="72.644" size="0.8128" layer="25" rot="R90" align="bottom-center"/>
 <attribute name="VALUE" x="35.56" y="72.644" size="0.254" layer="27" rot="R90" align="center"/>
@@
 <element name="J24" library="OSD3358-SM-RED Platform" package="H3-2.54" value="6p-2.54" x="98.425" y="105.41" smashed="yes">
 <attribute name="MPN" value="P125-1106A1BS116A1" x="98.425" y="105.41" size="1.778" layer="27" display="off"/>
+<attribute name="NAME" x="99.06" y="102.87" size="0.635" layer="33" ratio="10" rot="R90"/>
 <attribute name="NAME" x="98.425" y="101.3714" size="0.889" layer="25" ratio="10" align="top-center"/>
-<attribute name="NAME" x="99.06" y="102.87" size="0.635" layer="33" ratio="10" rot="R90"/>
 <attribute name="VALUE" x="98.425" y="104.14" size="0.254" layer="27" align="center"/>
 </element>

Commit message: Add files via upload
Parts:
- K1, K2, K3, K4, K5: value JS1-24V-F -> G5LE-14-CF DC24; device relay:JS-M -> Open-Source_Control_V2_R2:JS-M
Changed lines of the file:
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@@
 <element name="X6" library="OSD3358-BSP Ref Design" package="H6-2.54" value="6p-2.54" x="20.32" y="60.96" smashed="yes" rot="R270">
 <attribute name="MPN" value="P125-1106A1BS116A1" x="20.32" y="60.96" size="1.778" layer="27" rot="R270" display="off"/>
-<attribute name="NAME" x="28.067" y="62.357" size="1.016" layer="25" align="top-left"/>
 <attribute name="NAME" x="17.78" y="60.325" size="0.635" layer="33" ratio="10"/>
+<attribute name="NAME" x="28.067" y="62.357" size="1.016" layer="25" align="top-left"/>
 <attribute name="VALUE" x="20.32" y="60.452" size="0.254" layer="27" align="top-center"/>
 </element>
@@
 <attribute name="VALUE" x="116.205" y="76.2" size="0.889" layer="27" ratio="11" rot="R180"/>
 </element>
-<element name="K1" library="relay" library_urn="urn:adsk.eagle:library:339" package="JS-M" package3d_urn="urn:adsk.eagle:package:24452/1" value="JS1-24V-F" x="95.25" y="50.8" smashed="yes">
-<attribute name="MF" value="FARNELL" x="95.25" y="50.8" size="1.778" layer="27" display="off"/>
-<attribute name="MPN" value="JSM1-12V-5" x="95.25" y="50.8" size="1.778" layer="27" display="off"/>
+<element name="K1" library="Open-Source_Control_V2_R2" package="JS-M" value="G5LE-14-CF DC24" x="95.25" y="50.8" smashed="yes">
 <attribute name="NAME" x="105.2068" y="58.8518" size="1.016" layer="25"/>
-<attribute name="OC_FARNELL" value="910351" x="95.25" y="50.8" size="1.778" layer="27" display="off"/>
-<attribute name="OC_NEWARK" value="14J1764" x="95.25" y="50.8" size="1.778" layer="27" display="off"/>
 <attribute name="VALUE" x="95.25" y="50.8" size="0.8128" layer="27"/>
 </element>
-<element name="K2" library="relay" library_urn="urn:adsk.eagle:library:339" package="JS-M" package3d_urn="urn:adsk.eagle:package:24452/1" value="JS1-24V-F" x="72.39" y="50.8" smashed="yes">
-<attribute name="MF" value="FARNELL" x="50.3682" y="34.7726" size="1.778" layer="27" display="off"/>
-<attribute name="MPN" value="JSM1-12V-5" x="50.3682" y="34.7726" size="1.778" layer="27" display="off"/>
+<element name="K2" library="Open-Source_Control_V2_R2" package="JS-M" value="G5LE-14-CF DC24" x="72.39" y="50.8" smashed="yes">
 <attribute name="NAME" x="61.3664" y="58.8518" size="1.016" layer="25" align="top-right"/>
-<attribute name="OC_FARNELL" value="910351" x="50.3682" y="34.7726" size="1.778" layer="27" display="off"/>
-<attribute name="OC_NEWARK" value="14J1764" x="50.3682" y="34.7726" size="1.778" layer="27" display="off"/>
 <attribute name="VALUE" x="72.39" y="50.8" size="0.8128" layer="27"/>
 </element>
-<element name="K3" library="relay" library_urn="urn:adsk.eagle:library:339" package="JS-M" package3d_urn="urn:adsk.eagle:package:24452/1" value="JS1-24V-F" x="95.25" y="34.29" smashed="yes">
-<attribute name="MF" value="FARNELL" x="95.25" y="18.2626" size="1.778" layer="27" display="off"/>
-<attribute name="MPN" value="JSM1-12V-5" x="95.25" y="18.2626" size="1.778" layer="27" display="off"/>
+<element name="K3" library="Open-Source_Control_V2_R2" package="JS-M" value="G5LE-14-CF DC24" x="95.25" y="34.29" smashed="yes">
 <attribute name="NAME" x="84.2264" y="26.289" size="1.016" layer="25" align="top-right"/>
-<attribute name="OC_FARNELL" value="910351" x="95.25" y="18.2626" size="1.778" layer="27" display="off"/>
-<attribute name="OC_NEWARK" value="14J1764" x="95.25" y="18.2626" size="1.778" layer="27" display="off"/>
 <attribute name="VALUE" x="95.25" y="34.29" size="0.8128" layer="27"/>
 </element>
-<element name="K4" library="relay" library_urn="urn:adsk.eagle:library:339" package="JS-M" package3d_urn="urn:adsk.eagle:package:24452/1" value="JS1-24V-F" x="72.39" y="34.29" smashed="yes">
-<attribute name="MF" value="FARNELL" x="50.3682" y="2.2352" size="1.778" layer="27" display="off"/>
-<attribute name="MPN" value="JSM1-12V-5" x="50.3682" y="2.2352" size="1.778" layer="27" display="off"/>
+<element name="K4" library="Open-Source_Control_V2_R2" package="JS-M" value="G5LE-14-CF DC24" x="72.39" y="34.29" smashed="yes">
 <attribute name="NAME" x="61.3664" y="42.3418" size="1.016" layer="25" align="top-right"/>
-<attribute name="OC_FARNELL" value="910351" x="50.3682" y="2.2352" size="1.778" layer="27" display="off"/>
-<attribute name="OC_NEWARK" value="14J1764" x="50.3682" y="2.2352" size="1.778" layer="27" display="off"/>
 <attribute name="VALUE" x="72.39" y="34.29" size="0.8128" layer="27"/>
 </element>
-<element name="K5" library="relay" library_urn="urn:adsk.eagle:library:339" package="JS-M" package3d_urn="urn:adsk.eagle:package:24452/1" value="JS1-24V-F" x="95.25" y="17.78" smashed="yes">
-<attribute name="MF" value="FARNELL" x="95.25" y="-14.2748" size="1.778" layer="27" display="off"/>
-<attribute name="MPN" value="JSM1-12V-5" x="95.25" y="-14.2748" size="1.778" layer="27" display="off"/>
+<element name="K5" library="Open-Source_Control_V2_R2" package="JS-M" value="G5LE-14-CF DC24" x="95.25" y="17.78" smashed="yes">
 <attribute name="NAME" x="84.2264" y="9.779" size="1.016" layer="25" align="top-right"/>
-<attribute name="OC_FARNELL" value="910351" x="95.25" y="-14.2748" size="1.778" layer="27" display="off"/>
-<attribute name="OC_NEWARK" value="14J1764" x="95.25" y="-14.2748" size="1.778" layer="27" display="off"/>
 <attribute name="VALUE" x="95.25" y="17.78" size="0.8128" layer="27"/>
 </element>
@@
 <element name="J24" library="OSD3358-SM-RED Platform" package="H3-2.54" value="6p-2.54" x="98.425" y="105.41" smashed="yes">
 <attribute name="MPN" value="P125-1106A1BS116A1" x="98.425" y="105.41" size="1.778" layer="27" display="off"/>
-<attribute name="NAME" x="99.06" y="102.87" size="0.635" layer="33" ratio="10" rot="R90"/>
 <attribute name="NAME" x="98.425" y="101.3714" size="0.889" layer="25" ratio="10" align="top-center"/>
+<attribute name="NAME" x="99.06" y="102.87" size="0.635" layer="33" ratio="10" rot="R90"/>
 <attribute name="VALUE" x="98.425" y="104.14" size="0.254" layer="27" align="center"/>
 </element>
@@
 <via x="101.6" y="62.992" extent="1-16" drill="0.3048"/>
 <via x="102.616" y="62.992" extent="1-16" drill="0.3048"/>
+<wire x1="88.268" y1="106.7308" x2="98.425" y2="102.87" width="0" layer="19" extent="1-1"/>
+<wire x1="95.7834" y1="65.405" x2="98.425" y2="102.87" width="0" layer="19" extent="1-1"/>
+<wire x1="95.885" y1="64.643" x2="95.7834" y2="65.405" width="0" layer="19" extent="1-1"/>
+<wire x1="96.901" y1="64.643" x2="95.885" y2="64.643" width="0" layer="19" extent="1-1"/>
+<wire x1="94.869" y1="64.643" x2="95.885" y2="64.643" width="0" layer="19" extent="1-1"/>
+<wire x1="101.6" y1="65.024" x2="96.901" y2="64.643" width="0" layer="19" extent="1-1"/>
+<wire x1="102.616" y1="65.024" x2="101.6" y2="65.024" width="0" layer="19" extent="1-1"/>
+<wire x1="102.616" y1="64.008" x2="102.616" y2="65.024" width="0" layer="19" extent="1-1"/>
+<wire x1="101.6" y1="64.008" x2="101.6" y2="65.024" width="0" layer="19" extent="1-1"/>
+<wire x1="101.6" y1="62.992" x2="101.6" y2="64.008" width="0" layer="19" extent="1-1"/>
+<wire x1="102.616" y1="62.992" x2="102.616" y2="64.008" width="0" layer="19" extent="1-1"/>
+<wire x1="101.95" y1="56.8" x2="101.6" y2="62.992" width="0" layer="19" extent="1-1"/>
+<wire x1="109.8423" y1="59.436" x2="102.616" y2="62.992" width="0" layer="19" extent="1-1"/>
+<wire x1="109.8423" y1="51.816" x2="109.8423" y2="59.436" width="0" layer="19" extent="1-1"/>
+<wire x1="109.8423" y1="46.101" x2="109.8423" y2="51.816" width="0" layer="19" extent="1-1"/>
+<wire x1="109.8423" y1="44.196" x2="109.8423" y2="46.101" width="0" layer="19" extent="1-1"/>
+<wire x1="109.8423" y1="36.576" x2="109.8423" y2="44.196" width="0" layer="19" extent="1-1"/>
+<wire x1="109.8423" y1="30.861" x2="109.8423" y2="36.576" width="0" layer="19" extent="1-1"/>
+<wire x1="109.8423" y1="28.956" x2="109.8423" y2="30.861" width="0" layer="19" extent="1-1"/>
+<wire x1="113.792" y1="19.685" x2="109.8423" y2="28.956" width="0" layer="19" extent="1-1"/>
 </signal>
 <signal name="N$93">

Commit message: Add files via upload
Parts:
- D1: value LTST-C191KFKT -> LTST-C191KGKT; device OSD3358-BSP Ref Design:EIA-STD -> Open-Source_Control_V2_R2:EIA-STD
- D19: device OSD3358-SM-RED Platform:EIA-STD -> Open-Source_Control_V2_R2:EIA-STD
- X21: value MC10 -> MC12; device con-phoenix-381_l:MC10 -> con-phoenix-381_l:MC12
- moved J2 11.7 mm to (92.7, 76.2)
- moved J4 5.08 mm to (74.9, 20.3)
- moved J6 5.08 mm to (74.9, 15.2)
- moved R69 4.62 mm to (102.2, 75.3)
- moved K1 3.81 mm to (91.4, 50.8)
- moved K2 3.81 mm to (68.6, 50.8)
- moved K3 3.81 mm to (91.4, 34.3)
- moved K4 3.81 mm to (68.6, 34.3)
- moved K5 3.81 mm to (91.4, 17.8)
- moved D19 3.56 mm to (114.3, 126.9)
- moved R171 3.29 mm to (105.4, 57.1), turned to 180 degrees
- moved R172 3.29 mm to (105.4, 49.5), turned to 180 degrees
- moved R174 3.29 mm to (105.4, 34.3), turned to 180 degrees
- moved R175 3.29 mm to (105.4, 26.7), turned to 180 degrees
- moved R173 3.29 mm to (105.4, 41.9), turned to 180 degrees
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Connections:
- net 24VDC_AUX: now also X21.12
- net GND: now also X21.11
Routing:
- net N$129: track 122.5 -> 65.8 mm
- net N$124: track 108.1 -> 51.5 mm, vias 0 -> 2
- net N$119: track 91.6 -> 37.9 mm, vias 0 -> 2
- net 24VDC_AUX: track 113.1 -> 151.5 mm, vias 9 -> 8
- net PMIC_NRESET: track 54.0 -> 41.5 mm, vias 2 -> 1
- net N$120: track 87.3 -> 75.7 mm, vias 0 -> 1
- net EHRPWM1A: track 115.5 -> 105.0 mm
- net N$110: track 53.9 -> 62.6 mm, vias 1 -> 2
- net SPI1_D0: track 49.1 -> 55.7 mm
- net LCD_DATA2: track 46.3 -> 41.0 mm, vias 2 -> 3
- net EHRPWM2A: track 110.6 -> 105.6 mm
- net BO2_NO: track 52.3 -> 56.2 mm
- net BO1_NO: track 27.8 -> 31.7 mm
- net N$111: track 7.98 -> 11.8 mm
- net BO4_NO: track 52.9 -> 56.8 mm
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
Commit message: Add files via upload
Parts:
- moved J5 3.81 mm to (74.9, 14.0)
- moved J6 3.81 mm to (74.9, 11.4)
- moved J4 3.81 mm to (74.9, 16.5)
Routing:
- net EHRPWM2B: track 108.3 -> 109.9 mm
- net EHRPWM2A: track 105.6 -> 107.2 mm
- net EHRPWM1A: track 105.0 -> 106.5 mm
- net LCD_DATA0: track 30.1 -> 28.8 mm
- net LCD_DATA1: track 33.9 -> 32.8 mm
- net LCD_DATA2: track 41.0 -> 40.0 mm
- net LCD_DATA3: track 35.3 -> 34.5 mm
- net LCD_DATA4: track 28.2 -> 27.5 mm
- net LCD_DATA5: track 33.0 -> 32.5 mm
