File: Version_2.3/Open-Source_Control_V2_R3.sch (EAGLE design)
At the start: 352 parts, among them IC10 MCP6002SMT, IC11 MCP6002SMT, IC12 MCP6002SMT, IC14 MCP6002SMT, IC2 ULN2003AD, IC4 74HC165D, IC5 74HC165D, J24 6p-2.54, K1 JS1-24V-F, K2 JS1-24V-F, K3 JS1-24V-F, K4 JS1-24V-F, K5 JS1-24V-F, Q1 MMBT2907, T4 DA2304-AL, U1 OSD3358-512M-ICB, U16 AT97SC3205T-G3M4400B, U2 TPD4S012_DRY_6_P1_M, U27 LAN8710, U28 TCAN1051HV, U29 MAX3483EESA+T, U4 APX811-31UGSOT, U40 ISO3086TDW, U5 TLVH431, U6 SN74LVC2G241_DCU_8, X1 10118194-0001LF, X10 MC4, X11 MC4, X12 MC4, X2 J0011D01BNL, X21 MC10, X24 MSTBA2, X3 MC4, X4 CTI-JTAG, X41 MSTBA3, X5 DM3CS-SF, X6 6p-2.54, X7 TH-2X10, X8 MC4, Y7 ABM3-25.000MHZ-J2Y-T

Commit message: Add files via upload
Parts:
- Y7: value ABM3-25.000MHZ-J2Y-T -> ECS-250-12-30-GN-TR
Changed lines of the file:
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@@
 <part name="ER126" library="OSD3358-SM-RED Platform" deviceset="R-US_" device="R0402" value="0, 1%"/>
 <part name="GND132" library="OSD3358-SM-RED Platform" deviceset="GND" device=""/>
-<part name="Y7" library="Open-Source_Control_V2_R2" deviceset="CRYSTAL-2-SMD" device="" value="ABM3-25.000MHZ-J2Y-T"/>
+<part name="Y7" library="Open-Source_Control_V2_R2" deviceset="CRYSTAL-2-SMD" device="" value="ECS-250-12-30-GN-TR"/>
 <part name="ER127" library="OSD3358-SM-RED Platform" deviceset="R-US_" device="R0402" value="10, 1%"/>
 <part name="GND133" library="OSD3358-SM-RED Platform" deviceset="GND" device=""/>

Commit message: Add files via upload
Parts:
- K1, K2, K3, K4, K5: value JS1-24V-F -> G5LE-14-CF DC24; device relay:JS-M1-12V-5 -> Open-Source_Control_V2_R2:G5LE-14-CF
Changed lines of the file:
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@@
 <part name="GND159" library="OSD3358-SM-RED Platform" deviceset="GND" device=""/>
 <part name="J3" library="OSD3358-SM-RED Platform" deviceset="826646-2" device=""/>
-<part name="K1" library="relay" library_urn="urn:adsk.eagle:library:339" deviceset="JS-M1*" device="" package3d_urn="urn:adsk.eagle:package:24452/1" technology="-12V-5" value="JS1-24V-F"/>
-<part name="K2" library="relay" library_urn="urn:adsk.eagle:library:339" deviceset="JS-M1*" device="" package3d_urn="urn:adsk.eagle:package:24452/1" technology="-12V-5" value="JS1-24V-F"/>
-<part name="K3" library="relay" library_urn="urn:adsk.eagle:library:339" deviceset="JS-M1*" device="" package3d_urn="urn:adsk.eagle:package:24452/1" technology="-12V-5" value="JS1-24V-F"/>
-<part name="K4" library="relay" library_urn="urn:adsk.eagle:library:339" deviceset="JS-M1*" device="" package3d_urn="urn:adsk.eagle:package:24452/1" technology="-12V-5" value="JS1-24V-F"/>
-<part name="K5" library="relay" library_urn="urn:adsk.eagle:library:339" deviceset="JS-M1*" device="" package3d_urn="urn:adsk.eagle:package:24452/1" technology="-12V-5" value="JS1-24V-F"/>
+<part name="K1" library="Open-Source_Control_V2_R2" deviceset="G5LE" device="" technology="-14-CF" value="G5LE-14-CF DC24"/>
+<part name="K2" library="Open-Source_Control_V2_R2" deviceset="G5LE" device="" technology="-14-CF" value="G5LE-14-CF DC24"/>
+<part name="K3" library="Open-Source_Control_V2_R2" deviceset="G5LE" device="" technology="-14-CF" value="G5LE-14-CF DC24"/>
+<part name="K4" library="Open-Source_Control_V2_R2" deviceset="G5LE" device="" technology="-14-CF" value="G5LE-14-CF DC24"/>
+<part name="K5" library="Open-Source_Control_V2_R2" deviceset="G5LE" device="" technology="-14-CF" value="G5LE-14-CF DC24"/>
 <part name="X21" library="con-phoenix-381_l" deviceset="MC10" device=""/>
 <part name="IC2" library="uln-udn" library_urn="urn:adsk.eagle:library:407" deviceset="ULN2003A" device="D" package3d_urn="urn:adsk.eagle:package:30247/1"/>

Commit message: Add files via upload
Parts:
- D1: value LTST-C191KFKT -> LTST-C191KGKT; device OSD3358-SM-RED Platform:LTST-C191KFKTLED_EIA-STD -> Open-Source_Control_V2_R2:LTST-C191KGKTLED_EIA-STD
- D19: device OSD3358-SM-RED Platform:LTST-C191KGKTLED_EIA-STD -> Open-Source_Control_V2_R2:LTST-C191KGKTLED_EIA-STD
- X21: value MC10 -> MC12; device con-phoenix-381_l:MC10 -> con-phoenix-381_l:MC12
Connections:
- net 24VDC_AUX: now also X21.12.SK
- net GND: now also X21.11.SK
Other:
- moved on the sheet: X8.1

Commit message: Add files via upload
Other:
- note added: "Modular IO Connections"
- note removed: "Future AO Connect"
- moved on the sheet: J4, J5, J6
Changed lines of the file:
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@@
 should be added to reduce noise, if needed
 for your application.</text>
-<text x="1023.62" y="825.5" size="10.16" layer="94">Future AO Connect</text>
+<text x="1005.84" y="840.74" size="10.16" layer="94">Modular IO Connections</text>
 <text x="1041.4" y="393.7" size="2.54" layer="150" rot="MR0" align="top-center">TENS</text>
 <text x="1041.4" y="419.1" size="2.54" layer="150" rot="MR0" align="top-center">ONES</text>
@@
 <attribute name="VALUE" x="762" y="1004.824" size="1.778" layer="96" align="center"/>
 </instance>
-<instance part="J4" gate="G$1" x="1094.74" y="802.64" smashed="yes" rot="MR0">
-<attribute name="NAME" x="1094.74" y="810.26" size="1.778" layer="95" ratio="10" rot="MR0"/>
-<attribute name="VALUE" x="1094.74" y="800.1" size="1.778" layer="96" ratio="10" rot="MR0"/>
-</instance>
-<instance part="J5" gate="G$1" x="1094.74" y="784.86" smashed="yes" rot="MR0">
-<attribute name="NAME" x="1094.74" y="792.48" size="1.778" layer="95" ratio="10" rot="MR0"/>
-<attribute name="VALUE" x="1094.74" y="782.32" size="1.778" layer="96" ratio="10" rot="MR0"/>
-</instance>
-<instance part="J6" gate="G$1" x="1094.74" y="767.08" smashed="yes" rot="MR0">
-<attribute name="NAME" x="1094.74" y="774.7" size="1.778" layer="95" ratio="10" rot="MR0"/>
-<attribute name="VALUE" x="1094.74" y="764.54" size="1.778" layer="96" ratio="10" rot="MR0"/>
+<instance part="J4" gate="G$1" x="1094.74" y="795.02" smashed="yes" rot="MR0">
+<attribute name="NAME" x="1094.74" y="802.64" size="1.778" layer="95" ratio="10" rot="MR0"/>
+<attribute name="VALUE" x="1094.74" y="792.48" size="1.778" layer="96" ratio="10" rot="MR0"/>
+</instance>
+<instance part="J5" gate="G$1" x="1094.74" y="777.24" smashed="yes" rot="MR0">
+<attribute name="NAME" x="1094.74" y="784.86" size="1.778" layer="95" ratio="10" rot="MR0"/>
+<attribute name="VALUE" x="1094.74" y="774.7" size="1.778" layer="96" ratio="10" rot="MR0"/>
+</instance>
+<instance part="J6" gate="G$1" x="1094.74" y="759.46" smashed="yes" rot="MR0">
+<attribute name="NAME" x="1094.74" y="767.08" size="1.778" layer="95" ratio="10" rot="MR0"/>
+<attribute name="VALUE" x="1094.74" y="756.92" size="1.778" layer="96" ratio="10" rot="MR0"/>
 </instance>
-<instance part="GND24" gate="1" x="1082.04" y="800.1" smashed="yes">
-<attribute name="VALUE" x="1079.5" y="797.56" size="1.778" layer="96"/>
+<instance part="GND24" gate="1" x="1082.04" y="792.48" smashed="yes">
+<attribute name="VALUE" x="1079.5" y="789.94" size="1.778" layer="96"/>
 </instance>
-<instance part="GND30" gate="1" x="1082.04" y="782.32" smashed="yes">
-<attribute name="VALUE" x="1079.5" y="779.78" size="1.778" layer="96"/>
+<instance part="GND30" gate="1" x="1082.04" y="774.7" smashed="yes">
+<attribute name="VALUE" x="1079.5" y="772.16" size="1.778" layer="96"/>
 </instance>
-<instance part="GND31" gate="1" x="1082.04" y="764.54" smashed="yes">
-<attribute name="VALUE" x="1079.5" y="762" size="1.778" layer="96"/>
+<instance part="GND31" gate="1" x="1082.04" y="756.92" smashed="yes">
+<attribute name="VALUE" x="1079.5" y="754.38" size="1.778" layer="96"/>
 </instance>
 <instance part="TP17" gate="G$1" x="60.96" y="86.36" smashed="yes" rot="R180">
@@
 <pinref part="J4" gate="G$1" pin="2"/>
 <pinref part="GND24" gate="1" pin="GND"/>
-<wire x1="1084.58" y1="805.18" x2="1082.04" y2="805.18" width="0.1524" layer="91"/>
-<wire x1="1082.04" y1="805.18" x2="1082.04" y2="802.64" width="0.1524" layer="91"/>
+<wire x1="1084.58" y1="797.56" x2="1082.04" y2="797.56" width="0.1524" layer="91"/>
+<wire x1="1082.04" y1="797.56" x2="1082.04" y2="795.02" width="0.1524" layer="91"/>
 </segment>
 <segment>
 <pinref part="J5" gate="G$1" pin="2"/>
-<wire x1="1084.58" y1="787.4" x2="1082.04" y2="787.4" width="0.1524" layer="91"/>
+<wire x1="1084.58" y1="779.78" x2="1082.04" y2="779.78" width="0.1524" layer="91"/>
 <pinref part="GND30" gate="1" pin="GND"/>
-<wire x1="1082.04" y1="787.4" x2="1082.04" y2="784.86" width="0.1524" layer="91"/>
+<wire x1="1082.04" y1="779.78" x2="1082.04" y2="777.24" width="0.1524" layer="91"/>
 </segment>
 <segment>
 <pinref part="J6" gate="G$1" pin="2"/>
-<wire x1="1084.58" y1="769.62" x2="1082.04" y2="769.62" width="0.1524" layer="91"/>
+<wire x1="1084.58" y1="762" x2="1082.04" y2="762" width="0.1524" layer="91"/>
 <pinref part="GND31" gate="1" pin="GND"/>
-<wire x1="1082.04" y1="769.62" x2="1082.04" y2="767.08" width="0.1524" layer="91"/>
+<wire x1="1082.04" y1="762" x2="1082.04" y2="759.46" width="0.1524" layer="91"/>
 </segment>
 <segment>
@@
 <segment>
 <pinref part="J6" gate="G$1" pin="1"/>
-<wire x1="1084.58" y1="772.16" x2="1064.26" y2="772.16" width="0.1524" layer="91"/>
-<label x="1064.26" y="772.16" size="1.778" layer="95"/>
+<wire x1="1084.58" y1="764.54" x2="1064.26" y2="764.54" width="0.1524" layer="91"/>
+<label x="1064.26" y="764.54" size="1.778" layer="95"/>
 </segment>
 </net>
@@
 <segment>
 <pinref part="J5" gate="G$1" pin="1"/>
-<wire x1="1084.58" y1="789.94" x2="1064.26" y2="789.94" width="0.1524" layer="91"/>
-<label x="1064.26" y="789.94" size="1.778" layer="95"/>
+<wire x1="1084.58" y1="782.32" x2="1064.26" y2="782.32" width="0.1524" layer="91"/>
+<label x="1064.26" y="782.32" size="1.778" layer="95"/>
 </segment>
 </net>
@@
 <segment>
 <pinref part="J4" gate="G$1" pin="1"/>
-<wire x1="1084.58" y1="807.72" x2="1064.26" y2="807.72" width="0.1524" layer="91"/>
-<label x="1064.26" y="807.72" size="1.778" layer="95"/>
+<wire x1="1084.58" y1="800.1" x2="1064.26" y2="800.1" width="0.1524" layer="91"/>
+<label x="1064.26" y="800.1" size="1.778" layer="95"/>
 </segment>
 </net>
