File: Version_3.0/Open-Source_Control_V3_R0.brd (EAGLE design)
At the start: 121.9 x 129.5 mm, 348 parts, among them IC10 MCP6002SMT, IC11 MCP6002SMT, IC12 MCP6002SMT, IC14 MCP6002SMT, IC2 ULN2003AD, IC4 74HC165D, IC5 74HC165D, J24 6p-2.54, K1 G5LE-14-CF DC24, K2 G5LE-14-CF DC24, K3 G5LE-14-CF DC24, K4 G5LE-14-CF DC24, Q1 MMBT2907, T4 DA2304-AL, U1 OSD3358-512M-ICB, U16 AT97SC3205T-G3M4400B, U2 TPD4S012_DRY_6_P1_M, U27 LAN8710, U28 TCAN1051HV, U29 MAX3483EESA+T, U4 APX811-31UGSOT, U40 ISO3086TDW, U5 TLVH431, U6 SN74LVC2G241_DCU_8, X1 10118194-0001LF, X10 MC4, X11 MC4, X12 MC4, X2 J0011D01BNL, X21 MC12, X24 MSTBA2, X3 MC4, X31 MC4, X4 CTI-JTAG, X41 MSTBA3, X5 DM3CS-SF, X6 6p-2.54, X7 TH-2X10, X8 TH-2X10, X9 5600200420, Y7 ECS-250-12-30-GN-TR

Commit message: Add files via upload
Parts:
- moved X8 1.27 mm to (88.9, 14.0)
Connections:
- net 24VDC_AUX: now also X8.11; no longer X8.12, X8.20
- net PMIC_NRESET: now also X8.12; no longer X8.11
Routing:
- net BO3: track 48.7 -> 67.7 mm
- net BO2: track 42.0 -> 58.0 mm, vias 1 -> 0
- net BO4: track 17.1 -> 27.2 mm
- net 24VDC_AUX: track 92.2 -> 85.8 mm
- net PMIC_NRESET: track 101.7 -> 105.5 mm
- net EHRPWM2B: track 100.1 -> 101.4 mm
- net EHRPWM1A: track 100.6 -> 101.9 mm
- net BO2_AUTO: track 59.1 -> 60.4 mm
- net BO1_AUTO: track 61.0 -> 62.3 mm
- net EHRPWM2A: track 97.4 -> 98.6 mm
- net BO5_AUTO: track 58.7 -> 60.0 mm
- net BO4_AUTO: track 58.6 -> 59.9 mm
- net BO3_AUTO: track 58.5 -> 59.7 mm
- net BO1: track 78.9 -> 80.2 mm

Commit message: Add files via upload
Connections:
- net SYS_VDD1_3P3V: no longer C801.1, U28.3
- net VDD_5V: now also C801.1, U28.3
Routing:
- net VDD_5V: track 15.5 -> 172.3 mm, vias 3 -> 7
- net SYS_VDD1_3P3V: track 78.9 -> 75.7 mm, vias 43 -> 42
- net VDD_BAT: track 18.3 -> 18.8 mm
Changed lines of the file:
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@@
 <wire x1="53.721" y1="120.904" x2="51.311" y2="123.314" width="0.8128" layer="1"/>
 <wire x1="51.311" y1="123.314" x2="49.276" y2="123.314" width="0.8128" layer="1"/>
+<contactref element="C801" pad="1"/>
+<contactref element="U28" pad="3"/>
+<via x="93.472" y="5.715" extent="1-16" drill="0.3048"/>
+<wire x1="94.2594" y1="6.5024" x2="117.3988" y2="6.5024" width="0.254" layer="16"/>
+<wire x1="117.3988" y1="6.5024" x2="118.6688" y2="7.7724" width="0.254" layer="16"/>
+<wire x1="118.6688" y1="7.7724" x2="118.6688" y2="75.7428" width="0.254" layer="16"/>
+<wire x1="118.6688" y1="75.7428" x2="117.3988" y2="77.0128" width="0.254" layer="16"/>
+<wire x1="117.3988" y1="77.0128" x2="116.078" y2="77.0128" width="0.254" layer="16"/>
+<wire x1="116.078" y1="77.0128" x2="114.808" y2="78.2828" width="0.254" layer="16"/>
+<wire x1="114.808" y1="78.2828" x2="114.808" y2="87.249" width="0.254" layer="16"/>
+<wire x1="114.808" y1="87.249" x2="113.538" y2="88.519" width="0.254" layer="16"/>
+<wire x1="113.538" y1="88.519" x2="100.33" y2="88.519" width="0.254" layer="16"/>
+<wire x1="100.33" y1="88.519" x2="99.06" y2="89.789" width="0.254" layer="16"/>
+<wire x1="99.06" y1="89.789" x2="99.06" y2="96.012" width="0.254" layer="16"/>
+<wire x1="93.472" y1="5.715" x2="94.2594" y2="6.5024" width="0.254" layer="16"/>
+<via x="81.026" y="102.235" extent="1-16" drill="0.3048"/>
+<wire x1="81.026" y1="102.235" x2="81.026" y2="100.6348" width="0.254" layer="16"/>
+<via x="92.71" y="100.33" extent="1-16" drill="0.3048"/>
+<via x="99.06" y="96.012" extent="1-16" drill="0.3048"/>
+<wire x1="81.3308" y1="100.33" x2="92.71" y2="100.33" width="0.254" layer="16"/>
+<wire x1="81.026" y1="100.6348" x2="81.3308" y2="100.33" width="0.254" layer="16"/>
+<wire x1="92.71" y1="100.33" x2="94.869" y2="100.33" width="0.254" layer="1"/>
+<wire x1="94.869" y1="100.33" x2="96.139" y2="99.06" width="0.254" layer="1"/>
+<wire x1="96.139" y1="99.06" x2="96.139" y2="97.282" width="0.254" layer="1"/>
+<wire x1="96.139" y1="97.282" x2="97.409" y2="96.012" width="0.254" layer="1"/>
+<wire x1="97.409" y1="96.012" x2="99.06" y2="96.012" width="0.254" layer="1"/>
+<wire x1="93.472" y1="5.715" x2="92.1512" y2="5.715" width="0.254" layer="1"/>
+<wire x1="92.1512" y1="5.715" x2="92.075" y2="5.7912" width="0.254" layer="1"/>
+<wire x1="93.472" y1="5.715" x2="95.3262" y2="5.715" width="0.254" layer="1"/>
 </signal>
 <signal name="GND">
@@
 <vertex x="75.692" y="10.1092"/>
 </polygon>
-<wire x1="95.3262" y1="6.985" x2="93.472" y2="6.985" width="0.1524" layer="1"/>
-<wire x1="93.472" y1="6.985" x2="92.1512" y2="6.985" width="0.1524" layer="1"/>
-<wire x1="92.1512" y1="6.985" x2="92.075" y2="6.9088" width="0.1524" layer="1"/>
 <via x="32.004" y="58.42" extent="1-16" drill="0.3048"/>
 <via x="29.718" y="57.15" extent="1-16" drill="0.3048"/>
@@
 <vertex x="69.9262" y="56.7944"/>
 </polygon>
+<wire x1="93.472" y1="6.985" x2="95.3262" y2="6.985" width="0.254" layer="1"/>
+<wire x1="93.472" y1="6.985" x2="92.1512" y2="6.985" width="0.254" layer="1"/>
+<wire x1="92.1512" y1="6.985" x2="92.075" y2="6.9088" width="0.254" layer="1"/>
 </signal>
 <signal name="PWR_BUT">
@@
 <vertex x="76.835" y="99.187"/>
 </polygon>
-<wire x1="78.1558" y1="98.8314" x2="76.5556" y2="98.8314" width="0.8128" layer="16"/>
+<wire x1="76.5556" y1="98.8314" x2="77.7748" y2="98.8314" width="0.8128" layer="16"/>
+<wire x1="77.7748" y1="98.8314" x2="79.0448" y2="100.1014" width="0.8128" layer="16"/>
+<wire x1="79.0448" y1="100.1014" x2="79.0448" y2="102.87" width="0.8128" layer="16"/>
+<wire x1="79.0448" y1="102.87" x2="80.3148" y2="104.14" width="0.8128" layer="16"/>
+<wire x1="80.3148" y1="104.14" x2="91.44" y2="104.14" width="0.8128" layer="16"/>
 <wire x1="76.454" y1="98.933" x2="76.5556" y2="98.8314" width="0.6096" layer="16"/>
-<wire x1="78.1558" y1="98.8314" x2="80.1624" y2="100.838" width="0.8128" layer="16"/>
-<wire x1="80.1624" y1="100.838" x2="80.1624" y2="102.6922" width="0.8128" layer="16"/>
-<wire x1="80.1624" y1="102.6922" x2="81.6102" y2="104.14" width="0.8128" layer="16"/>
-<wire x1="81.6102" y1="104.14" x2="91.44" y2="104.14" width="0.8128" layer="16"/>
 </signal>
 <signal name="VDD_ETH_PHY">
@@
 <vertex x="32.258" y="89.154"/>
 </polygon>
-<contactref element="U28" pad="3"/>
 <wire x1="52.2732" y1="68.6943" x2="52.2732" y2="68.19391875" width="0.254" layer="1"/>
 <via x="52.1462" y="69.1896" extent="1-16" drill="0.3048"/>
@@
 <wire x1="21.6662" y1="64.135" x2="20.6502" y2="64.135" width="0.254" layer="1"/>
 <wire x1="20.6502" y1="64.135" x2="20.0914" y2="63.5762" width="0.254" layer="1"/>
-<via x="93.472" y="5.715" extent="1-16" drill="0.3048"/>
-<contactref element="C801" pad="1"/>
 <contactref element="IC14" pad="8"/>
 <via x="61.468" y="5.08" extent="1-16" drill="0.3048"/>
@@
 <vertex x="71.882" y="12.6746"/>
 </polygon>
-<wire x1="95.3262" y1="5.715" x2="93.472" y2="5.715" width="0.1524" layer="1"/>
-<wire x1="93.472" y1="5.715" x2="92.1512" y2="5.715" width="0.1524" layer="1"/>
-<wire x1="92.1512" y1="5.715" x2="92.075" y2="5.7912" width="0.1524" layer="1"/>
 </signal>
 <signal name="SYS_VDD_1P8V">

Commit message: Add files via upload
Parts:
- R801, R802: value 1K -> 500
- turned D801 to 90 degrees
- turned D802 to 90 degrees
- turned R801 to 90 degrees
- turned R802 to 90 degrees
Connections:
- removed net VIO: U28.5
- net CAN1_RXD: now also D802.2; no longer D802.1
- net CAN1_TXD: now also D801.2; no longer D801.1
- net GND: no longer R801.2, R802.2
- net N$5: now also D802.1, R802.2; no longer D802.2, R802.1
- net N$6: now also D801.1, R801.2; no longer D801.2, R801.1
- net SYS_VDD1_3P3V: now also U28.5
- net VDD_5V: now also R801.1, R802.1
Routing:
- net VDD_5V: track 172.3 -> 189.7 mm, vias 7 -> 8
- net CAN1_TXD: track 176.0 -> 192.8 mm, vias 5 -> 4
- net GND: track 182.5 -> 180.5 mm, vias 200 -> 199
- net SYS_VDD1_3P3V: track 75.7 -> 77.5 mm, vias 42 -> 43

Commit message: Add files via upload
Parts:
- added C802: 0.1uF, 6.3V, OSD3358-SM-RED Platform:C0402
- added C803: 4.7uF, 6.3V, OSD3358-SM-RED Platform:C0402
Connections:
- net GND: now also C802.2, C803.2
- net SYS_VDD1_3P3V: now also C802.1, R801.1, R802.1
- net VDD_5V: now also C803.1; no longer R801.1, R802.1
Routing:
- net VDD_5V: track 189.7 -> 173.3 mm, vias 8 -> 7
- net SYS_VDD1_3P3V: track 77.5 -> 80.8 mm, vias 43 -> 44
- net GND: track 180.5 -> 182.6 mm, vias 199 -> 200
- net CAN1_RXD: track 171.6 -> 172.3 mm
Changed lines of the file:
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@@
 <element name="X6" library="OSD3358-BSP Ref Design" package="H6-2.54" value="6p-2.54" x="20.32" y="60.96" smashed="yes" rot="R270">
 <attribute name="MPN" value="P125-1106A1BS116A1" x="20.32" y="60.96" size="1.778" layer="27" rot="R270" display="off"/>
-<attribute name="NAME" x="28.067" y="62.357" size="1.016" layer="25" align="top-left"/>
 <attribute name="NAME" x="17.78" y="60.325" size="0.635" layer="33" ratio="10"/>
+<attribute name="NAME" x="28.067" y="62.357" size="1.016" layer="25" align="top-left"/>
 <attribute name="VALUE" x="20.32" y="60.452" size="0.254" layer="27" align="top-center"/>
 </element>
@@
 </element>
 <element name="C801" library="OSD3358-SM-RED Platform" package="C0402" value="0.1uF, 6.3V" x="92.075" y="6.35" smashed="yes" rot="R90">
-<attribute name="NAME" x="91.5416" y="6.35" size="0.8128" layer="25" align="center-right"/>
-<attribute name="VALUE" x="92.075" y="5.2324" size="0.254" layer="27" align="top-center"/>
+<attribute name="NAME" x="92.075" y="5.2324" size="0.8128" layer="25" rot="R90" align="center-right"/>
+<attribute name="VALUE" x="92.583" y="6.35" size="0.254" layer="27" rot="R90" align="top-center"/>
 </element>
 <element name="R303" library="OSD3358-SM-RED Platform" package="R0402" value="1K, DNI" x="18.288" y="64.135" smashed="yes" rot="R270">
@@
 <element name="J24" library="OSD3358-SM-RED Platform" package="H3-2.54" value="6p-2.54" x="98.425" y="105.41" smashed="yes">
 <attribute name="MPN" value="P125-1106A1BS116A1" x="98.425" y="105.41" size="1.778" layer="27" display="off"/>
-<attribute name="NAME" x="99.06" y="102.87" size="0.635" layer="33" ratio="10" rot="R90"/>
 <attribute name="NAME" x="98.425" y="101.3714" size="0.889" layer="25" ratio="10" align="top-center"/>
+<attribute name="NAME" x="99.06" y="102.87" size="0.635" layer="33" ratio="10" rot="R90"/>
 <attribute name="VALUE" x="98.425" y="104.14" size="0.254" layer="27" align="center"/>
 </element>
@@
 <attribute name="VALUE" x="89.8398" y="10.0076" size="0.889" layer="27" ratio="11"/>
 </element>
+<element name="C802" library="OSD3358-SM-RED Platform" package="C0402" value="0.1uF, 6.3V" x="103.886" y="4.445" smashed="yes">
+<attribute name="NAME" x="102.7684" y="4.953" size="0.8128" layer="25"/>
+<attribute name="VALUE" x="102.997" y="3.683" size="0.254" layer="27"/>
+</element>
+<element name="C803" library="OSD3358-SM-RED Platform" package="C0402" value="4.7uF, 6.3V" x="91.059" y="6.35" smashed="yes" rot="R90">
+<attribute name="NAME" x="91.059" y="5.2324" size="0.8128" layer="25" rot="R90" align="center-right"/>
+<attribute name="VALUE" x="90.551" y="6.35" size="0.254" layer="27" rot="R90" align="bottom-center"/>
+</element>
 </elements>
 <signals>
@@
 <wire x1="96.139" y1="97.282" x2="97.409" y2="96.012" width="0.254" layer="1"/>
 <wire x1="97.409" y1="96.012" x2="99.06" y2="96.012" width="0.254" layer="1"/>
-<contactref element="R802" pad="1"/>
-<contactref element="R801" pad="1"/>
 <contactref element="C801" pad="1"/>
 <contactref element="U28" pad="3"/>
@@
 <wire x1="92.1512" y1="5.715" x2="92.075" y2="5.7912" width="0.254" layer="1"/>
 <wire x1="93.472" y1="5.715" x2="95.3262" y2="5.715" width="0.254" layer="1"/>
-<via x="108.204" y="4.2672" extent="1-16" drill="0.3048"/>
-<wire x1="93.472" y1="5.715" x2="97.1296" y2="5.715" width="0.254" layer="16"/>
-<wire x1="107.3912" y1="5.08" x2="108.204" y2="4.2672" width="0.254" layer="16"/>
-<wire x1="107.3912" y1="5.08" x2="97.7646" y2="5.08" width="0.254" layer="16"/>
-<wire x1="97.1296" y1="5.715" x2="97.7646" y2="5.08" width="0.254" layer="16"/>
-<wire x1="108.204" y1="4.2672" x2="107.188" y2="4.2672" width="0.254" layer="1"/>
-<wire x1="108.204" y1="4.2672" x2="109.22" y2="4.2672" width="0.254" layer="1"/>
+<contactref element="C803" pad="1"/>
+<wire x1="91.059" y1="5.7912" x2="92.075" y2="5.7912" width="0.254" layer="1"/>
 </signal>
 <signal name="GND">
@@
 <wire x1="93.472" y1="6.985" x2="92.1512" y2="6.985" width="0.254" layer="1"/>
 <wire x1="92.1512" y1="6.985" x2="92.075" y2="6.9088" width="0.254" layer="1"/>
+<contactref element="C802" pad="2"/>
+<contactref element="C803" pad="2"/>
+<wire x1="91.059" y1="6.9088" x2="92.075" y2="6.9088" width="0.254" layer="1"/>
+<via x="105.537" y="4.445" extent="1-16" drill="0.3048"/>
+<wire x1="105.537" y1="4.445" x2="104.4448" y2="4.445" width="0.254" layer="1"/>
 </signal>
 <signal name="PWR_BUT">
@@
 <via x="30.861" y="57.785" extent="1-16" drill="0.3048"/>
 <via x="70.3834" y="19.431" extent="1-16" drill="0.3048"/>
-<wire x1="93.472" y1="8.255" x2="92.075" y2="9.652" width="0.1524" layer="16"/>
-<wire x1="92.075" y1="9.652" x2="76.7334" y2="9.652" width="0.1524" layer="16"/>
-<wire x1="76.7334" y1="9.652" x2="75.7174" y2="10.668" width="0.1524" layer="16"/>
-<wire x1="75.7174" y1="10.668" x2="71.6534" y2="10.668" width="0.1524" layer="16"/>
+<wire x1="93.472" y1="8.255" x2="91.059" y2="10.668" width="0.1524" layer="16"/>
+<wire x1="91.059" y1="10.668" x2="71.6534" y2="10.668" width="0.1524" layer="16"/>
 <wire x1="71.6534" y1="10.668" x2="70.3834" y2="11.938" width="0.1524" layer="16"/>
 <wire x1="70.3834" y1="11.938" x2="70.3834" y2="19.431" width="0.1524" layer="16"/>
@@
 <wire x1="67.2846" y1="57.4294" x2="67.2846" y2="19.431" width="0.1524" layer="1"/>
 <contactref element="D802" pad="2"/>
-<wire x1="95.3262" y1="4.445" x2="96.7994" y2="4.445" width="0.1524" layer="1"/>
-<wire x1="96.7994" y1="4.445" x2="97.4344" y2="3.81" width="0.1524" layer="1"/>
-<wire x1="97.4344" y1="3.81" x2="105.537" y2="3.81" width="0.1524" layer="1"/>
-<wire x1="105.537" y1="3.81" x2="106.172" y2="4.445" width="0.1524" layer="1"/>
-<wire x1="106.172" y1="4.445" x2="106.172" y2="8.1534" width="0.1524" layer="1"/>
+<wire x1="95.3262" y1="4.445" x2="97.2312" y2="4.445" width="0.1524" layer="1"/>
+<wire x1="97.2312" y1="4.445" x2="98.3742" y2="3.302" width="0.1524" layer="1"/>
+<wire x1="98.3742" y1="3.302" x2="105.537" y2="3.302" width="0.1524" layer="1"/>
+<wire x1="105.537" y1="3.302" x2="106.172" y2="3.937" width="0.1524" layer="1"/>
+<wire x1="106.172" y1="3.937" x2="106.172" y2="8.1534" width="0.1524" layer="1"/>
 <wire x1="106.172" y1="8.1534" x2="107.1499" y2="9.1313" width="0.1524" layer="1"/>
 <wire x1="107.1499" y1="9.1313" x2="107.188" y2="9.1313" width="0.1524" layer="1"/>
@@
 <vertex x="71.882" y="12.6746"/>
 </polygon>
-<contactref element="U28" pad="5"/>
 <via x="102.108" y="4.445" extent="1-16" drill="0.3048"/>
+<contactref element="U28" pad="5"/>
+<contactref element="C802" pad="1"/>
+<contactref element="R802" pad="1"/>
+<contactref element="R801" pad="1"/>
+<via x="108.204" y="4.2672" extent="1-16" drill="0.3048"/>
+<wire x1="108.204" y1="4.2672" x2="107.188" y2="4.2672" width="0.254" layer="1"/>
+<wire x1="108.204" y1="4.2672" x2="109.22" y2="4.2672" width="0.254" layer="1"/>
 <wire x1="102.108" y1="4.445" x2="100.2538" y2="4.445" width="0.254" layer="1"/>
+<wire x1="102.108" y1="4.445" x2="103.3272" y2="4.445" width="0.254" layer="1"/>
 </signal>
 <signal name="SYS_VDD_1P8V">

Commit message: Add files via upload
Parts:
- R801, R802: value 500 -> 1K
Changed lines of the file:
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@@
 <element name="X6" library="OSD3358-BSP Ref Design" package="H6-2.54" value="6p-2.54" x="20.32" y="60.96" smashed="yes" rot="R270">
 <attribute name="MPN" value="P125-1106A1BS116A1" x="20.32" y="60.96" size="1.778" layer="27" rot="R270" display="off"/>
+<attribute name="NAME" x="28.067" y="62.357" size="1.016" layer="25" align="top-left"/>
 <attribute name="NAME" x="17.78" y="60.325" size="0.635" layer="33" ratio="10"/>
-<attribute name="NAME" x="28.067" y="62.357" size="1.016" layer="25" align="top-left"/>
 <attribute name="VALUE" x="20.32" y="60.452" size="0.254" layer="27" align="top-center"/>
 </element>
@@
 <attribute name="VALUE" x="106.553" y="8.382" size="0.2" layer="27" rot="R270" align="top-center"/>
 </element>
-<element name="R802" library="OSD3358-SM-RED Platform" package="R0402" value="500" x="107.188" y="4.826" smashed="yes" rot="R90">
+<element name="R802" library="OSD3358-SM-RED Platform" package="R0402" value="1K" x="107.188" y="4.826" smashed="yes" rot="R90">
 <attribute name="NAME" x="106.68" y="3.7084" size="0.8128" layer="25" align="top-right"/>
 <attribute name="VALUE" x="107.6706" y="4.826" size="0.254" layer="27" rot="R90" align="top-center"/>
 </element>
-<element name="R801" library="OSD3358-SM-RED Platform" package="R0402" value="500" x="109.22" y="4.826" smashed="yes" rot="R90">
+<element name="R801" library="OSD3358-SM-RED Platform" package="R0402" value="1K" x="109.22" y="4.826" smashed="yes" rot="R90">
 <attribute name="NAME" x="109.728" y="3.7084" size="0.8128" layer="25" align="top-left"/>
 <attribute name="VALUE" x="109.7026" y="4.826" size="0.254" layer="27" rot="R90" align="top-center"/>
@@
 <element name="J24" library="OSD3358-SM-RED Platform" package="H3-2.54" value="6p-2.54" x="98.425" y="105.41" smashed="yes">
 <attribute name="MPN" value="P125-1106A1BS116A1" x="98.425" y="105.41" size="1.778" layer="27" display="off"/>
+<attribute name="NAME" x="99.06" y="102.87" size="0.635" layer="33" ratio="10" rot="R90"/>
 <attribute name="NAME" x="98.425" y="101.3714" size="0.889" layer="25" ratio="10" align="top-center"/>
-<attribute name="NAME" x="99.06" y="102.87" size="0.635" layer="33" ratio="10" rot="R90"/>
 <attribute name="VALUE" x="98.425" y="104.14" size="0.254" layer="27" align="center"/>
 </element>

Commit message: Add files via upload
Routing:
- net CAN1_TXD: track 192.8 -> 141.5 mm
- net CAN1_RXD: track 172.3 -> 125.0 mm
- net SYS_RESETN: track 198.1 -> 204.7 mm
- net N$110: track 61.5 -> 60.8 mm
- net I2C0_SCL: track 35.0 -> 35.4 mm, vias 1 -> 2

Commit message: Add files via upload
Routing:
- net BO3: track 67.7 -> 68.6 mm
- net 24VDC_AUX: vias 8 -> 6
Changed lines of the file:
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@@
 <element name="X6" library="OSD3358-BSP Ref Design" package="H6-2.54" value="6p-2.54" x="20.32" y="60.96" smashed="yes" rot="R270">
 <attribute name="MPN" value="P125-1106A1BS116A1" x="20.32" y="60.96" size="1.778" layer="27" rot="R270" display="off"/>
-<attribute name="NAME" x="17.78" y="60.325" size="0.635" layer="33" ratio="10"/>
 <attribute name="NAME" x="28.067" y="62.357" size="1.016" layer="25" align="top-left"/>
+<attribute name="NAME" x="17.78" y="60.325" size="0.635" layer="33" ratio="10"/>
 <attribute name="VALUE" x="20.32" y="60.452" size="0.254" layer="27" align="top-center"/>
 </element>
@@
 <element name="J24" library="OSD3358-SM-RED Platform" package="H3-2.54" value="6p-2.54" x="98.425" y="105.41" smashed="yes">
 <attribute name="MPN" value="P125-1106A1BS116A1" x="98.425" y="105.41" size="1.778" layer="27" display="off"/>
-<attribute name="NAME" x="98.425" y="101.3714" size="0.889" layer="25" ratio="10" align="top-center"/>
 <attribute name="NAME" x="99.06" y="102.87" size="0.635" layer="33" ratio="10" rot="R90"/>
+<attribute name="NAME" x="98.425" y="101.3714" size="0.889" layer="25" ratio="10" align="top-center"/>
 <attribute name="VALUE" x="98.425" y="104.14" size="0.254" layer="27" align="center"/>
 </element>
@@
 <contactref element="IC2" pad="9"/>
 <via x="97.536" y="65.532" extent="1-16" drill="0.3048"/>
-<via x="97.536" y="66.548" extent="1-16" drill="0.3048"/>
 <contactref element="C106" pad="1"/>
 <wire x1="88.265" y1="110.109" x2="88.265" y2="106.7338" width="0.508" layer="1"/>
@@
 <vertex x="97.536" y="100.076"/>
 <vertex x="97.282" y="99.822"/>
-<vertex x="97.282" y="68.0212"/>
-<vertex x="97.917" y="67.3862"/>
-<vertex x="98.425" y="67.3862"/>
-<vertex x="99.06" y="66.7512"/>
-<vertex x="99.06" y="64.77"/>
-<vertex x="98.425" y="64.135"/>
-<vertex x="95.5675" y="64.135"/>
-<vertex x="95.25" y="64.4525"/>
+<vertex x="97.282" y="74.93"/>
+<vertex x="97.536" y="74.676"/>
+<vertex x="98.806" y="74.676"/>
+<vertex x="99.06" y="74.422"/>
+<vertex x="99.06" y="64.389"/>
+<vertex x="98.806" y="64.135"/>
+<vertex x="95.504" y="64.135"/>
+<vertex x="95.25" y="64.389"/>
 <vertex x="95.25" y="107.315"/>
 <vertex x="94.615" y="107.95"/>
@@
 <via x="97.536" y="64.516" extent="1-16" drill="0.3048"/>
 <wire x1="113.5507" y1="126.873" x2="92.075" y2="126.873" width="0.2032" layer="1"/>
-<via x="98.552" y="66.548" extent="1-16" drill="0.3048"/>
 <via x="98.552" y="65.532" extent="1-16" drill="0.3048"/>
 <via x="98.552" y="64.516" extent="1-16" drill="0.3048"/>
@@
 <vertex x="99.695" y="61.722"/>
 <vertex x="99.06" y="62.357"/>
-<vertex x="99.06" y="66.7512"/>
-<vertex x="98.425" y="67.3862"/>
-<vertex x="95.885" y="67.3862"/>
-<vertex x="95.25" y="66.7512"/>
+<vertex x="99.06" y="65.786"/>
+<vertex x="98.806" y="66.04"/>
+<vertex x="95.504" y="66.04"/>
+<vertex x="95.25" y="65.786"/>
 <vertex x="95.25" y="32.131"/>
 <vertex x="95.885" y="31.496"/>
@@
 <wire x1="95.25" y1="22.86" x2="95.25" y2="25.9588" width="0.254" layer="1"/>
 <wire x1="95.25" y1="25.9588" x2="104.8512" y2="35.56" width="0.254" layer="1"/>
-<wire x1="95.25" y1="12.7" x2="93.4212" y2="10.8712" width="0.254" layer="1"/>
+<wire x1="95.25" y1="12.7" x2="92.5068" y2="9.9568" width="0.254" layer="1"/>
 <wire x1="78.74" y1="17.972" x2="75.28" y2="21.432" width="0.254" layer="1"/>
-<wire x1="93.4212" y1="10.8712" x2="79.375" y2="10.8712" width="0.254" layer="1"/>
-<wire x1="79.375" y1="10.8712" x2="78.74" y2="11.5062" width="0.254" layer="1"/>
-<wire x1="78.74" y1="11.5062" x2="78.74" y2="17.972" width="0.254" layer="1"/>
+<wire x1="92.5068" y1="9.9568" x2="80.01" y2="9.9568" width="0.254" layer="1"/>
+<wire x1="80.01" y1="9.9568" x2="78.74" y2="11.2268" width="0.254" layer="1"/>
+<wire x1="78.74" y1="11.2268" x2="78.74" y2="17.972" width="0.254" layer="1"/>
 </signal>
 <signal name="BO2">
