File: Version_3.0/Open-Source_Control_V3_R0.brd (EAGLE design)
At the start: 121.9 x 129.5 mm, 350 parts, among them IC10 MCP6002SMT, IC11 MCP6002SMT, IC12 MCP6002SMT, IC14 MCP6002SMT, IC2 ULN2003AD, IC4 74HC165D, IC5 74HC165D, J24 6p-2.54, K1 G5LE-14-CF DC24, K2 G5LE-14-CF DC24, K3 G5LE-14-CF DC24, K4 G5LE-14-CF DC24, Q1 MMBT2907, T4 DA2304-AL, U1 OSD3358-512M-ICB, U16 AT97SC3205T-G3M4400B, U2 TPD4S012_DRY_6_P1_M, U27 LAN8710, U28 TCAN1051HV, U29 MAX3483EESA+T, U4 APX811-31UGSOT, U40 ISO3086TDW, U5 TLVH431, U6 SN74LVC2G241_DCU_8, X1 10118194-0001LF, X10 MC4, X11 MC4, X12 MC4, X2 J0011D01BNL, X21 MC12, X24 MSTBA2, X3 MC4, X31 MC4, X4 CTI-JTAG, X41 MSTBA3, X5 DM3CS-SF, X6 6p-2.54, X7 TH-2X10, X8 TH-2X10, X9 5600200420, Y7 ECS-250-12-30-GN-TR

Commit message: Add files via upload
Parts:
- added C901: 0.1uF, 6.3V, OSD3358-SM-RED Platform:C0402
- added R901, R902: 1.5K, 1% DNI, OSD3358-SM-RED Platform:R0402
Connections:
- net GND: now also C901.2
- net I2C2_SCL: now also R901.1
- net I2C2_SDA: now also R902.1
- net SYS_VDD1_3P3V: now also C901.1, R901.2, R902.2
Routing:
- net SYS_VDD1_3P3V: track 80.8 -> 88.5 mm
- net I2C2_SCL: track 93.4 -> 99.4 mm
- net GND: track 182.6 -> 185.8 mm
- net I2C2_SDA: track 97.2 -> 100.1 mm
Changed lines of the file:
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@@
 <element name="X6" library="OSD3358-BSP Ref Design" package="H6-2.54" value="6p-2.54" x="20.32" y="60.96" smashed="yes" rot="R270">
 <attribute name="MPN" value="P125-1106A1BS116A1" x="20.32" y="60.96" size="1.778" layer="27" rot="R270" display="off"/>
-<attribute name="NAME" x="17.78" y="60.325" size="0.635" layer="33" ratio="10"/>
 <attribute name="NAME" x="28.067" y="62.357" size="1.016" layer="25" align="top-left"/>
+<attribute name="NAME" x="17.78" y="60.325" size="0.635" layer="33" ratio="10"/>
 <attribute name="VALUE" x="20.32" y="60.452" size="0.254" layer="27" align="top-center"/>
 </element>
@@
 <element name="J24" library="OSD3358-SM-RED Platform" package="H3-2.54" value="6p-2.54" x="98.425" y="105.41" smashed="yes">
 <attribute name="MPN" value="P125-1106A1BS116A1" x="98.425" y="105.41" size="1.778" layer="27" display="off"/>
-<attribute name="NAME" x="98.425" y="101.3714" size="0.889" layer="25" ratio="10" align="top-center"/>
 <attribute name="NAME" x="99.06" y="102.87" size="0.635" layer="33" ratio="10" rot="R90"/>
+<attribute name="NAME" x="98.425" y="101.3714" size="0.889" layer="25" ratio="10" align="top-center"/>
 <attribute name="VALUE" x="98.425" y="104.14" size="0.254" layer="27" align="center"/>
 </element>
@@
 <attribute name="VALUE" x="90.551" y="6.35" size="0.254" layer="27" rot="R90" align="bottom-center"/>
 </element>
+<element name="C901" library="OSD3358-SM-RED Platform" package="C0402" value="0.1uF, 6.3V" x="77.47" y="8.636" smashed="yes" rot="R180">
+<attribute name="NAME" x="78.5876" y="8.6868" size="0.8128" layer="25" align="center-left"/>
+<attribute name="VALUE" x="77.47" y="8.1534" size="0.254" layer="27" align="top-center"/>
+</element>
+<element name="R901" library="OSD3358-SM-RED Platform" package="R0402" value="1.5K, 1% DNI" x="77.47" y="9.652" smashed="yes">
+<attribute name="NAME" x="78.613" y="9.652" size="0.8128" layer="25" align="center-left"/>
+<attribute name="VALUE" x="77.47" y="9.1694" size="0.254" layer="27" align="top-center"/>
+</element>
+<element name="R902" library="OSD3358-SM-RED Platform" package="R0402" value="1.5K, 1% DNI" x="77.47" y="7.62" smashed="yes">
+<attribute name="NAME" x="78.5876" y="7.62" size="0.8128" layer="25" align="center-left"/>
+<attribute name="VALUE" x="77.47" y="7.1374" size="0.254" layer="27" align="top-center"/>
+</element>
 </elements>
 <signals>
@@
 <wire x1="79.39" y1="101.2594" x2="79.39" y2="102.235" width="0.8128" layer="1"/>
 <wire x1="78.232" y1="100.1014" x2="79.39" y2="101.2594" width="0.8128" layer="1"/>
-<polygon width="0.254" layer="1" rank="2">
+<polygon width="0.254" layer="1" thermals="no" rank="2">
 <vertex x="79.1972" y="106.68"/>
 <vertex x="61.214" y="106.68"/>
@@
 <wire x1="73.152" y1="120.65" x2="73.152" y2="120.142" width="0.1524" layer="1"/>
 <wire x1="73.152" y1="112.3188" x2="73.152" y2="117.094" width="0.8128" layer="1"/>
-<polygon width="0.254" layer="1">
+<polygon width="0.254" layer="1" thermals="no">
 <vertex x="112.395" y="121.031"/>
 <vertex x="112.395" y="125.73"/>
@@
 <vertex x="109.1438" y="125.984"/>
 <vertex x="108.8898" y="125.73"/>
-<vertex x="108.8898" y="118.2878"/>
-<vertex x="109.7788" y="117.3988"/>
+<vertex x="108.8898" y="117.6528"/>
+<vertex x="109.1438" y="117.3988"/>
 <vertex x="114.1476" y="117.3988"/>
 <vertex x="115.0874" y="118.3386"/>
@@
 <via x="82.55" y="101.219" extent="1-16" drill="0.3048"/>
 <via x="82.55" y="102.235" extent="1-16" drill="0.3048"/>
-<polygon width="0.254" layer="1">
+<polygon width="0.254" layer="1" thermals="no">
 <vertex x="86.106" y="100.5078"/>
 <vertex x="82.55" y="100.5078"/>
@@
 <contactref element="X8" pad="16"/>
 <via x="72.136" y="8.89" extent="1-16" drill="0.3048"/>
-<polygon width="0.254" layer="1">
+<polygon width="0.254" layer="1" thermals="no">
 <vertex x="75.438" y="10.3632"/>
 <vertex x="71.882" y="10.3632"/>
@@
 <vertex x="54.991" y="61.3664"/>
 </polygon>
+<contactref element="C901" pad="2"/>
+<wire x1="76.9112" y1="8.636" x2="76.073" y2="8.636" width="0.1524" layer="1"/>
+<wire x1="76.073" y1="8.636" x2="75.0316" y2="9.6774" width="0.1524" layer="1"/>
+<wire x1="75.0316" y1="9.6774" x2="74.1172" y2="9.6774" width="0.1524" layer="1"/>
 </signal>
 <signal name="PWR_BUT">
@@
 <via x="72.136" y="12.446" extent="1-16" drill="0.3048"/>
 <via x="72.136" y="11.43" extent="1-16" drill="0.3048"/>
-<polygon width="0.254" layer="1">
+<polygon width="0.254" layer="1" thermals="no">
 <vertex x="71.628" y="12.4206"/>
 <vertex x="71.628" y="11.2268"/>
@@
 <wire x1="102.108" y1="4.445" x2="100.2538" y2="4.445" width="0.254" layer="1"/>
 <wire x1="102.108" y1="4.445" x2="103.3272" y2="4.445" width="0.254" layer="1"/>
+<contactref element="C901" pad="1"/>
+<contactref element="R901" pad="2"/>
+<contactref element="R902" pad="2"/>
+<wire x1="78.0288" y1="8.636" x2="77.5208" y2="9.144" width="0.1524" layer="1"/>
+<wire x1="77.5208" y1="9.144" x2="76.3778" y2="9.144" width="0.1524" layer="1"/>
+<wire x1="76.3778" y1="9.144" x2="76.1238" y2="9.398" width="0.1524" layer="1"/>
+<wire x1="76.1238" y1="9.398" x2="76.1238" y2="10.3886" width="0.1524" layer="1"/>
+<wire x1="76.1238" y1="10.3886" x2="74.8538" y2="11.6586" width="0.1524" layer="1"/>
+<wire x1="74.8538" y1="11.6586" x2="74.1172" y2="11.6586" width="0.1524" layer="1"/>
+<wire x1="78.0288" y1="9.652" x2="78.0288" y2="8.636" width="0.1524" layer="1"/>
+<wire x1="78.0288" y1="7.62" x2="78.0288" y2="8.636" width="0.1524" layer="1"/>
 </signal>
 <signal name="SYS_VDD_1P8V">
@@
 <contactref element="L2" pad="1"/>
 <contactref element="D18" pad="C"/>
-<polygon width="0.254" layer="1" rank="2">
+<polygon width="0.254" layer="1" thermals="no" rank="2">
 <vertex x="72.0598" y="114.4524"/>
 <vertex x="72.0598" y="109.7534"/>
@@
 <via x="68.58" y="112.776" extent="1-16" drill="0.3048"/>
 <via x="68.58" y="110.744" extent="1-16" drill="0.3048"/>
-<polygon width="0.254" layer="1">
+<polygon width="0.254" layer="1" thermals="no">
 <vertex x="65.913" y="110.4646"/>
 <vertex x="70.104" y="110.4646"/>
 <vertex x="70.358" y="110.7186"/>
-<vertex x="70.358" y="113.411"/>
+<vertex x="70.358" y="113.157"/>
+<vertex x="70.104" y="113.411"/>
 <vertex x="65.913" y="113.411"/>
 <vertex x="65.659" y="113.157"/>
@@
 <via x="66.548" y="112.776" extent="1-16" drill="0.3048"/>
 <contactref element="J24" pad="2"/>
-<polygon width="0.254" layer="1" isolate="0.3048">
+<polygon width="0.254" layer="1" isolate="0.3048" thermals="no">
 <vertex x="104.5972" y="103.8352"/>
 <vertex x="104.5972" y="107.4166"/>
@@
 <contactref element="D3" pad="A"/>
 <contactref element="F1" pad="P$2"/>
-<polygon width="0.254" layer="1">
+<polygon width="0.254" layer="1" thermals="no">
 <vertex x="108.712" y="107.696"/>
 <vertex x="108.9406" y="107.696"/>
@@
 <contactref element="F1" pad="P$1"/>
 <contactref element="X3" pad="4"/>
-<polygon width="0.254" layer="16">
+<polygon width="0.254" layer="16" thermals="no">
 <vertex x="104.5972" y="107.9246"/>
 <vertex x="104.5972" y="110.363"/>
 <vertex x="105.2322" y="110.998"/>
-<vertex x="114.3" y="110.998"/>
-<vertex x="115.57" y="112.268"/>
-<vertex x="115.57" y="115.062"/>
-<vertex x="113.792" y="116.84"/>
+<vertex x="114.935" y="110.998"/>
+<vertex x="115.57" y="111.633"/>
+<vertex x="115.57" y="116.205"/>
+<vertex x="114.935" y="116.84"/>
 <vertex x="103.378" y="116.84"/>
 <vertex x="103.124" y="116.586"/>
@@
 <vertex x="104.3432" y="107.6706"/>
 </polygon>
-<polygon width="0.254" layer="15" isolate="0.254" rank="2">
-<vertex x="114.3" y="110.998"/>
+<polygon width="0.254" layer="15" isolate="0.254" thermals="no" rank="2">
+<vertex x="115.57" y="116.205"/>
+<vertex x="115.57" y="111.633"/>
+<vertex x="114.935" y="110.998"/>
 <vertex x="104.394" y="110.998"/>
 <vertex x="103.124" y="112.268"/>
@@
 <vertex x="107.188" y="117.475"/>
 <vertex x="107.823" y="116.84"/>
-<vertex x="113.792" y="116.84"/>
-<vertex x="115.57" y="115.062"/>
-<vertex x="115.57" y="112.268"/>
+<vertex x="114.935" y="116.84"/>
 </polygon>
 </signal>
@@
 <wire x1="65.913" y1="15.0114" x2="67.2592" y2="13.6652" width="0.1524" layer="1"/>
 <wire x1="67.2592" y1="13.6652" x2="74.1172" y2="13.6652" width="0.1524" layer="1"/>
+<contactref element="R901" pad="1"/>
+<wire x1="76.9112" y1="9.652" x2="76.9112" y2="11.0998" width="0.1524" layer="1"/>
+<wire x1="76.2" y1="11.811" x2="76.2" y2="13.0302" width="0.1524" layer="1"/>
+<wire x1="76.2" y1="13.0302" x2="75.565" y2="13.6652" width="0.1524" layer="1"/>
+<wire x1="75.565" y1="13.6652" x2="74.1172" y2="13.6652" width="0.1524" layer="1"/>
+<wire x1="76.9112" y1="11.0998" x2="76.2" y2="11.811" width="0.1524" layer="1"/>
 </signal>
 <signal name="I2C2_SDA">
@@
 <wire x1="65.3796" y1="8.9408" x2="66.6496" y2="7.6708" width="0.1524" layer="1"/>
 <wire x1="66.6496" y1="7.6708" x2="74.1172" y2="7.6708" width="0.1524" layer="1"/>
+<contactref element="R902" pad="1"/>
+<wire x1="74.1172" y1="7.6708" x2="76.8604" y2="7.6708" width="0.1524" layer="1"/>
+<wire x1="76.8604" y1="7.6708" x2="76.9112" y2="7.62" width="0.1524" layer="1"/>
 </signal>
 <signal name="485_RXD">

Commit message: Add files via upload
Connections:
- net 41_A: now also X41.2; no longer X41.1
- net 41_B: now also X41.1; no longer X41.2
Routing:
- net 41_B: track 6.37 -> 9.96 mm
- net 41_A: track 6.37 -> 9.96 mm
Changed lines of the file:
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@@
 </signal>
 <signal name="ISO_GND">
-<contactref element="X41" pad="3"/>
 <contactref element="U40" pad="15"/>
 <contactref element="U40" pad="9"/>
@@
 </polygon>
 <contactref element="C406" pad="-"/>
+<contactref element="X41" pad="3"/>
 </signal>
 <signal name="ISO_VIN">
@@
 <signal name="41_A">
 <contactref element="F401" pad="1"/>
-<contactref element="X41" pad="1"/>
 <contactref element="GDT1" pad="2"/>
-<wire x1="10.16" y1="123.19" x2="13.1572" y2="123.19" width="1.27" layer="16"/>
-<wire x1="14.4272" y1="124.46" x2="16.002" y2="124.46" width="1.27" layer="16"/>
-<wire x1="13.1572" y1="123.19" x2="14.4272" y2="124.46" width="1.27" layer="16"/>
 <polygon width="0.254" layer="1" rank="3">
 <vertex x="23.3426" y="123.698"/>
@@
 <vertex x="23.5966" y="123.952"/>
 </polygon>
+<contactref element="X41" pad="2"/>
+<wire x1="10.16" y1="118.11" x2="10.16" y2="119.38" width="1.27" layer="1"/>
+<wire x1="10.16" y1="119.38" x2="11.43" y2="120.65" width="1.27" layer="1"/>
+<wire x1="11.43" y1="120.65" x2="12.446" y2="120.65" width="1.27" layer="1"/>
+<wire x1="12.446" y1="120.65" x2="13.716" y2="121.92" width="1.27" layer="1"/>
+<wire x1="13.716" y1="121.92" x2="13.716" y2="123.19" width="1.27" layer="1"/>
+<wire x1="13.716" y1="123.19" x2="14.986" y2="124.46" width="1.27" layer="1"/>
+<wire x1="14.986" y1="124.46" x2="16.002" y2="124.46" width="1.27" layer="1"/>
 </signal>
 <signal name="41_B">
@@
 </polygon>
 <contactref element="F402" pad="1"/>
-<contactref element="X41" pad="2"/>
 <contactref element="GDT1" pad="1"/>
-<wire x1="10.16" y1="118.11" x2="13.1572" y2="118.11" width="1.27" layer="16"/>
-<wire x1="14.4272" y1="116.84" x2="16.002" y2="116.84" width="1.27" layer="16"/>
-<wire x1="13.1572" y1="118.11" x2="14.4272" y2="116.84" width="1.27" layer="16"/>
+<contactref element="X41" pad="1"/>
+<wire x1="10.16" y1="123.19" x2="10.16" y2="121.92" width="1.27" layer="16"/>
+<wire x1="10.16" y1="121.92" x2="11.43" y2="120.65" width="1.27" layer="16"/>
+<wire x1="11.43" y1="120.65" x2="12.446" y2="120.65" width="1.27" layer="16"/>
+<wire x1="12.446" y1="120.65" x2="13.716" y2="119.38" width="1.27" layer="16"/>
+<wire x1="13.716" y1="119.38" x2="13.716" y2="118.11" width="1.27" layer="16"/>
+<wire x1="13.716" y1="118.11" x2="14.986" y2="116.84" width="1.27" layer="16"/>
+<wire x1="14.986" y1="116.84" x2="16.002" y2="116.84" width="1.27" layer="16"/>
 </signal>
 <signal name="24LIN_IN">

Commit message: Add files via upload
Parts:
- turned D301 to 90 degrees
- turned D302 to 90 degrees
- turned D401 to 90 degrees
- turned D402 to 90 degrees
- turned R301 to 270 degrees
- turned R302 to 270 degrees
- turned R401 to 270 degrees
- turned R402 to 270 degrees
Connections:
- removed net N$20: D302.2, R302.1
- removed net N$52: D401.2, R401.1
- removed net N$86: D402.2, R402.1
- new net N$16: D402.1, R402.2
- new net N$17: D401.1, R401.2
- new net N$18: D301.1, R301.2
- net 485_RXD: now also D402.2; no longer D402.1
- net 485_TXD: now also D401.2; no longer D401.1
- net GND: no longer R301.2, R302.2, R401.2, R402.2
- net N$19: now also D302.1, R302.2; no longer D301.2, R301.1
- net SYS_VDD1_3P3V: now also R301.1, R302.1, R401.1, R402.1
- net UART2_RXD: now also D302.2; no longer D302.1
- net UART2_TXD: now also D301.2; no longer D301.1
Routing:
- net N$20: track 5.20 -> 0.00 mm
- net SYS_VDD1_3P3V: track 88.5 -> 93.7 mm, vias 44 -> 47
- net N$19: track 1.55 -> 5.52 mm
- net GND: track 185.8 -> 182.2 mm, vias 200 -> 198
- net N$18: track 0.00 -> 1.55 mm
- net N$86: track 1.35 -> 0.00 mm
- net N$52: track 1.35 -> 0.00 mm
- net N$17: track 0.00 -> 1.35 mm
- net N$16: track 0.00 -> 1.35 mm

Commit message: Add files via upload
Connections:
- net 41_A: now also F402.1, GDT1.1; no longer F401.1, GDT1.2
- net 41_B: now also F401.1, GDT1.2; no longer F402.1, GDT1.1
- net ISO_485_A: now also D405.2, F402.3; no longer D405.1, F401.3
- net ISO_485_B: now also D405.1, F401.3; no longer D405.2, F402.3
Routing:
- net ISO_485_A: track 17.7 -> 23.0 mm
- net 41_B: track 9.96 -> 6.37 mm
- net 41_A: track 9.96 -> 6.37 mm
- net ISO_485_B: track 15.6 -> 12.9 mm
Changed lines of the file:
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@@
 </polygon>
 </signal>
-<signal name="ISO_485_B">
-<contactref element="U40" pad="12"/>
-<contactref element="U40" pad="13"/>
-<contactref element="D405" pad="2"/>
-<wire x1="46.355" y1="118.8212" x2="45.085" y2="118.8212" width="0.508" layer="1"/>
-<contactref element="F402" pad="3"/>
-<wire x1="35.703" y1="114.239" x2="44.8716" y2="114.239" width="0.508" layer="1"/>
-<wire x1="46.355" y1="115.7224" x2="46.355" y2="118.8212" width="0.508" layer="1"/>
-<wire x1="44.8716" y1="114.239" x2="46.355" y2="115.7224" width="0.508" layer="1"/>
+<signal name="ISO_485_A">
 <polygon width="0.254" layer="1">
 <vertex x="17.5514" y="115.0366"/>
@@
 <vertex x="17.8054" y="115.2906"/>
 </polygon>
-</signal>
-<signal name="ISO_485_A">
+<contactref element="U40" pad="11"/>
+<contactref element="F402" pad="3"/>
 <contactref element="U40" pad="14"/>
-<contactref element="U40" pad="11"/>
-<contactref element="D405" pad="1"/>
+<contactref element="D405" pad="2"/>
 <wire x1="43.815" y1="118.8212" x2="43.815" y2="120.269" width="0.508" layer="1"/>
 <wire x1="43.815" y1="120.269" x2="44.45" y2="120.904" width="0.508" layer="1"/>
@@
 <wire x1="46.99" y1="120.904" x2="47.625" y2="120.269" width="0.508" layer="1"/>
 <wire x1="47.625" y1="120.269" x2="47.625" y2="118.8212" width="0.508" layer="1"/>
-<contactref element="F401" pad="3"/>
-<wire x1="35.703" y1="116.139" x2="43.18" y2="116.139" width="0.508" layer="1"/>
-<wire x1="43.18" y1="116.139" x2="43.815" y2="116.774" width="0.508" layer="1"/>
-<wire x1="43.815" y1="116.774" x2="43.815" y2="118.8212" width="0.508" layer="1"/>
-<polygon width="0.254" layer="1">
-<vertex x="23.3426" y="122.682"/>
-<vertex x="19.3294" y="122.682"/>
-<vertex x="19.0754" y="122.428"/>
-<vertex x="19.0754" y="119.7864"/>
-<vertex x="20.2438" y="118.618"/>
-<vertex x="20.2438" y="116.1034"/>
-<vertex x="20.8788" y="115.4684"/>
-<vertex x="36.1188" y="115.4684"/>
-<vertex x="36.1188" y="116.586"/>
-<vertex x="24.2316" y="116.586"/>
-<vertex x="23.5966" y="117.221"/>
-<vertex x="23.5966" y="122.428"/>
-</polygon>
+<wire x1="47.625" y1="118.8212" x2="47.625" y2="115.5954" width="0.508" layer="1"/>
+<wire x1="35.703" y1="114.239" x2="35.769" y2="114.173" width="0.508" layer="1"/>
+<wire x1="46.2026" y1="114.173" x2="35.769" y2="114.173" width="0.508" layer="1"/>
+<wire x1="47.625" y1="115.5954" x2="46.2026" y2="114.173" width="0.508" layer="1"/>
 </signal>
 <signal name="ISO_VCC">
@@
 <wire x1="88.138" y1="74.295" x2="89.6366" y2="74.295" width="0.1524" layer="1"/>
 </signal>
-<signal name="41_A">
+<signal name="41_B">
 <contactref element="F401" pad="1"/>
 <contactref element="GDT1" pad="2"/>
@@
 <vertex x="23.5966" y="123.952"/>
 </polygon>
-<contactref element="X41" pad="2"/>
-<wire x1="10.16" y1="118.11" x2="10.16" y2="119.38" width="1.27" layer="1"/>
-<wire x1="10.16" y1="119.38" x2="11.43" y2="120.65" width="1.27" layer="1"/>
-<wire x1="11.43" y1="120.65" x2="12.446" y2="120.65" width="1.27" layer="1"/>
-<wire x1="12.446" y1="120.65" x2="13.716" y2="121.92" width="1.27" layer="1"/>
-<wire x1="13.716" y1="121.92" x2="13.716" y2="123.19" width="1.27" layer="1"/>
-<wire x1="13.716" y1="123.19" x2="14.986" y2="124.46" width="1.27" layer="1"/>
-<wire x1="14.986" y1="124.46" x2="16.002" y2="124.46" width="1.27" layer="1"/>
-</signal>
-<signal name="41_B">
+<contactref element="X41" pad="1"/>
+<wire x1="10.16" y1="123.19" x2="13.462" y2="123.19" width="1.524" layer="16"/>
+<wire x1="14.732" y1="124.46" x2="16.002" y2="124.46" width="1.524" layer="16"/>
+<wire x1="14.732" y1="124.46" x2="13.462" y2="123.19" width="1.524" layer="16"/>
+</signal>
+<signal name="41_A">
 <polygon width="0.254" layer="1">
 <vertex x="16.51" y="110.998"/>
@@
 <contactref element="F402" pad="1"/>
 <contactref element="GDT1" pad="1"/>
-<contactref element="X41" pad="1"/>
-<wire x1="10.16" y1="123.19" x2="10.16" y2="121.92" width="1.27" layer="16"/>
-<wire x1="10.16" y1="121.92" x2="11.43" y2="120.65" width="1.27" layer="16"/>
-<wire x1="11.43" y1="120.65" x2="12.446" y2="120.65" width="1.27" layer="16"/>
-<wire x1="12.446" y1="120.65" x2="13.716" y2="119.38" width="1.27" layer="16"/>
-<wire x1="13.716" y1="119.38" x2="13.716" y2="118.11" width="1.27" layer="16"/>
-<wire x1="13.716" y1="118.11" x2="14.986" y2="116.84" width="1.27" layer="16"/>
-<wire x1="14.986" y1="116.84" x2="16.002" y2="116.84" width="1.27" layer="16"/>
+<contactref element="X41" pad="2"/>
+<wire x1="10.16" y1="118.11" x2="13.462" y2="118.11" width="1.524" layer="16"/>
+<wire x1="14.732" y1="116.84" x2="13.462" y2="118.11" width="1.524" layer="16"/>
+<wire x1="14.732" y1="116.84" x2="16.002" y2="116.84" width="1.524" layer="16"/>
 </signal>
 <signal name="24LIN_IN">
@@
 <wire x1="16.9164" y1="68.834" x2="19.9263" y2="68.834" width="0.1524" layer="1"/>
 </signal>
+<signal name="ISO_485_B">
+<contactref element="U40" pad="13"/>
+<contactref element="F401" pad="3"/>
+<contactref element="U40" pad="12"/>
+<contactref element="D405" pad="1"/>
+<polygon width="0.254" layer="1">
+<vertex x="23.3426" y="122.682"/>
+<vertex x="19.3294" y="122.682"/>
+<vertex x="19.0754" y="122.428"/>
+<vertex x="19.0754" y="119.7864"/>
+<vertex x="20.2438" y="118.618"/>
+<vertex x="20.2438" y="116.1034"/>
+<vertex x="20.8788" y="115.4684"/>
+<vertex x="36.1188" y="115.4684"/>
+<vertex x="36.1188" y="116.586"/>
+<vertex x="24.2316" y="116.586"/>
+<vertex x="23.5966" y="117.221"/>
+<vertex x="23.5966" y="122.428"/>
+</polygon>
+<wire x1="45.085" y1="118.8212" x2="46.355" y2="118.8212" width="0.508" layer="1"/>
+<wire x1="45.085" y1="118.8212" x2="45.085" y2="116.84" width="0.508" layer="1"/>
+<wire x1="45.085" y1="116.84" x2="44.45" y2="116.205" width="0.508" layer="1"/>
+<wire x1="44.45" y1="116.205" x2="35.769" y2="116.205" width="0.508" layer="1"/>
+<wire x1="35.769" y1="116.205" x2="35.703" y2="116.139" width="0.508" layer="1"/>
+</signal>
 </signals>

Commit message: Add files via upload
Parts:
- R169, R170: value 1.5K, 1% -> 10K, 1%
Changed lines of the file:
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@@
 <attribute name="VALUE" x="65.8114" y="68.1736" size="0.254" layer="27" align="top-center"/>
 </element>
-<element name="R169" library="OSD3358-SM-RED Platform" package="R0402" value="1.5K, 1%" x="68.0466" y="66.548" smashed="yes" rot="R180">
+<element name="R169" library="OSD3358-SM-RED Platform" package="R0402" value="10K, 1%" x="68.0466" y="66.548" smashed="yes" rot="R180">
 <attribute name="NAME" x="69.1642" y="66.548" size="0.8128" layer="25"/>
 <attribute name="VALUE" x="68.0466" y="66.1162" size="0.254" layer="27" align="top-center"/>
 </element>
-<element name="R170" library="OSD3358-SM-RED Platform" package="R0402" value="1.5K, 1%" x="68.0466" y="67.564" smashed="yes" rot="R180">
+<element name="R170" library="OSD3358-SM-RED Platform" package="R0402" value="10K, 1%" x="68.0466" y="67.564" smashed="yes" rot="R180">
 <attribute name="NAME" x="69.1642" y="67.564" size="0.8128" layer="25"/>
 <attribute name="VALUE" x="68.0466" y="67.1322" size="0.254" layer="27" align="top-center"/>

Commit message: Add files via upload
Parts:
- moved R902 0.51 mm to (77.5, 7.11)
- moved C901 0.51 mm to (77.5, 8.13)
- moved R901 0.51 mm to (77.5, 9.14)
- moved X9 0.51 mm to (65.5, 10.2)
Routing:
- net I2C2_SDA: track 100.1 -> 100.6 mm

Commit message: Add files via upload
Parts:
- removed MGT1, MGT2, MGT3, MGT4: MOUNTING_HOLE, OSD3358-BSP Ref Design:MOUNTING_HOLE
- added H4, MTG1, MTG2, MTG3: MOUNT-PAD-ROUND3.6, holes:3,6-PAD
- moved R211 1.65 mm to (38.7, 52.5)
- moved R221 1.65 mm to (38.7, 44.8)
- moved R231 1.65 mm to (38.7, 35.4)
- moved R251 1.65 mm to (38.7, 18.4)
- moved R261 1.65 mm to (38.7, 10.8)
- moved R241 1.65 mm to (38.7, 27.8)
- moved C111 1.27 mm to (31.8, 54.5)
- moved C121 1.27 mm to (31.8, 46.9)
- moved C131 1.27 mm to (31.8, 37.5)
- moved C141 1.27 mm to (31.8, 29.8)
- moved C151 1.27 mm to (31.8, 20.4)
- moved C161 1.27 mm to (31.8, 12.8)
- moved D405 0.89 mm to (36.7, 114.3)
- moved VREG4 0.63 mm to (36.7, 119.1)
- moved C403 0.51 mm to (36.2, 116.8)
Connections:
- net CGND: now also H4.B3,6, MTG1.B3,6, MTG2.B3,6, MTG3.B3,6; no longer MGT1.P$1, MGT2.P$1, MGT3.P$1, MGT4.P$1
Routing:
- net GND: track 182.2 -> 196.4 mm
- net N$61: track 17.3 -> 19.8 mm
- net N$45: track 17.3 -> 19.8 mm
- net N$68: track 17.3 -> 19.8 mm
- net N$44: track 17.3 -> 19.8 mm
- net N$38: track 17.3 -> 19.8 mm
- net N$75: track 17.3 -> 19.8 mm
- net 1P8V_REF_1: track 103.2 -> 100.7 mm
- net 1P8V_REF_2: track 51.6 -> 50.4 mm
- net ISO_485_B: track 12.9 -> 13.9 mm
- net ISO_485_A: track 23.0 -> 23.9 mm
- net CAN1_RXD: track 125.0 -> 124.2 mm
