File: Version_3.0/Open-Source_Control_V3_R0.sch (EAGLE design)
At the start: 347 parts, among them IC10 MCP6002SMT, IC11 MCP6002SMT, IC12 MCP6002SMT, IC14 MCP6002SMT, IC2 ULN2003AD, IC4 74HC165D, IC5 74HC165D, J24 6p-2.54, K1 G5LE-14-CF DC24, K2 G5LE-14-CF DC24, K3 G5LE-14-CF DC24, K4 G5LE-14-CF DC24, Q1 MMBT2907, T4 DA2304-AL, U1 OSD3358-512M-ICB, U16 AT97SC3205T-G3M4400B, U2 TPD4S012_DRY_6_P1_M, U27 LAN8710, U28 TCAN1051HV, U29 MAX3483EESA+T, U4 APX811-31UGSOT, U40 ISO3086TDW, U5 TLVH431, U6 SN74LVC2G241_DCU_8, X1 10118194-0001LF, X10 MC4, X11 MC4, X12 MC4, X13 TH-2X10, X2 J0011D01BNL, X21 MC12, X24 MSTBA2, X3 MC4, X4 CTI-JTAG, X41 MSTBA3, X5 DM3CS-SF, X6 6p-2.54, X7 TH-2X10, X8 MC4, X9 5600200420, Y7 ECS-250-12-30-GN-TR

Commit message: Add files via upload
Parts:
- removed X13: TH-2X10, OSD3358-SM-RED Platform:TH-2X10
- added X31: MC4, con-phoenix-381_l:MC4
- X8: value MC4 -> TH-2X10; device con-phoenix-381_l:MC4 -> OSD3358-SM-RED Platform:TH-2X10
Connections:
- net 24VDC_AUX: now also X31.4.SK, X8.12, X8.19, X8.20; no longer X13.12, X13.19, X13.20, X8.4.SK
- net BO1: now also X8.10; no longer X13.10
- net BO1_AUTO: now also X8.9; no longer X13.9
- net BO2: now also X8.8; no longer X13.8
- net BO2_AUTO: now also X8.7; no longer X13.7
- net BO3: now also X8.6; no longer X13.6
- net BO3_AUTO: now also X8.5; no longer X13.5
- net BO4: now also X8.4; no longer X13.4
- net BO4_AUTO: now also X8.3; no longer X13.3
- net BO5_AUTO: now also X8.1; no longer X13.1
- net CAN_H: now also X31.3.SK; no longer X8.3.SK
- net CAN_L: now also X31.2.SK; no longer X8.2.SK
- net EHRPWM1A: now also X8.15; no longer X13.15
- net EHRPWM2A: now also X8.13; no longer X13.13
- net EHRPWM2B: now also X8.14; no longer X13.14
- net GND: now also X31.1.SK, X8.16, X8.2; no longer X13.16, X13.2, X8.1.SK
- net PMIC_NRESET: now also X8.11; no longer X13.11
Changed lines of the file:
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@@
 <part name="C100" library="OSD3358-SM-RED Platform" deviceset="UHE1H102MHD6" device="" value="1000uF, 50V, UHE1H102MHD6"/>
 <part name="R35" library="GHI-BasicComponents" deviceset="RESISTOR.NETWORK-(4)" device="" value="1K"/>
-<part name="X8" library="con-phoenix-381_l" deviceset="MC4" device=""/>
+<part name="X31" library="con-phoenix-381_l" deviceset="MC4" device=""/>
 <part name="U29" library="OSD3358-SM-RED Platform" deviceset="MAX3483EESA+T" device=""/>
 <part name="SUPPLY4" library="OSD3358-SM-RED Platform" deviceset="SYS_VDD1_3P3V" device=""/>
@@
 <part name="SUPPLY35" library="OSD3358-SM-RED Platform" deviceset="SYS_VDD1_3P3V" device=""/>
 <part name="GND35" library="OSD3358-SM-RED Platform" deviceset="GND" device=""/>
-<part name="X13" library="OSD3358-SM-RED Platform" deviceset="TH-2X10" device=""/>
+<part name="X8" library="OSD3358-SM-RED Platform" deviceset="TH-2X10" device=""/>
 </parts>
 <sheets>
@@
 <attribute name="VALUE" x="485.14" y="322.58" size="1.778" layer="96" align="top-right"/>
 </instance>
-<instance part="X8" gate=".1" x="335.28" y="1013.46" smashed="yes" rot="MR0">
+<instance part="X31" gate=".1" x="335.28" y="1013.46" smashed="yes" rot="MR0">
 <attribute name="NAME" x="342.9" y="1015.365" size="1.524" layer="95" rot="MR0"/>
 </instance>
-<instance part="X8" gate=".2" x="998.22" y="683.26" smashed="yes" rot="MR0">
+<instance part="X31" gate=".2" x="998.22" y="683.26" smashed="yes" rot="MR0">
 <attribute name="NAME" x="1005.84" y="685.165" size="1.524" layer="95" rot="MR0"/>
 </instance>
-<instance part="X8" gate=".3" x="998.22" y="693.42" smashed="yes" rot="MR0">
+<instance part="X31" gate=".3" x="998.22" y="693.42" smashed="yes" rot="MR0">
 <attribute name="NAME" x="1005.84" y="695.325" size="1.524" layer="95" rot="MR0"/>
 </instance>
-<instance part="X8" gate=".4" x="335.28" y="1021.08" smashed="yes" rot="MR0">
+<instance part="X31" gate=".4" x="335.28" y="1021.08" smashed="yes" rot="MR0">
 <attribute name="NAME" x="342.9" y="1022.985" size="1.524" layer="95" rot="MR0"/>
 </instance>
@@
 <attribute name="VALUE" x="1059.18" y="807.72" size="1.778" layer="96"/>
 </instance>
-<instance part="X13" gate="G$1" x="1087.12" y="779.78" smashed="yes">
+<instance part="X8" gate="G$1" x="1087.12" y="779.78" smashed="yes">
 <attribute name="NAME" x="1079.5" y="792.48" size="1.778" layer="95" ratio="10"/>
 <attribute name="VALUE" x="1079.5" y="762" size="1.778" layer="96" ratio="10"/>
@@
 <pinref part="GND23" gate="1" pin="GND"/>
 <wire x1="325.12" y1="1013.46" x2="325.12" y2="1005.84" width="0.1524" layer="91"/>
-<pinref part="X8" gate=".1" pin="SK"/>
+<pinref part="X31" gate=".1" pin="SK"/>
 <wire x1="335.28" y1="1013.46" x2="325.12" y2="1013.46" width="0.1524" layer="91"/>
 </segment>
@@
 <pinref part="GND31" gate="1" pin="GND"/>
 <wire x1="1145.54" y1="767.08" x2="1145.54" y2="772.16" width="0.1524" layer="91"/>
-<pinref part="X13" gate="G$1" pin="2"/>
+<pinref part="X8" gate="G$1" pin="2"/>
 <wire x1="1145.54" y1="772.16" x2="1145.54" y2="789.94" width="0.1524" layer="91"/>
 <wire x1="1099.82" y1="789.94" x2="1145.54" y2="789.94" width="0.1524" layer="91"/>
-<pinref part="X13" gate="G$1" pin="16"/>
+<pinref part="X8" gate="G$1" pin="16"/>
 <wire x1="1099.82" y1="772.16" x2="1145.54" y2="772.16" width="0.1524" layer="91"/>
 <junction x="1145.54" y="772.16"/>
@@
 </segment>
 <segment>
-<pinref part="X13" gate="G$1" pin="14"/>
+<pinref part="X8" gate="G$1" pin="14"/>
 <wire x1="1099.82" y1="774.7" x2="1137.92" y2="774.7" width="0.1524" layer="91"/>
 <label x="1137.92" y="774.7" size="1.778" layer="95" align="bottom-right"/>
@@
 </segment>
 <segment>
-<pinref part="X13" gate="G$1" pin="13"/>
+<pinref part="X8" gate="G$1" pin="13"/>
 <wire x1="1074.42" y1="774.7" x2="1036.32" y2="774.7" width="0.1524" layer="91"/>
 <label x="1036.32" y="774.7" size="1.778" layer="95"/>
@@
 </segment>
 <segment>
-<pinref part="X13" gate="G$1" pin="15"/>
+<pinref part="X8" gate="G$1" pin="15"/>
 <wire x1="1074.42" y1="772.16" x2="1036.32" y2="772.16" width="0.1524" layer="91"/>
 <label x="1036.32" y="772.16" size="1.778" layer="95"/>
@@
 <junction x="256.54" y="1033.78"/>
 <junction x="325.12" y="1033.78"/>
-<pinref part="X8" gate=".4" pin="SK"/>
+<pinref part="X31" gate=".4" pin="SK"/>
 <wire x1="325.12" y1="1021.08" x2="325.12" y2="1033.78" width="0.1524" layer="91"/>
 <wire x1="335.28" y1="1021.08" x2="325.12" y2="1021.08" width="0.1524" layer="91"/>
@@
 </segment>
 <segment>
-<pinref part="X13" gate="G$1" pin="12"/>
+<pinref part="X8" gate="G$1" pin="12"/>
 <wire x1="1099.82" y1="777.24" x2="1137.92" y2="777.24" width="0.1524" layer="91"/>
 <label x="1137.92" y="777.24" size="1.778" layer="95" align="bottom-right"/>
 </segment>
 <segment>
-<pinref part="X13" gate="G$1" pin="19"/>
+<pinref part="X8" gate="G$1" pin="19"/>
 <wire x1="1074.42" y1="767.08" x2="1036.32" y2="767.08" width="0.1524" layer="91"/>
 <label x="1036.32" y="767.08" size="1.778" layer="95"/>
 </segment>
 <segment>
-<pinref part="X13" gate="G$1" pin="20"/>
+<pinref part="X8" gate="G$1" pin="20"/>
 <wire x1="1099.82" y1="767.08" x2="1137.92" y2="767.08" width="0.1524" layer="91"/>
 <label x="1137.92" y="767.08" size="1.778" layer="95" align="bottom-right"/>
@@
 <pinref part="D805" gate="G$1" pin="2"/>
 <wire x1="980.44" y1="680.72" x2="980.44" y2="693.42" width="0.1524" layer="91"/>
-<pinref part="X8" gate=".3" pin="SK"/>
+<pinref part="X31" gate=".3" pin="SK"/>
 <wire x1="980.44" y1="693.42" x2="998.22" y2="693.42" width="0.1524" layer="91"/>
 <junction x="980.44" y="693.42"/>
@@
 <pinref part="D805" gate="G$1" pin="1"/>
 <wire x1="990.6" y1="680.72" x2="990.6" y2="683.26" width="0.1524" layer="91"/>
-<pinref part="X8" gate=".2" pin="SK"/>
+<pinref part="X31" gate=".2" pin="SK"/>
 <wire x1="990.6" y1="683.26" x2="998.22" y2="683.26" width="0.1524" layer="91"/>
 <junction x="990.6" y="683.26"/>
@@
 </segment>
 <segment>
-<pinref part="X13" gate="G$1" pin="9"/>
+<pinref part="X8" gate="G$1" pin="9"/>
 <wire x1="1074.42" y1="779.78" x2="1036.32" y2="779.78" width="0.1524" layer="91"/>
 <label x="1036.32" y="779.78" size="1.778" layer="95"/>
@@
 </segment>
 <segment>
-<pinref part="X13" gate="G$1" pin="7"/>
+<pinref part="X8" gate="G$1" pin="7"/>
 <wire x1="1074.42" y1="782.32" x2="1036.32" y2="782.32" width="0.1524" layer="91"/>
 <label x="1036.32" y="782.32" size="1.778" layer="95"/>
@@
 </segment>
 <segment>
-<pinref part="X13" gate="G$1" pin="5"/>
+<pinref part="X8" gate="G$1" pin="5"/>
 <wire x1="1074.42" y1="784.86" x2="1036.32" y2="784.86" width="0.1524" layer="91"/>
 <label x="1036.32" y="784.86" size="1.778" layer="95"/>
@@
 </segment>
 <segment>
-<pinref part="X13" gate="G$1" pin="3"/>
+<pinref part="X8" gate="G$1" pin="3"/>
 <wire x1="1074.42" y1="787.4" x2="1036.32" y2="787.4" width="0.1524" layer="91"/>
 <label x="1036.32" y="787.4" size="1.778" layer="95"/>
@@
 </segment>
 <segment>
-<pinref part="X13" gate="G$1" pin="1"/>
+<pinref part="X8" gate="G$1" pin="1"/>
 <wire x1="1074.42" y1="789.94" x2="1036.32" y2="789.94" width="0.1524" layer="91"/>
 <label x="1036.32" y="789.94" size="1.778" layer="95"/>
@@
 </segment>
 <segment>
-<pinref part="X13" gate="G$1" pin="11"/>
+<pinref part="X8" gate="G$1" pin="11"/>
 <wire x1="1074.42" y1="777.24" x2="1036.32" y2="777.24" width="0.1524" layer="91"/>
 <label x="1036.32" y="777.24" size="1.778" layer="95"/>
@@
 <net name="BO4" class="0">
 <segment>
-<pinref part="X13" gate="G$1" pin="4"/>
+<pinref part="X8" gate="G$1" pin="4"/>
 <wire x1="1099.82" y1="787.4" x2="1137.92" y2="787.4" width="0.1524" layer="91"/>
 <label x="1137.92" y="787.4" size="1.778" layer="95" align="bottom-right"/>
@@
 <net name="BO3" class="0">
 <segment>
-<pinref part="X13" gate="G$1" pin="6"/>
+<pinref part="X8" gate="G$1" pin="6"/>
 <wire x1="1099.82" y1="784.86" x2="1137.92" y2="784.86" width="0.1524" layer="91"/>
 <label x="1137.92" y="784.86" size="1.778" layer="95" align="bottom-right"/>
@@
 <net name="BO2" class="0">
 <segment>
-<pinref part="X13" gate="G$1" pin="8"/>
+<pinref part="X8" gate="G$1" pin="8"/>
 <wire x1="1099.82" y1="782.32" x2="1137.92" y2="782.32" width="0.1524" layer="91"/>
 <label x="1137.92" y="782.32" size="1.778" layer="95" align="bottom-right"/>
@@
 <net name="BO1" class="0">
 <segment>
-<pinref part="X13" gate="G$1" pin="10"/>
+<pinref part="X8" gate="G$1" pin="10"/>
 <wire x1="1099.82" y1="779.78" x2="1137.92" y2="779.78" width="0.1524" layer="91"/>
 <label x="1137.92" y="779.78" size="1.778" layer="95" align="bottom-right"/>

Commit message: Add files via upload
Connections:
- net N$17 renamed 24LIN_IN
Changed lines of the file:
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@@
 </segment>
 </net>
-<net name="N$17" class="0">
+<net name="24LIN_IN" class="0">
 <segment>
 <pinref part="VREG2" gate="A" pin="IN"/>

Commit message: Add files via upload
Connections:
- net 24VDC_AUX: now also X8.11; no longer X8.12, X8.20
- net PMIC_NRESET: now also X8.12; no longer X8.11
Changed lines of the file:
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@@
-</segment>
-<segment>
-<pinref part="X8" gate="G$1" pin="12"/>
-<wire x1="1099.82" y1="777.24" x2="1137.92" y2="777.24" width="0.1524" layer="91"/>
-<label x="1137.92" y="777.24" size="1.778" layer="95" align="bottom-right"/>
 </segment>
 <segment>
@@
 </segment>
 <segment>
-<pinref part="X8" gate="G$1" pin="20"/>
-<wire x1="1099.82" y1="767.08" x2="1137.92" y2="767.08" width="0.1524" layer="91"/>
-<label x="1137.92" y="767.08" size="1.778" layer="95" align="bottom-right"/>
+<pinref part="X8" gate="G$1" pin="11"/>
+<wire x1="1074.42" y1="777.24" x2="1036.32" y2="777.24" width="0.1524" layer="91"/>
+<label x="1036.32" y="777.24" size="1.778" layer="95"/>
 </segment>
 </net>
@@
 </segment>
 <segment>
-<pinref part="X8" gate="G$1" pin="11"/>
-<wire x1="1074.42" y1="777.24" x2="1036.32" y2="777.24" width="0.1524" layer="91"/>
-<label x="1036.32" y="777.24" size="1.778" layer="95"/>
-</segment>
-</net>
+<pinref part="X8" gate="G$1" pin="12"/>
+<wire x1="1099.82" y1="777.24" x2="1137.92" y2="777.24" width="0.1524" layer="91"/>
+<label x="1137.92" y="777.24" size="1.778" layer="95" align="bottom-right"/>
+</segment>
+</net>

Commit message: Add files via upload
Connections:
- net SYS_VDD1_3P3V: no longer C801.1, U28.VCC
- net VDD_5V: now also C801.1, U28.VCC
Changed lines of the file:
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@@
 <part name="U28" library="BeagleBone_Blue" deviceset="TCAN1051HV" device=""/>
 <part name="GND148" library="OSD3358-SM-RED Platform" deviceset="GND" device=""/>
-<part name="SUPPLY121" library="OSD3358-SM-RED Platform" deviceset="SYS_VDD1_3P3V" device=""/>
 <part name="GND149" library="OSD3358-SM-RED Platform" deviceset="GND" device=""/>
 <part name="GND150" library="OSD3358-SM-RED Platform" deviceset="GND" device=""/>
@@
 <part name="GND35" library="OSD3358-SM-RED Platform" deviceset="GND" device=""/>
 <part name="X8" library="OSD3358-SM-RED Platform" deviceset="TH-2X10" device=""/>
+<part name="SUPPLY36" library="OSD3358-SM-RED Platform" deviceset="VDD_5V" device=""/>
 </parts>
 <sheets>
@@
 <attribute name="VALUE" x="878.84" y="675.64" size="1.778" layer="96"/>
 </instance>
-<instance part="SUPPLY121" gate="G$1" x="881.38" y="713.74" smashed="yes">
-<attribute name="VALUE" x="881.38" y="717.804" size="1.778" layer="96" align="center"/>
-</instance>
 <instance part="GND149" gate="1" x="119.38" y="388.62" smashed="yes">
 <attribute name="VALUE" x="116.84" y="386.08" size="1.778" layer="96"/>
@@
 <attribute name="VALUE" x="1079.5" y="762" size="1.778" layer="96" ratio="10"/>
 </instance>
+<instance part="SUPPLY36" gate="G$1" x="881.38" y="711.2" smashed="yes">
+<attribute name="VALUE" x="881.38" y="715.264" size="1.778" layer="96" align="center"/>
+</instance>
 </instances>
 <busses>
@@
 <junction x="121.92" y="226.06"/>
 </segment>
+<segment>
+<pinref part="SUPPLY36" gate="G$1" pin="VDD_5V"/>
+<pinref part="C801" gate="G$1" pin="1"/>
+<wire x1="881.38" y1="708.66" x2="881.38" y2="703.58" width="0.1524" layer="91"/>
+<pinref part="U28" gate="G$1" pin="VCC"/>
+<wire x1="886.46" y1="698.5" x2="886.46" y2="703.58" width="0.1524" layer="91"/>
+<wire x1="886.46" y1="703.58" x2="881.38" y2="703.58" width="0.1524" layer="91"/>
+<junction x="881.38" y="703.58"/>
+</segment>
 </net>
 <net name="PWR_EN" class="0">
@@
 </segment>
 <segment>
-<pinref part="U28" gate="G$1" pin="VCC"/>
-<pinref part="SUPPLY121" gate="G$1" pin="SYS_VDD1_3P3V"/>
-<pinref part="C801" gate="G$1" pin="1"/>
-<wire x1="881.38" y1="703.58" x2="881.38" y2="706.12" width="0.1524" layer="91"/>
-<wire x1="881.38" y1="706.12" x2="881.38" y2="711.2" width="0.1524" layer="91"/>
-<wire x1="886.46" y1="706.12" x2="886.46" y2="698.5" width="0.1524" layer="91"/>
-<wire x1="886.46" y1="706.12" x2="881.38" y2="706.12" width="0.1524" layer="91"/>
-<junction x="881.38" y="706.12"/>
-</segment>
-<segment>

Commit message: Add files via upload
Parts:
- R801, R802: value 1K -> 500
Connections:
- net CAN1_RXD: now also D802.C; no longer D802.A
- net CAN1_TXD: now also D801.C; no longer D801.A
- net GND: no longer R801.2, R802.2
- net N$5: now also D802.A, R802.2; no longer D802.C, R802.1
- net N$6: now also D801.A, R801.2; no longer D801.C, R801.1
- net SYS_VDD1_3P3V: now also U28.VIO
- net VDD_5V: now also R801.1, R802.1
Other:
- moved on the sheet: C801, D801, D802, D805, R801, R802, U28, X31.2, X31.3

Commit message: Add files via upload
Parts:
- added C802: 0.1uF, 6.3V, OSD3358-SM-RED Platform:CC0402
- added C803: 4.7uF, 6.3V, OSD3358-SM-RED Platform:CC0402
Connections:
- net GND: now also C802.2, C803.2
- net SYS_VDD1_3P3V: now also C802.1, R801.1, R802.1
- net VDD_5V: now also C803.1; no longer R801.1, R802.1
Changed lines of the file:
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@@
 <part name="SUPPLY36" library="OSD3358-SM-RED Platform" deviceset="VDD_5V" device=""/>
 <part name="SUPPLY37" library="OSD3358-SM-RED Platform" deviceset="SYS_VDD1_3P3V" device=""/>
+<part name="C802" library="OSD3358-SM-RED Platform" deviceset="C" device="C0402" value="0.1uF, 6.3V"/>
+<part name="GND1" library="OSD3358-SM-RED Platform" deviceset="GND" device=""/>
+<part name="SUPPLY39" library="OSD3358-SM-RED Platform" deviceset="SYS_VDD1_3P3V" device=""/>
+<part name="C803" library="OSD3358-SM-RED Platform" deviceset="C" device="C0402" value="4.7uF, 6.3V"/>
 </parts>
 <sheets>
@@
 </instance>
 <instance part="D801" gate="G$1" x="853.44" y="685.8" smashed="yes">
-<attribute name="NAME" x="855.98" y="685.8" size="1.778" layer="95"/>
-<attribute name="VALUE" x="855.98" y="680.72" size="1.778" layer="96"/>
+<attribute name="NAME" x="850.9" y="685.8" size="1.778" layer="95" align="bottom-right"/>
+<attribute name="VALUE" x="853.44" y="680.72" size="1.778" layer="96" align="bottom-right"/>
 </instance>
 <instance part="D802" gate="G$1" x="830.58" y="685.8" smashed="yes">
-<attribute name="NAME" x="833.12" y="685.8" size="1.778" layer="95"/>
-<attribute name="VALUE" x="833.12" y="680.72" size="1.778" layer="96"/>
+<attribute name="NAME" x="828.04" y="685.8" size="1.778" layer="95" align="bottom-right"/>
+<attribute name="VALUE" x="830.58" y="680.72" size="1.778" layer="96" align="bottom-right"/>
 </instance>
 <instance part="R802" gate="G$1" x="830.58" y="695.96" smashed="yes" rot="R270">
@@
 </instance>
 <instance part="C801" gate="G$1" x="881.38" y="683.26" smashed="yes">
-<attribute name="NAME" x="878.84" y="685.8" size="1.778" layer="95" align="bottom-right"/>
-<attribute name="VALUE" x="878.84" y="678.18" size="1.778" layer="96" align="top-right"/>
+<attribute name="NAME" x="881.38" y="685.8" size="1.778" layer="95" align="bottom-right"/>
+<attribute name="VALUE" x="881.38" y="678.18" size="1.778" layer="96" align="top-right"/>
 </instance>
 <instance part="R303" gate="G$1" x="962.66" y="812.8" smashed="yes" rot="R90">
@@
 <attribute name="VALUE" x="881.38" y="710.184" size="1.778" layer="96" align="center"/>
 </instance>
-<instance part="SUPPLY37" gate="G$1" x="927.1" y="706.12" smashed="yes">
-<attribute name="VALUE" x="927.1" y="710.184" size="1.778" layer="96" align="center"/>
+<instance part="SUPPLY37" gate="G$1" x="929.64" y="706.12" smashed="yes">
+<attribute name="VALUE" x="929.64" y="710.184" size="1.778" layer="96" align="center"/>
+</instance>
+<instance part="C802" gate="G$1" x="929.64" y="683.26" smashed="yes">
+<attribute name="NAME" x="929.64" y="685.8" size="1.778" layer="95"/>
+<attribute name="VALUE" x="929.64" y="678.18" size="1.778" layer="96" align="top-left"/>
+</instance>
+<instance part="GND1" gate="1" x="929.64" y="660.4" smashed="yes">
+<attribute name="VALUE" x="927.1" y="657.86" size="1.778" layer="96"/>
+</instance>
+<instance part="SUPPLY39" gate="G$1" x="838.2" y="706.12" smashed="yes">
+<attribute name="VALUE" x="838.2" y="710.184" size="1.778" layer="96" align="center"/>
+</instance>
+<instance part="C803" gate="G$1" x="866.14" y="683.26" smashed="yes">
+<attribute name="NAME" x="866.14" y="685.8" size="1.778" layer="95" align="bottom-right"/>
+<attribute name="VALUE" x="866.14" y="678.18" size="1.778" layer="96" align="top-right"/>
 </instance>
 </instances>
@@
 <segment>
 <pinref part="SUPPLY36" gate="G$1" pin="VDD_5V"/>
-<pinref part="R802" gate="G$1" pin="1"/>
-<wire x1="881.38" y1="703.58" x2="853.44" y2="703.58" width="0.1524" layer="91"/>
-<wire x1="853.44" y1="703.58" x2="830.58" y2="703.58" width="0.1524" layer="91"/>
-<wire x1="830.58" y1="703.58" x2="830.58" y2="701.04" width="0.1524" layer="91"/>
-<pinref part="R801" gate="G$1" pin="1"/>
-<wire x1="853.44" y1="701.04" x2="853.44" y2="703.58" width="0.1524" layer="91"/>
-<junction x="853.44" y="703.58"/>
 <pinref part="C801" gate="G$1" pin="1"/>
 <wire x1="881.38" y1="703.58" x2="881.38" y2="685.8" width="0.1524" layer="91"/>
@@
 <wire x1="886.46" y1="680.72" x2="886.46" y2="703.58" width="0.1524" layer="91"/>
 <wire x1="886.46" y1="703.58" x2="881.38" y2="703.58" width="0.1524" layer="91"/>
+<wire x1="881.38" y1="703.58" x2="866.14" y2="703.58" width="0.1524" layer="91"/>
+<pinref part="C803" gate="G$1" pin="1"/>
+<wire x1="866.14" y1="703.58" x2="866.14" y2="685.8" width="0.1524" layer="91"/>
 </segment>
 </net>
@@
 <wire x1="881.38" y1="678.18" x2="881.38" y2="665.48" width="0.1524" layer="91"/>
 <junction x="881.38" y="665.48"/>
+<pinref part="C803" gate="G$1" pin="2"/>
+<wire x1="866.14" y1="678.18" x2="866.14" y2="665.48" width="0.1524" layer="91"/>
+<wire x1="866.14" y1="665.48" x2="881.38" y2="665.48" width="0.1524" layer="91"/>
 </segment>
 <segment>
@@
 <junction x="1145.54" y="772.16"/>
 </segment>
+<segment>
+<pinref part="C802" gate="G$1" pin="2"/>
+<pinref part="GND1" gate="1" pin="GND"/>
+<wire x1="929.64" y1="678.18" x2="929.64" y2="662.94" width="0.1524" layer="91"/>
+</segment>
 </net>
 <net name="PWR_BUT" class="0">
@@
 <pinref part="U28" gate="G$1" pin="VIO"/>
 <pinref part="SUPPLY37" gate="G$1" pin="SYS_VDD1_3P3V"/>
-<wire x1="924.56" y1="680.72" x2="927.1" y2="680.72" width="0.1524" layer="91"/>
-<wire x1="927.1" y1="680.72" x2="927.1" y2="703.58" width="0.1524" layer="91"/>
+<wire x1="924.56" y1="680.72" x2="924.56" y2="703.58" width="0.1524" layer="91"/>
+<wire x1="924.56" y1="703.58" x2="929.64" y2="703.58" width="0.1524" layer="91"/>
+<pinref part="C802" gate="G$1" pin="1"/>
+<wire x1="929.64" y1="685.8" x2="929.64" y2="703.58" width="0.1524" layer="91"/>
+<junction x="929.64" y="703.58"/>
+</segment>
+<segment>
+<pinref part="SUPPLY39" gate="G$1" pin="SYS_VDD1_3P3V"/>
+<pinref part="R802" gate="G$1" pin="1"/>
+<wire x1="838.2" y1="703.58" x2="830.58" y2="703.58" width="0.1524" layer="91"/>
+<wire x1="830.58" y1="703.58" x2="830.58" y2="701.04" width="0.1524" layer="91"/>
+<pinref part="R801" gate="G$1" pin="1"/>
+<wire x1="853.44" y1="701.04" x2="853.44" y2="703.58" width="0.1524" layer="91"/>
+<wire x1="853.44" y1="703.58" x2="838.2" y2="703.58" width="0.1524" layer="91"/>
+<junction x="838.2" y="703.58"/>
 </segment>
 </net>
