File: Version_3.0/Open-Source_Control_V3_R0.sch (EAGLE design)
At the start: 349 parts, among them IC10 MCP6002SMT, IC11 MCP6002SMT, IC12 MCP6002SMT, IC14 MCP6002SMT, IC2 ULN2003AD, IC4 74HC165D, IC5 74HC165D, J24 6p-2.54, K1 G5LE-14-CF DC24, K2 G5LE-14-CF DC24, K3 G5LE-14-CF DC24, K4 G5LE-14-CF DC24, Q1 MMBT2907, T4 DA2304-AL, U1 OSD3358-512M-ICB, U16 AT97SC3205T-G3M4400B, U2 TPD4S012_DRY_6_P1_M, U27 LAN8710, U28 TCAN1051HV, U29 MAX3483EESA+T, U4 APX811-31UGSOT, U40 ISO3086TDW, U5 TLVH431, U6 SN74LVC2G241_DCU_8, X1 10118194-0001LF, X10 MC4, X11 MC4, X12 MC4, X2 J0011D01BNL, X21 MC12, X24 MSTBA2, X3 MC4, X31 MC4, X4 CTI-JTAG, X41 MSTBA3, X5 DM3CS-SF, X6 6p-2.54, X7 TH-2X10, X8 TH-2X10, X9 5600200420, Y7 ECS-250-12-30-GN-TR

Commit message: Add files via upload
Parts:
- R801, R802: value 500 -> 1K
Other:
- moved on the sheet: D801, R801
Changed lines of the file:
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@@
 <part name="D801" library="OSD3358-SM-RED Platform" deviceset="LTST-C191KRKT" device="LED_EIA-STD" value="LTST-C191KRKT"/>
 <part name="D802" library="OSD3358-SM-RED Platform" deviceset="LTST-C191KGKT" device="LED_EIA-STD" value="LTST-C191KGKT"/>
-<part name="R802" library="OSD3358-SM-RED Platform" deviceset="R-US_" device="R0402" value="500"/>
-<part name="R801" library="OSD3358-SM-RED Platform" deviceset="R-US_" device="R0402" value="500"/>
+<part name="R802" library="OSD3358-SM-RED Platform" deviceset="R-US_" device="R0402" value="1K"/>
+<part name="R801" library="OSD3358-SM-RED Platform" deviceset="R-US_" device="R0402" value="1K"/>
 <part name="FRAME17" library="OSD3358-SM-RED Platform" deviceset="FRAMES_GEN" device=""/>
 <part name="FRAME1" library="OSD3358-SM-RED Platform" deviceset="FRAMES_GEN" device=""/>
@@
 <attribute name="NAME" x="96.52" y="1071.245" size="1.524" layer="95" rot="MR0"/>
 </instance>
-<instance part="D801" gate="G$1" x="853.44" y="685.8" smashed="yes">
-<attribute name="NAME" x="850.9" y="685.8" size="1.778" layer="95" align="bottom-right"/>
-<attribute name="VALUE" x="853.44" y="680.72" size="1.778" layer="96" align="bottom-right"/>
+<instance part="D801" gate="G$1" x="850.9" y="685.8" smashed="yes">
+<attribute name="NAME" x="848.36" y="685.8" size="1.778" layer="95" align="bottom-right"/>
+<attribute name="VALUE" x="850.9" y="680.72" size="1.778" layer="96" align="bottom-right"/>
 </instance>
 <instance part="D802" gate="G$1" x="830.58" y="685.8" smashed="yes">
@@
 <attribute name="VALUE" x="833.12" y="693.42" size="1.778" layer="96"/>
 </instance>
-<instance part="R801" gate="G$1" x="853.44" y="695.96" smashed="yes" rot="R270">
-<attribute name="NAME" x="855.98" y="698.5" size="1.778" layer="95"/>
-<attribute name="VALUE" x="855.98" y="693.42" size="1.778" layer="96"/>
+<instance part="R801" gate="G$1" x="850.9" y="695.96" smashed="yes" rot="R270">
+<attribute name="NAME" x="853.44" y="698.5" size="1.778" layer="95"/>
+<attribute name="VALUE" x="853.44" y="693.42" size="1.778" layer="96"/>
 </instance>
 <instance part="FRAME17" gate="G$1" x="0" y="0" smashed="yes">
@@
 <pinref part="U28" gate="G$1" pin="TXD"/>
 <label x="815.34" y="675.64" size="1.778" layer="95"/>
-<wire x1="886.46" y1="675.64" x2="853.44" y2="675.64" width="0.1524" layer="91"/>
+<wire x1="886.46" y1="675.64" x2="850.9" y2="675.64" width="0.1524" layer="91"/>
 <pinref part="D801" gate="G$1" pin="C"/>
-<wire x1="853.44" y1="675.64" x2="815.34" y2="675.64" width="0.1524" layer="91"/>
-<wire x1="853.44" y1="680.72" x2="853.44" y2="675.64" width="0.1524" layer="91"/>
-<junction x="853.44" y="675.64"/>
+<wire x1="850.9" y1="675.64" x2="815.34" y2="675.64" width="0.1524" layer="91"/>
+<wire x1="850.9" y1="680.72" x2="850.9" y2="675.64" width="0.1524" layer="91"/>
+<junction x="850.9" y="675.64"/>
 </segment>
 <segment>
@@
 <wire x1="830.58" y1="703.58" x2="830.58" y2="701.04" width="0.1524" layer="91"/>
 <pinref part="R801" gate="G$1" pin="1"/>
-<wire x1="853.44" y1="701.04" x2="853.44" y2="703.58" width="0.1524" layer="91"/>
-<wire x1="853.44" y1="703.58" x2="838.2" y2="703.58" width="0.1524" layer="91"/>
 <junction x="838.2" y="703.58"/>
+<wire x1="850.9" y1="703.58" x2="838.2" y2="703.58" width="0.1524" layer="91"/>
+<wire x1="850.9" y1="701.04" x2="850.9" y2="703.58" width="0.1524" layer="91"/>
 </segment>
 </net>
@@
 <pinref part="R801" gate="G$1" pin="2"/>
 <pinref part="D801" gate="G$1" pin="A"/>
-<wire x1="853.44" y1="690.88" x2="853.44" y2="688.34" width="0.1524" layer="91"/>
+<wire x1="850.9" y1="690.88" x2="850.9" y2="688.34" width="0.1524" layer="91"/>
 </segment>
 </net>

Commit message: Add files via upload
Parts:
- added C901: 0.1uF, 6.3V, OSD3358-SM-RED Platform:CC0402
- added R901, R902: 1.5K, 1% DNI, OSD3358-SM-RED Platform:R-US_R0402
Connections:
- net GND: now also C901.2
- net I2C2_SCL: now also R901.1
- net I2C2_SDA: now also R902.1
- net SYS_VDD1_3P3V: now also C901.1, R901.2, R902.2
Other:
- note added: "Airflow Sensor Conn"
- moved on the sheet: X8, X9
