File: Version_3.0/Open-Source_Control_V3_R0.sch (EAGLE design)
At the start: 352 parts, among them IC10 MCP6002SMT, IC11 MCP6002SMT, IC12 MCP6002SMT, IC14 MCP6002SMT, IC2 ULN2003AD, IC4 74HC165D, IC5 74HC165D, J24 6p-2.54, K1 G5LE-14-CF DC24, K2 G5LE-14-CF DC24, K3 G5LE-14-CF DC24, K4 G5LE-14-CF DC24, Q1 MMBT2907, T4 DA2304-AL, U1 OSD3358-512M-ICB, U16 AT97SC3205T-G3M4400B, U2 TPD4S012_DRY_6_P1_M, U27 LAN8710, U28 TCAN1051HV, U29 MAX3483EESA+T, U4 APX811-31UGSOT, U40 ISO3086TDW, U5 TLVH431, U6 SN74LVC2G241_DCU_8, X1 10118194-0001LF, X10 MC4, X11 MC4, X12 MC4, X2 J0011D01BNL, X21 MC12, X24 MSTBA2, X3 MC4, X31 MC4, X4 CTI-JTAG, X41 MSTBA3, X5 DM3CS-SF, X6 6p-2.54, X7 TH-2X10, X8 TH-2X10, X9 5600200420, Y7 ECS-250-12-30-GN-TR

Commit message: Add files via upload
Connections:
- net 41_A: now also X41-2.1; no longer X41-1.1
- net 41_B: now also X41-1.1; no longer X41-2.1
Other:
- moved on the sheet: X41-1, X41-2, X41-3
Changed lines of the file:
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@@
 <attribute name="VALUE" x="647.7" y="969.264" size="1.778" layer="96" align="center"/>
 </instance>
-<instance part="X41" gate="-1" x="45.72" y="723.9" smashed="yes">
-<attribute name="NAME" x="39.116" y="724.789" size="1.778" layer="95" rot="R180"/>
+<instance part="X41" gate="-1" x="35.56" y="718.82" smashed="yes">
+<attribute name="NAME" x="28.956" y="719.709" size="1.778" layer="95" rot="R180"/>
 </instance>
-<instance part="X41" gate="-2" x="45.72" y="718.82" smashed="yes">
-<attribute name="NAME" x="39.116" y="719.709" size="1.778" layer="95" rot="R180"/>
+<instance part="X41" gate="-2" x="35.56" y="723.9" smashed="yes">
+<attribute name="NAME" x="28.956" y="724.789" size="1.778" layer="95" rot="R180"/>
 </instance>
-<instance part="X41" gate="-3" x="45.72" y="713.74" smashed="yes">
-<attribute name="VALUE" x="38.1" y="709.93" size="1.778" layer="96"/>
-<attribute name="NAME" x="39.116" y="714.629" size="1.778" layer="95" rot="R180"/>
+<instance part="X41" gate="-3" x="35.56" y="728.98" smashed="yes">
+<attribute name="VALUE" x="30.48" y="712.47" size="1.778" layer="96"/>
+<attribute name="NAME" x="28.956" y="729.869" size="1.778" layer="95" rot="R180"/>
 </instance>
 <instance part="VREG4" gate="A" x="114.3" y="772.16" smashed="yes">
@@
 <net name="ISO_GND" class="0">
 <segment>
-<pinref part="X41" gate="-3" pin="1"/>
 <pinref part="SUPPLY106" gate="G$1" pin="ISO_GND"/>
-<wire x1="50.8" y1="713.74" x2="53.34" y2="713.74" width="0.1524" layer="91"/>
-<wire x1="53.34" y1="713.74" x2="53.34" y2="690.88" width="0.1524" layer="91"/>
+<wire x1="53.34" y1="728.98" x2="53.34" y2="690.88" width="0.1524" layer="91"/>
+<pinref part="X41" gate="-3" pin="1"/>
+<wire x1="40.64" y1="728.98" x2="53.34" y2="728.98" width="0.1524" layer="91"/>
 </segment>
 <segment>
@@
 <segment>
 <pinref part="F401" gate="G$1" pin="1"/>
-<pinref part="X41" gate="-1" pin="1"/>
 <wire x1="91.44" y1="723.9" x2="83.82" y2="723.9" width="0.1524" layer="91"/>
 <pinref part="GDT1" gate="G$1" pin="2"/>
-<wire x1="83.82" y1="723.9" x2="50.8" y2="723.9" width="0.1524" layer="91"/>
 <wire x1="83.82" y1="706.12" x2="83.82" y2="723.9" width="0.1524" layer="91"/>
+<pinref part="X41" gate="-2" pin="1"/>
+<wire x1="83.82" y1="723.9" x2="40.64" y2="723.9" width="0.1524" layer="91"/>
 <junction x="83.82" y="723.9"/>
 </segment>
@@
 <segment>
 <pinref part="F402" gate="G$1" pin="1"/>
-<pinref part="X41" gate="-2" pin="1"/>
 <wire x1="91.44" y1="718.82" x2="68.58" y2="718.82" width="0.1524" layer="91"/>
 <pinref part="GDT1" gate="G$1" pin="1"/>
-<wire x1="68.58" y1="718.82" x2="50.8" y2="718.82" width="0.1524" layer="91"/>
 <wire x1="68.58" y1="706.12" x2="68.58" y2="718.82" width="0.1524" layer="91"/>
+<pinref part="X41" gate="-1" pin="1"/>
+<wire x1="68.58" y1="718.82" x2="40.64" y2="718.82" width="0.1524" layer="91"/>
 <junction x="68.58" y="718.82"/>
 </segment>

Commit message: Add files via upload
Connections:
- removed net N$20: D302.C, R302.1
- removed net N$52: D401.C, R401.1
- removed net N$86: D402.C, R402.1
- new net N$16: D402.A, R402.2
- new net N$17: D401.A, R401.2
- new net N$18: D301.A, R301.2
- net 485_RXD: now also D402.C; no longer D402.A
- net 485_TXD: now also D401.C; no longer D401.A
- net GND: no longer R301.2, R302.2, R401.2, R402.2
- net N$19: now also D302.A, R302.2; no longer D301.C, R301.1
- net SYS_VDD1_3P3V: now also R301.1, R302.1, R401.1, R402.1
- net UART2_RXD: now also D302.C; no longer D302.A
- net UART2_TXD: now also D301.C; no longer D301.A
Other:
- moved on the sheet: C301, D301, D302, D305, D401, D402, R301, R302, R303, R304, R305, R401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

Commit message: Add files via upload
Connections:
- net 41_A: now also F402.1, GDT1.1; no longer F401.1, GDT1.2
- net 41_B: now also F401.1, GDT1.2; no longer F402.1, GDT1.1
- net ISO_485_A: now also D405.2, F402.3; no longer D405.1, F401.3
- net ISO_485_B: now also D405.1, F401.3; no longer D405.2, F402.3
Other:
- moved on the sheet: D405, F401, F402, GDT1, X41-1, X41-2, X41-3

Commit message: Add files via upload
Parts:
- R169, R170: value 1.5K, 1% -> 10K, 1%
Changed lines of the file:
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@@
 <part name="R164" library="OSD3358-SM-RED Platform" deviceset="R-US_" device="R0402" value="1.5K, 1%"/>
 <part name="SUPPLY129" library="OSD3358-SM-RED Platform" deviceset="SYS_VDD1_3P3V" device=""/>
-<part name="R169" library="OSD3358-SM-RED Platform" deviceset="R-US_" device="R0402" value="1.5K, 1%"/>
-<part name="R170" library="OSD3358-SM-RED Platform" deviceset="R-US_" device="R0402" value="1.5K, 1%"/>
+<part name="R169" library="OSD3358-SM-RED Platform" deviceset="R-US_" device="R0402" value="10K, 1%"/>
+<part name="R170" library="OSD3358-SM-RED Platform" deviceset="R-US_" device="R0402" value="10K, 1%"/>
 <part name="GND159" library="OSD3358-SM-RED Platform" deviceset="GND" device=""/>
 <part name="J3" library="OSD3358-SM-RED Platform" deviceset="826646-2" device=""/>

Commit message: Add files via upload
Parts:
- removed MGT1, MGT2, MGT3, MGT4: MOUNTING_HOLE, OSD3358-SM-RED Platform:MOUNTING_HOLE
- added H4, MTG1, MTG2, MTG3: MOUNT-PAD-ROUND3.6, holes:MOUNT-PAD-ROUND3.6
Connections:
- net CGND: now also H4.MOUNT, MTG1.MOUNT, MTG2.MOUNT, MTG3.MOUNT; no longer MGT1.P$1, MGT2.P$1, MGT3.P$1, MGT4.P$1
Changed lines of the file:
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@@
 <part name="C22" library="OSD3358-SM-RED Platform" deviceset="C" device="C0402" value="0.1uF, 6.3V"/>
 <part name="R92" library="OSD3358-SM-RED Platform" deviceset="R-US_" device="R0402" value="10K, 1%"/>
-<part name="MGT1" library="OSD3358-SM-RED Platform" deviceset="MOUNTING_HOLE" device=""/>
-<part name="MGT2" library="OSD3358-SM-RED Platform" deviceset="MOUNTING_HOLE" device=""/>
-<part name="MGT3" library="OSD3358-SM-RED Platform" deviceset="MOUNTING_HOLE" device=""/>
-<part name="MGT4" library="OSD3358-SM-RED Platform" deviceset="MOUNTING_HOLE" device=""/>
 <part name="SUPPLY21" library="OSD3358-SM-RED Platform" deviceset="CGND" device=""/>
 <part name="TP8" library="OSD3358-SM-RED Platform" deviceset="TESTPAD/W_HOLE_1X1" device=""/>
@@
 <part name="SUPPLY40" library="OSD3358-SM-RED Platform" deviceset="SYS_VDD1_3P3V" device=""/>
 <part name="SUPPLY41" library="OSD3358-SM-RED Platform" deviceset="SYS_VDD1_3P3V" device=""/>
+<part name="MTG1" library="holes" library_urn="urn:adsk.eagle:library:237" deviceset="MOUNT-PAD-ROUND" device="3.6" package3d_urn="urn:adsk.eagle:package:14284/1"/>
+<part name="MTG2" library="holes" library_urn="urn:adsk.eagle:library:237" deviceset="MOUNT-PAD-ROUND" device="3.6" package3d_urn="urn:adsk.eagle:package:14284/1"/>
+<part name="MTG3" library="holes" library_urn="urn:adsk.eagle:library:237" deviceset="MOUNT-PAD-ROUND" device="3.6" package3d_urn="urn:adsk.eagle:package:14284/1"/>
+<part name="H4" library="holes" library_urn="urn:adsk.eagle:library:237" deviceset="MOUNT-PAD-ROUND" device="3.6" package3d_urn="urn:adsk.eagle:package:14284/1"/>
 </parts>
 <sheets>
@@
 YOU. SHOULD THE DESIGN PROVE DEFECTIVE, YOU ASSUME THE
 COST OF ALL NECESSARY SERVICING, REPAIR OR CORRECTION. </text>
-<text x="99.06" y="337.82" size="2.54" layer="150">Mounting holes and other connector shields are part
+<text x="48.26" y="314.96" size="2.54" layer="150">Mounting holes and other connector shields are part
 of a ground ring, CGND.  This ring is connected to
 ground via a resistor on Page 1.</text>
@@
 <attribute name="VALUE" x="725.17" y="497.84" size="1.778" layer="96" rot="R90"/>
 </instance>
-<instance part="MGT1" gate="G$1" x="38.1" y="345.44" smashed="yes">
-<attribute name="NAME" x="38.862" y="343.408" size="1.27" layer="95"/>
-</instance>
-<instance part="MGT2" gate="G$1" x="53.34" y="345.44" smashed="yes">
-<attribute name="NAME" x="54.102" y="343.408" size="1.27" layer="95"/>
-</instance>
-<instance part="MGT3" gate="G$1" x="68.58" y="345.44" smashed="yes">
-<attribute name="NAME" x="69.342" y="343.408" size="1.27" layer="95"/>
-</instance>
-<instance part="MGT4" gate="G$1" x="83.82" y="345.44" smashed="yes">
-<attribute name="NAME" x="84.582" y="343.408" size="1.27" layer="95"/>
-</instance>
-<instance part="SUPPLY21" gate="G$1" x="83.82" y="327.66" smashed="yes">
-<attribute name="VALUE" x="83.82" y="324.104" size="1.778" layer="96" align="center"/>
+<instance part="SUPPLY21" gate="G$1" x="38.1" y="327.66" smashed="yes">
+<attribute name="VALUE" x="38.1" y="324.104" size="1.778" layer="96" align="center"/>
 </instance>
 <instance part="TP8" gate="G$1" x="104.14" y="182.88" smashed="yes" rot="R180">
@@
 <attribute name="VALUE" x="845.82" y="827.024" size="1.778" layer="96" align="center"/>
 </instance>
+<instance part="MTG1" gate="G$1" x="45.72" y="337.82" smashed="yes">
+<attribute name="NAME" x="48.514" y="338.4042" size="1.778" layer="95"/>
+<attribute name="VALUE" x="48.514" y="335.3562" size="1.778" layer="96"/>
+</instance>
+<instance part="MTG2" gate="G$1" x="83.82" y="337.82" smashed="yes">
+<attribute name="NAME" x="86.614" y="338.4042" size="1.778" layer="95"/>
+<attribute name="VALUE" x="86.614" y="335.3562" size="1.778" layer="96"/>
+</instance>
+<instance part="MTG3" gate="G$1" x="45.72" y="353.06" smashed="yes">
+<attribute name="NAME" x="48.514" y="353.6442" size="1.778" layer="95"/>
+<attribute name="VALUE" x="48.514" y="350.5962" size="1.778" layer="96"/>
+</instance>
+<instance part="H4" gate="G$1" x="83.82" y="353.06" smashed="yes">
+<attribute name="NAME" x="86.614" y="353.6442" size="1.778" layer="95"/>
+<attribute name="VALUE" x="86.614" y="350.5962" size="1.778" layer="96"/>
+</instance>
 </instances>
 <busses>
@@
 <net name="CGND" class="0">
 <segment>
-<pinref part="MGT1" gate="G$1" pin="P$1"/>
-<wire x1="38.1" y1="340.36" x2="38.1" y2="335.28" width="0.1524" layer="91"/>
-<pinref part="SUPPLY21" gate="G$1" pin="CGND"/>
-<wire x1="38.1" y1="335.28" x2="53.34" y2="335.28" width="0.1524" layer="91"/>
-<pinref part="MGT2" gate="G$1" pin="P$1"/>
-<wire x1="53.34" y1="335.28" x2="68.58" y2="335.28" width="0.1524" layer="91"/>
-<wire x1="68.58" y1="335.28" x2="83.82" y2="335.28" width="0.1524" layer="91"/>
-<wire x1="83.82" y1="335.28" x2="83.82" y2="330.2" width="0.1524" layer="91"/>
-<wire x1="53.34" y1="340.36" x2="53.34" y2="335.28" width="0.1524" layer="91"/>
-<pinref part="MGT3" gate="G$1" pin="P$1"/>
-<wire x1="68.58" y1="340.36" x2="68.58" y2="335.28" width="0.1524" layer="91"/>
-<pinref part="MGT4" gate="G$1" pin="P$1"/>
-<wire x1="83.82" y1="340.36" x2="83.82" y2="335.28" width="0.1524" layer="91"/>
-<junction x="83.82" y="335.28"/>
-<junction x="68.58" y="335.28"/>
-<junction x="53.34" y="335.28"/>
-</segment>
-<segment>
 <pinref part="SUPPLY1" gate="G$1" pin="CGND"/>
 <wire x1="454.66" y1="81.28" x2="447.04" y2="81.28" width="0.1524" layer="91"/>
@@
 <junction x="637.54" y="464.82"/>
 </segment>
+<segment>
+<pinref part="SUPPLY21" gate="G$1" pin="CGND"/>
+<wire x1="76.2" y1="330.2" x2="38.1" y2="330.2" width="0.1524" layer="91"/>
+<wire x1="38.1" y1="330.2" x2="38.1" y2="337.82" width="0.1524" layer="91"/>
+<pinref part="MTG1" gate="G$1" pin="MOUNT"/>
+<wire x1="38.1" y1="337.82" x2="43.18" y2="337.82" width="0.1524" layer="91"/>
+<pinref part="MTG2" gate="G$1" pin="MOUNT"/>
+<wire x1="81.28" y1="337.82" x2="76.2" y2="337.82" width="0.1524" layer="91"/>
+<wire x1="76.2" y1="337.82" x2="76.2" y2="330.2" width="0.1524" layer="91"/>
+<pinref part="H4" gate="G$1" pin="MOUNT"/>
+<wire x1="81.28" y1="353.06" x2="76.2" y2="353.06" width="0.1524" layer="91"/>
+<wire x1="76.2" y1="353.06" x2="76.2" y2="337.82" width="0.1524" layer="91"/>
+<junction x="76.2" y="337.82"/>
+<pinref part="MTG3" gate="G$1" pin="MOUNT"/>
+<wire x1="43.18" y1="353.06" x2="38.1" y2="353.06" width="0.1524" layer="91"/>
+<wire x1="38.1" y1="353.06" x2="38.1" y2="337.82" width="0.1524" layer="91"/>
+<junction x="38.1" y="337.82"/>
+<junction x="38.1" y="330.2"/>
+</segment>
 </net>

Commit message: Add files via upload
Parts:
- renumbered H4 to MTG4
Changed lines of the file:
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@@
 <part name="MTG2" library="holes" library_urn="urn:adsk.eagle:library:237" deviceset="MOUNT-PAD-ROUND" device="3.6" package3d_urn="urn:adsk.eagle:package:14284/1"/>
 <part name="MTG3" library="holes" library_urn="urn:adsk.eagle:library:237" deviceset="MOUNT-PAD-ROUND" device="3.6" package3d_urn="urn:adsk.eagle:package:14284/1"/>
-<part name="H4" library="holes" library_urn="urn:adsk.eagle:library:237" deviceset="MOUNT-PAD-ROUND" device="3.6" package3d_urn="urn:adsk.eagle:package:14284/1"/>
+<part name="MTG4" library="holes" library_urn="urn:adsk.eagle:library:237" deviceset="MOUNT-PAD-ROUND" device="3.6" package3d_urn="urn:adsk.eagle:package:14284/1"/>
 </parts>
 <sheets>
@@
 <attribute name="VALUE" x="48.514" y="350.5962" size="1.778" layer="96"/>
 </instance>
-<instance part="H4" gate="G$1" x="83.82" y="353.06" smashed="yes">
+<instance part="MTG4" gate="G$1" x="83.82" y="353.06" smashed="yes">
 <attribute name="NAME" x="86.614" y="353.6442" size="1.778" layer="95"/>
 <attribute name="VALUE" x="86.614" y="350.5962" size="1.778" layer="96"/>
@@
 <wire x1="81.28" y1="337.82" x2="76.2" y2="337.82" width="0.1524" layer="91"/>
 <wire x1="76.2" y1="337.82" x2="76.2" y2="330.2" width="0.1524" layer="91"/>
-<pinref part="H4" gate="G$1" pin="MOUNT"/>
+<pinref part="MTG4" gate="G$1" pin="MOUNT"/>
 <wire x1="81.28" y1="353.06" x2="76.2" y2="353.06" width="0.1524" layer="91"/>
 <wire x1="76.2" y1="353.06" x2="76.2" y2="337.82" width="0.1524" layer="91"/>

Commit message: Add files via upload
Fixed CAN1_TXD CAN1_RXD criss-crossed
Connections:
- net CAN1_RXD: now also U1C.UART1_TXD; no longer U1C.UART1_RXD
- net CAN1_TXD: now also U1C.UART1_RXD; no longer U1C.UART1_TXD
Changed lines of the file:
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@@
 </segment>
 </net>
-<net name="CAN1_TXD" class="0">
-<segment>
-<pinref part="U28" gate="G$1" pin="TXD"/>
-<label x="815.34" y="675.64" size="1.778" layer="95"/>
-<wire x1="886.46" y1="675.64" x2="850.9" y2="675.64" width="0.1524" layer="91"/>
-<pinref part="D801" gate="G$1" pin="C"/>
-<wire x1="850.9" y1="675.64" x2="815.34" y2="675.64" width="0.1524" layer="91"/>
-<wire x1="850.9" y1="680.72" x2="850.9" y2="675.64" width="0.1524" layer="91"/>
-<junction x="850.9" y="675.64"/>
-</segment>
+<net name="CAN1_RXD" class="0">
 <segment>
 <pinref part="U1" gate="C" pin="UART1_TXD"/>
@@
 <label x="861.06" y="119.38" size="1.778" layer="95"/>
 </segment>
-</net>
-<net name="CAN1_RXD" class="0">
 <segment>
 <pinref part="U28" gate="G$1" pin="RXD"/>
 <wire x1="886.46" y1="673.1" x2="830.58" y2="673.1" width="0.1524" layer="91"/>
-<label x="815.34" y="673.1" size="1.778" layer="95"/>
+<label x="810.26" y="673.1" size="1.778" layer="95"/>
 <pinref part="D802" gate="G$1" pin="C"/>
-<wire x1="830.58" y1="673.1" x2="815.34" y2="673.1" width="0.1524" layer="91"/>
+<wire x1="830.58" y1="673.1" x2="810.26" y2="673.1" width="0.1524" layer="91"/>
 <wire x1="830.58" y1="680.72" x2="830.58" y2="673.1" width="0.1524" layer="91"/>
 <junction x="830.58" y="673.1"/>
 </segment>
+</net>
+<net name="CAN1_TXD" class="0">
 <segment>
 <pinref part="U1" gate="C" pin="UART1_RXD"/>
@@
 <label x="861.06" y="116.84" size="1.778" layer="95"/>
 </segment>
+<segment>
+<pinref part="U28" gate="G$1" pin="TXD"/>
+<wire x1="886.46" y1="675.64" x2="850.9" y2="675.64" width="0.1524" layer="91"/>
+<label x="810.26" y="675.64" size="1.778" layer="95"/>
+<pinref part="D801" gate="G$1" pin="C"/>
+<wire x1="850.9" y1="675.64" x2="810.26" y2="675.64" width="0.1524" layer="91"/>
+<wire x1="850.9" y1="680.72" x2="850.9" y2="675.64" width="0.1524" layer="91"/>
+<junction x="850.9" y="675.64"/>
+</segment>
 </net>

Commit message: Added 6th B-output BO_6
Added 6th B-output BO_6 to expansion header. Now a total of 6 relay outputs are possible
Connections:
- new net BO6_AUTO: IC2.O6, X8.12
- net GPIO1_16: now also IC2.I6, U1C.GPMC_A0; no longer U1C.GPMC_CSN3
- net PMIC_NRESET: now also X8.18; no longer X8.12
Changed lines of the file:
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@@
 <pinref part="GND31" gate="1" pin="GND"/>
 <wire x1="1145.54" y1="759.46" x2="1145.54" y2="764.54" width="0.1524" layer="91"/>
-<pinref part="X8" gate="G$1" pin="2"/>
-<wire x1="1145.54" y1="764.54" x2="1145.54" y2="782.32" width="0.1524" layer="91"/>
-<wire x1="1099.82" y1="782.32" x2="1145.54" y2="782.32" width="0.1524" layer="91"/>
 <pinref part="X8" gate="G$1" pin="16"/>
 <wire x1="1099.82" y1="764.54" x2="1145.54" y2="764.54" width="0.1524" layer="91"/>
+<pinref part="X8" gate="G$1" pin="2"/>
+<wire x1="1099.82" y1="782.32" x2="1145.54" y2="782.32" width="0.1524" layer="91"/>
+<wire x1="1145.54" y1="782.32" x2="1145.54" y2="764.54" width="0.1524" layer="91"/>
 <junction x="1145.54" y="764.54"/>
 </segment>
@@
 </segment>
 </net>
-<net name="GPIO1_16" class="0">
-<segment>
-<pinref part="U1" gate="C" pin="GPMC_CSN3"/>
-<wire x1="975.36" y1="81.28" x2="1031.24" y2="81.28" width="0.1524" layer="91"/>
-<label x="1018.54" y="81.28" size="1.778" layer="95"/>
-</segment>
-</net>
 <net name="XDMA_EVENT_INTR0" class="0">
 <segment>
@@
 </segment>
 <segment>
-<pinref part="X8" gate="G$1" pin="12"/>
-<wire x1="1099.82" y1="769.62" x2="1137.92" y2="769.62" width="0.1524" layer="91"/>
-<label x="1137.92" y="769.62" size="1.778" layer="95" align="bottom-right"/>
+<pinref part="X8" gate="G$1" pin="18"/>
+<wire x1="1099.82" y1="762" x2="1137.92" y2="762" width="0.1524" layer="91"/>
+<label x="1120.14" y="762" size="1.778" layer="95"/>
 </segment>
 </net>
@@
 </segment>
 </net>
+<net name="GPIO1_16" class="0">
+<segment>
+<pinref part="U1" gate="C" pin="GPMC_A0"/>
+<wire x1="975.36" y1="129.54" x2="1031.24" y2="129.54" width="0.1524" layer="91"/>
+<label x="1018.54" y="129.54" size="1.778" layer="95"/>
+</segment>
+<segment>
+<pinref part="IC2" gate="A" pin="I6"/>
+<wire x1="886.46" y1="967.74" x2="845.82" y2="967.74" width="0.1524" layer="91"/>
+<label x="845.82" y="967.74" size="1.778" layer="95"/>
+</segment>
+</net>
+<net name="BO6_AUTO" class="0">
+<segment>
+<pinref part="IC2" gate="A" pin="O6"/>
+<wire x1="911.86" y1="967.74" x2="955.04" y2="967.74" width="0.1524" layer="91"/>
+<label x="939.8" y="967.74" size="1.778" layer="95"/>
+</segment>
+<segment>
+<pinref part="X8" gate="G$1" pin="12"/>
+<wire x1="1099.82" y1="769.62" x2="1137.92" y2="769.62" width="0.1524" layer="91"/>
+<label x="1125.22" y="769.62" size="1.778" layer="95"/>
+</segment>
+</net>
